File: template/template.kicad_pcb (KiCad board)
At the start: 2 copper layers, 88.9 x 30.5 mm, 5 parts, among them J1 Conn_01x08_Male, J2 Conn_01x08_Male, J3 Conn_01x08_Male, J4 Conn_01x04_Male

Commit message: Add latch
Parts:
- added U1: 74LS573, Package_DIP:DIP-20_W7.62mm, F.Cu at (104.1, 45.7)
- moved C1 5.08 mm to (108.0, 58.4), turned to 0 degrees
Connections:
- J4 pad 2: VCC -> GND
- J4 pad 3: GND -> VCC
Routing:
- net GND: track 0.00 -> 49.9 mm
- net Net-(J4-Pad4): track 0.00 -> 40.5 mm
- net Net-(J4-Pad1): track 0.00 -> 29.6 mm
- net VCC: track 0.00 -> 12.9 mm
- net Net-(J3-Pad8): track 0.00 -> 10.8 mm
- net Net-(J3-Pad7): track 0.00 -> 10.8 mm
- net Net-(J3-Pad6): track 0.00 -> 10.8 mm
- net Net-(J3-Pad5): track 0.00 -> 10.8 mm
- net Net-(J3-Pad4): track 0.00 -> 10.8 mm
- net Net-(J3-Pad3): track 0.00 -> 10.8 mm
- net Net-(J3-Pad2): track 0.00 -> 10.8 mm
- net Net-(J3-Pad1): track 0.00 -> 10.8 mm
Changed lines of the file:
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@@
     (thickness 1.6)
     (drawings 4)
-    (tracks 0)
+    (tracks 28)
     (zones 0)
-    (modules 5)
-    (nets 29)
+    (modules 6)
+    (nets 37)
   )
   (page A4 portrait)
@@
   )
   (setup
-    (last_trace_width 0.25)
+    (last_trace_width 0.5)
+    (user_trace_width 0.5)
+    (user_trace_width 0.6)
+    (user_trace_width 0.8)
     (trace_clearance 0.2)
     (zone_clearance 0.508)
@@
   (net 27 VCC)
   (net 28 GND)
+  (net 29 "Net-(U1-Pad2)")
+  (net 30 "Net-(U1-Pad3)")
+  (net 31 "Net-(U1-Pad4)")
+  (net 32 "Net-(U1-Pad5)")
+  (net 33 "Net-(U1-Pad6)")
+  (net 34 "Net-(U1-Pad7)")
+  (net 35 "Net-(U1-Pad8)")
+  (net 36 "Net-(U1-Pad9)")
   (net_class Default "This is the default net class."
     (clearance 0.2)
@@
     (add_net "Net-(J4-Pad1)")
     (add_net "Net-(J4-Pad4)")
+    (add_net "Net-(U1-Pad2)")
+    (add_net "Net-(U1-Pad3)")
+    (add_net "Net-(U1-Pad4)")
+    (add_net "Net-(U1-Pad5)")
+    (add_net "Net-(U1-Pad6)")
+    (add_net "Net-(U1-Pad7)")
+    (add_net "Net-(U1-Pad8)")
+    (add_net "Net-(U1-Pad9)")
     (add_net VCC)
   )
@@
       (net 25 "Net-(J4-Pad4)"))
     (pad 3 thru_hole oval (at 0 5.08 270) (size 1.7 1.7) (drill 1) (layers *.Cu *.Mask)
+      (net 27 VCC))
+    (pad 2 thru_hole oval (at 0 2.54 270) (size 1.7 1.7) (drill 1) (layers *.Cu *.Mask)
       (net 28 GND))
-    (pad 2 thru_hole oval (at 0 2.54 270) (size 1.7 1.7) (drill 1) (layers *.Cu *.Mask)
-      (net 27 VCC))
     (pad 1 thru_hole rect (at 0 0 270) (size 1.7 1.7) (drill 1) (layers *.Cu *.Mask)
       (net 26 "Net-(J4-Pad1)"))
@@
   )
   (module Capacitor_THT:C_Disc_D4.7mm_W2.5mm_P5.00mm (layer F.Cu)
-    (at 113.03 58.42 180)
+    (at 107.95 58.42)
     (descr "C, Disc series, Radial, pin pitch=5.00mm, , diameter*width=4.7*2.5mm^2, Capacitor, http://www.vishay.com/docs/45233/krseries.pdf")
     (tags "C Disc series Radial pin pitch 5.00mm  diameter 4.7mm width 2.5mm Capacitor")
@@
       (effects (font (size 0.94 0.94) (thickness 0.141)))
     )
-    (pad 1 thru_hole circle (at 0 0 180) (size 1.6 1.6) (drill 0.8) (layers *.Cu *.Mask)
+    (pad 1 thru_hole circle (at 0 0) (size 1.6 1.6) (drill 0.8) (layers *.Cu *.Mask)
       (net 27 VCC))
-    (pad 2 thru_hole circle (at 5 0 180) (size 1.6 1.6) (drill 0.8) (layers *.Cu *.Mask)
+    (pad 2 thru_hole circle (at 5 0) (size 1.6 1.6) (drill 0.8) (layers *.Cu *.Mask)
       (net 28 GND))
     (model ${KISYS3DMOD}/Capacitor_THT.3dshapes/C_Disc_D4.7mm_W2.5mm_P5.00mm.wrl
@@
     )
   )
-  (gr_line (start 31.75 35.56) (end 31.75 66.04) (layer Edge.Cuts) (width 0.05))
-  (gr_line (start 120.65 35.56) (end 31.75 35.56) (layer Edge.Cuts) (width 0.05))
-  (gr_line (start 120.65 66.04) (end 120.65 35.56) (layer Edge.Cuts) (width 0.05))
-  (gr_line (start 31.75 66.04) (end 120.65 66.04) (layer Edge.Cuts) (width 0.05))
+  (module Package_DIP:DIP-20_W7.62mm (layer F.Cu)
+    (at 104.14 45.72 270)
+    (descr "20-lead though-hole mounted DIP package, row spacing 7.62 mm (300 mils)")
+    (tags "THT DIP DIL PDIP 2.54mm 7.62mm 300mil")
+    (fp_text reference U1 (at 3.81 -2.33 90) (layer F.SilkS)
+      (effects (font (size 1 1) (thickness 0.15)))
+    )
+    (fp_text value 74LS573 (at 3.81 25.19 90) (layer F.Fab)
+      (effects (font (size 1 1) (thickness 0.15)))
+    )
+    (fp_arc (start 3.81 -1.33) (end 2.81 -1.33) (angle -180) (layer F.SilkS) (width 0.12))
+    (fp_line (start 1.635 -1.27) (end 6.985 -1.27) (layer F.Fab) (width 0.1))
+    (fp_line (start 6.985 -1.27) (end 6.985 24.13) (layer F.Fab) (width 0.1))
+    (fp_line (start 6.985 24.13) (end 0.635 24.13) (layer F.Fab) (width 0.1))
+    (fp_line (start 0.635 24.13) (end 0.635 -0.27) (layer F.Fab) (width 0.1))
+    (fp_line (start 0.635 -0.27) (end 1.635 -1.27) (layer F.Fab) (width 0.1))
+    (fp_line (start 2.81 -1.33) (end 1.16 -1.33) (layer F.SilkS) (width 0.12))
+    (fp_line (start 1.16 -1.33) (end 1.16 24.19) (layer F.SilkS) (width 0.12))
+    (fp_line (start 1.16 24.19) (end 6.46 24.19) (layer F.SilkS) (width 0.12))
+    (fp_line (start 6.46 24.19) (end 6.46 -1.33) (layer F.SilkS) (width 0.12))
+    (fp_line (start 6.46 -1.33) (end 4.81 -1.33) (layer F.SilkS) (width 0.12))
+    (fp_line (start -1.1 -1.55) (end -1.1 24.4) (layer F.CrtYd) (width 0.05))
+    (fp_line (start -1.1 24.4) (end 8.7 24.4) (layer F.CrtYd) (width 0.05))
+    (fp_line (start 8.7 24.4) (end 8.7 -1.55) (layer F.CrtYd) (width 0.05))
+    (fp_line (start 8.7 -1.55) (end -1.1 -1.55) (layer F.CrtYd) (width 0.05))
+    (fp_text user %R (at 3.81 11.43 90) (layer F.Fab)
+      (effects (font (size 1 1) (thickness 0.15)))
+    )
+    (pad 1 thru_hole rect (at 0 0 270) (size 1.6 1.6) (drill 0.8) (layers *.Cu *.Mask)
+      (net 26 "Net-(J4-Pad1)"))
+    (pad 11 thru_hole oval (at 7.62 22.86 270) (size 1.6 1.6) (drill 0.8) (layers *.Cu *.Mask)
+      (net 25 "Net-(J4-Pad4)"))
+    (pad 2 thru_hole oval (at 0 2.54 270) (size 1.6 1.6) (drill 0.8) (layers *.Cu *.Mask)
+      (net 29 "Net-(U1-Pad2)"))
+    (pad 12 thru_hole oval (at 7.62 20.32 270) (size 1.6 1.6) (drill 0.8) (layers *.Cu *.Mask)
+      (net 17 "Net-(J3-Pad8)"))
+    (pad 3 thru_hole oval (at 0 5.08 270) (size 1.6 1.6) (drill 0.8) (layers *.Cu *.Mask)
+      (net 30 "Net-(U1-Pad3)"))
+    (pad 13 thru_hole oval (at 7.62 17.78 270) (size 1.6 1.6) (drill 0.8) (layers *.Cu *.Mask)
+      (net 18 "Net-(J3-Pad7)"))
+    (pad 4 thru_hole oval (at 0 7.62 270) (size 1.6 1.6) (drill 0.8) (layers *.Cu *.Mask)
+      (net 31 "Net-(U1-Pad4)"))
+    (pad 14 thru_hole oval (at 7.62 15.24 270) (size 1.6 1.6) (drill 0.8) (layers *.Cu *.Mask)
+      (net 19 "Net-(J3-Pad6)"))
+    (pad 5 thru_hole oval (at 0 10.16 270) (size 1.6 1.6) (drill 0.8) (layers *.Cu *.Mask)
+      (net 32 "Net-(U1-Pad5)"))
+    (pad 15 thru_hole oval (at 7.62 12.7 270) (size 1.6 1.6) (drill 0.8) (layers *.Cu *.Mask)
+      (net 20 "Net-(J3-Pad5)"))
+    (pad 6 thru_hole oval (at 0 12.7 270) (size 1.6 1.6) (drill 0.8) (layers *.Cu *.Mask)
+      (net 33 "Net-(U1-Pad6)"))
+    (pad 16 thru_hole oval (at 7.62 10.16 270) (size 1.6 1.6) (drill 0.8) (layers *.Cu *.Mask)
+      (net 21 "Net-(J3-Pad4)"))
+    (pad 7 thru_hole oval (at 0 15.24 270) (size 1.6 1.6) (drill 0.8) (layers *.Cu *.Mask)
+      (net 34 "Net-(U1-Pad7)"))
+    (pad 17 thru_hole oval (at 7.62 7.62 270) (size 1.6 1.6) (drill 0.8) (layers *.Cu *.Mask)
+      (net 22 "Net-(J3-Pad3)"))
+    (pad 8 thru_hole oval (at 0 17.78 270) (size 1.6 1.6) (drill 0.8) (layers *.Cu *.Mask)
+      (net 35 "Net-(U1-Pad8)"))
+    (pad 18 thru_hole oval (at 7.62 5.08 270) (size 1.6 1.6) (drill 0.8) (layers *.Cu *.Mask)
+      (net 23 "Net-(J3-Pad2)"))
+    (pad 9 thru_hole oval (at 0 20.32 270) (size 1.6 1.6) (drill 0.8) (layers *.Cu *.Mask)
+      (net 36 "Net-(U1-Pad9)"))
+    (pad 19 thru_hole oval (at 7.62 2.54 270) (size 1.6 1.6) (drill 0.8) (layers *.Cu *.Mask)
+      (net 24 "Net-(J3-Pad1)"))
+    (pad 10 thru_hole oval (at 0 22.86 270) (size 1.6 1.6) (drill 0.8) (layers *.Cu *.Mask)
+      (net 28 GND))
+    (pad 20 thru_hole oval (at 7.62 0 270) (size 1.6 1.6) (drill 0.8) (layers *.Cu *.Mask)
+      (net 27 VCC))
+    (model ${KISYS3DMOD}/Package_DIP.3dshapes/DIP-20_W7.62mm.wrl
+      (at (xyz 0 0 0))
+      (scale (xyz 1 1 1))
+      (rotate (xyz 0 0 0))
+    )
+  )
+  (gr_line (start 31.75 36.83) (end 31.75 67.31) (layer Edge.Cuts) (width 0.05))
+  (gr_line (start 120.65 36.83) (end 31.75 36.83) (layer Edge.Cuts) (width 0.05))
+  (gr_line (start 120.65 67.31) (end 120.65 36.83) (layer Edge.Cuts) (width 0.05))
+  (gr_line (start 31.75 67.31) (end 120.65 67.31) (layer Edge.Cuts) (width 0.05))
+  (segment (start 83.82 53.34) (end 83.82 64.135) (width 0.8) (layer B.Cu) (net 17))
+  (segment (start 86.36 53.34) (end 86.36 64.135) (width 0.8) (layer B.Cu) (net 18))
+  (segment (start 88.9 53.34) (end 88.9 64.135) (width 0.8) (layer B.Cu) (net 19))
+  (segment (start 91.44 53.34) (end 91.44 64.135) (width 0.8) (layer B.Cu) (net 20))
+  (segment (start 93.98 53.34) (end 93.98 64.135) (width 0.8) (layer B.Cu) (net 21))
+  (segment (start 96.52 53.34) (end 96.52 64.135) (width 0.8) (layer B.Cu) (net 22))
+  (segment (start 99.06 53.34) (end 99.06 64.135) (width 0.8) (layer B.Cu) (net 23))
+  (segment (start 101.6 53.34) (end 101.6 64.135) (width 0.8) (layer B.Cu) (net 24))
+  (segment (start 81.28 53.34) (end 81.28 66.04) (width 0.6) (layer B.Cu) (net 25))
+  (segment (start 81.28 66.04) (end 81.915 66.675) (width 0.6) (layer B.Cu) (net 25))
+  (segment (start 81.915 66.675) (end 106.045 66.675) (width 0.6) (layer B.Cu) (net 25))
+  (segment (start 106.045 66.675) (end 106.68 66.04) (width 0.6) (layer B.Cu) (net 25))
+  (segment (start 106.68 66.04) (end 106.68 64.135) (width 0.6) (layer B.Cu) (net 25))
+  (segment (start 114.3 64.135) (end 114.3 60.96) (width 0.8) (layer B.Cu) (net 26))
+  (segment (start 114.3 60.96) (end 115.57 59.69) (width 0.8) (layer B.Cu) (net 26))
+  (segment (start 115.57 59.69) (end 115.57 46.99) (width 0.8) (layer B.Cu) (net 26))
+  (segment (start 114.3 45.72) (end 104.14 45.72) (width 0.8) (layer B.Cu) (net 26))
+  (segment (start 115.57 46.99) (end 114.3 45.72) (width 0.8) (layer B.Cu) (net 26))
+  (segment (start 109.22 59.69) (end 107.95 58.42) (width 0.8) (layer B.Cu) (net 27))
+  (segment (start 109.22 64.135) (end 109.22 59.69) (width 0.8) (layer B.Cu) (net 27))
+  (segment (start 104.14 54.61) (end 107.95 58.42) (width 0.8) (layer B.Cu) (net 27))
+  (segment (start 104.14 53.34) (end 104.14 54.61) (width 0.8) (layer B.Cu) (net 27))
+  (segment (start 111.76 59.61) (end 112.95 58.42) (width 0.8) (layer B.Cu) (net 28))
+  (segment (start 111.76 64.135) (end 111.76 59.61) (width 0.8) (layer B.Cu) (net 28))
+  (segment (start 81.28 45.72) (end 81.28 48.26) (width 0.8) (layer B.Cu) (net 28))
+  (segment (start 81.28 48.26) (end 111.76 48.26) (width 0.8) (layer B.Cu) (net 28))
+  (segment (start 112.95 49.45) (end 111.76 48.26) (width 0.8) (layer B.Cu) (net 28))
+  (segment (start 112.95 58.42) (end 112.95 49.45) (width 0.8) (layer B.Cu) (net 28))
 )

Commit message: Add proto zone
Routing:
- net (no net): track 0.00 -> 203.2 mm, vias 0 -> 121
- net VCC: track 12.9 -> 89.1 mm, vias 0 -> 20
- net GND: track 49.9 -> 100.7 mm, vias 0 -> 20
- net Net-(U1-Pad9): track 0.00 -> 5.08 mm, vias 0 -> 2
- net Net-(U1-Pad8): track 0.00 -> 5.08 mm, vias 0 -> 2
- net Net-(U1-Pad7): track 0.00 -> 5.08 mm, vias 0 -> 2
- net Net-(U1-Pad6): track 0.00 -> 5.08 mm, vias 0 -> 2
- net Net-(U1-Pad5): track 0.00 -> 5.08 mm, vias 0 -> 2
- net Net-(U1-Pad4): track 0.00 -> 5.08 mm, vias 0 -> 2
- net Net-(U1-Pad3): track 0.00 -> 5.08 mm, vias 0 -> 2
- net Net-(U1-Pad2): track 0.00 -> 5.08 mm, vias 0 -> 2
- net Net-(J2-Pad8): track 0.00 -> 3.18 mm, vias 0 -> 1
- net Net-(J2-Pad7): track 0.00 -> 3.18 mm, vias 0 -> 1
- net Net-(J2-Pad6): track 0.00 -> 3.18 mm, vias 0 -> 1
- net Net-(J2-Pad5): track 0.00 -> 3.18 mm, vias 0 -> 1
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Other:
- rule solder_mask_min_width: 0.25 -> 0.1
- board text added: "0"
- board text added: "7"
- board text added: "74HC573"
- board text added: "A"
- board text added: "B"
- board text added: "Gnd"
- board text added: "Latch"
- board text added: "OE"
- board text added: "Out"
- board text added: "Vcc"

Commit message: Update command pcb template
Parts:
- added R1: 10k, Resistor_SMD:R_0805_2012Metric_Pad1.20x1.40mm_HandSolder, B.Cu at (110.5, 40.6)
- added R2: R, Resistor_SMD:R_0805_2012Metric_Pad1.20x1.40mm_HandSolder, B.Cu at (27.9, 53.3)
- added U2: 74AHC1G08, CommonLibrary:tssop5, B.Cu at (113.7, 43.5)
- J4: value Conn_01x04_Male -> Conn_01x05_Male; footprint Connector_PinHeader_2.54mm:PinHeader_1x04_P2.54mm_Horizontal -> Connector_PinHeader_2.54mm:PinHeader_1x05_P2.54mm_Horizontal
- moved J4 2.54 mm to (116.8, 64.1)
Connections:
- J4 pad 2: GND -> Net-(J4-Pad2)
- J4 pad 3: VCC -> GND
- J4 pad 4: Net-(J4-Pad4) -> VCC
- U1 pad 1: Net-(J4-Pad1) -> Net-(U1-Pad1)
- U1 pad 11: Net-(J4-Pad4) -> Net-(J4-Pad5)
Routing:
- net Net-(J4-Pad5): track 0.00 -> 40.5 mm
- net Net-(J4-Pad4): track 40.5 -> 0.00 mm
- net VCC: track 89.1 -> 113.1 mm, vias 20 -> 25
- net Net-(J4-Pad2): track 0.00 -> 21.5 mm, vias 0 -> 1
- net (no net): track 203.2 -> 221.0 mm, vias 121 -> 131
- net GND: track 100.7 -> 110.8 mm, vias 20 -> 23
- net Net-(U1-Pad1): track 0.00 -> 5.84 mm
- net Net-(R2-Pad1): track 0.00 -> 4.08 mm, vias 0 -> 2
- net Net-(J4-Pad1): track 29.6 -> 31.2 mm, vias 0 -> 1
Other:
- board size 88.9 x 30.5 mm -> 96.5 x 29.2 mm
- board text added: "OE(C)"
