File: template-b/template-b.sch (KiCad schematic (older format))
At the start: 12 parts, among them J1 Conn_01x08_Male, J2 Conn_01x08_Male, J3 Conn_01x08_Male, J4 Conn_01x05_Male, U1 74LS573, U2 74AHC1G08, U3 74AHC1G08, U4 74AHC1G08, U5 74AHC1G08

Commit message: Polishing mask
Parts:
- added R3: R, Resistor_SMD:R_0805_2012Metric_Pad1.20x1.40mm_HandSolder, symbol Device:R
Connections:
- net GND: now also R3.2
Changed lines of the file:
@@
 	1    0    0    1
 $EndComp
+$Comp
+L Device:R R3
+U 1 1 62101683
+P 2500 5150
+F 0 "R3" H 2570 5196 50  0000 L CNN
+F 1 "R" H 2570 5105 50  0000 L CNN
+F 2 "Resistor_SMD:R_0805_2012Metric_Pad1.20x1.40mm_HandSolder" V 2430 5150 50  0001 C CNN
+F 3 "~" H 2500 5150 50  0001 C CNN
+	1    2500 5150
+	1    0    0    -1
+$EndComp
+$Comp
+L power:GND #PWR0109
+U 1 1 62101689
+P 2500 5300
+F 0 "#PWR0109" H 2500 5050 50  0001 C CNN
+F 1 "GND" H 2505 5127 50  0000 C CNN
+F 2 "" H 2500 5300 50  0001 C CNN
+F 3 "" H 2500 5300 50  0001 C CNN
+	1    2500 5300
+	1    0    0    -1
+$EndComp
 $EndSCHEMATC
