File: template-b/template-b.kicad_pcb (KiCad board)
At the start: 2 copper layers, 96.5 x 48.6 mm, 12 parts, among them J1 Conn_01x08_Male, J2 Conn_01x08_Male, J3 Conn_01x08_Male, J4 Conn_01x05_Male, U1 74LS573, U2 74AHC1G08, U3 74AHC1G08, U4 74AHC1G08, U5 74AHC1G08

Commit message: Polishing mask
Parts:
- added R3: R, Resistor_SMD:R_0805_2012Metric_Pad1.20x1.40mm_HandSolder, B.Cu at (27.9, 33.0)
Routing:
- net (no net): track 444.5 -> 439.4 mm, vias 263 -> 259
- net Net-(R3-Pad1): track 0.00 -> 4.08 mm, vias 0 -> 2
- net GND: track 217.0 -> 218.5 mm

Commit message: Update cmd template pcb
Routing:
- net Net-(J4-Pad5): vias 0 -> 1
Changed lines of the file:
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@@
   (general
     (thickness 1.6)
-    (drawings 529)
-    (tracks 828)
+    (drawings 538)
+    (tracks 830)
     (zones 0)
     (modules 13)
@@
   )
   (setup
-    (last_trace_width 0.5)
+    (last_trace_width 0.25)
     (user_trace_width 0.4)
     (user_trace_width 0.5)
@@
       (effects (font (size 1 1) (thickness 0.15)) (justify mirror))
     )
-    (fp_text user %R (at 0 0 90) (layer B.Fab)
-      (effects (font (size 0.5 0.5) (thickness 0.08)) (justify mirror))
-    )
     (fp_line (start -1 -0.625) (end -1 0.625) (layer B.Fab) (width 0.1))
     (fp_line (start -1 0.625) (end 1 0.625) (layer B.Fab) (width 0.1))
@@
     (fp_line (start 1.85 0.95) (end 1.85 -0.95) (layer B.CrtYd) (width 0.05))
     (fp_line (start 1.85 -0.95) (end -1.85 -0.95) (layer B.CrtYd) (width 0.05))
+    (fp_text user %R (at 0 0 90) (layer B.Fab)
+      (effects (font (size 0.5 0.5) (thickness 0.08)) (justify mirror))
+    )
     (pad 2 smd roundrect (at 1 0 90) (size 1.2 1.4) (layers B.Cu B.Paste B.Mask) (roundrect_rratio 0.208333)
       (net 27 GND))
@@
       (net 38 "Net-(J4-Pad2)"))
   )
+  (gr_text Gnd (at 23.8125 31.75 90) (layer F.SilkS)
+    (effects (font (size 1 1) (thickness 0.15)))
+  )
+  (gr_text Gnd (at 23.8125 52.07 90) (layer F.SilkS)
+    (effects (font (size 1 1) (thickness 0.15)))
+  )
+  (gr_text Vcc (at 23.8125 27.305 90) (layer F.SilkS)
+    (effects (font (size 1 1) (thickness 0.15)))
+  )
+  (gr_text Vcc (at 23.8125 47.625 90) (layer F.SilkS)
+    (effects (font (size 1 1) (thickness 0.15)))
+  )
+  (gr_text "OE(C)" (at 117.475 48.895 90) (layer F.SilkS)
+    (effects (font (size 1 1) (thickness 0.15)))
+  )
+  (gr_text OE (at 114.935 49.53 90) (layer F.SilkS)
+    (effects (font (size 1 1) (thickness 0.15)))
+  )
+  (gr_text Latch (at 84.455 58.42) (layer F.SilkS)
+    (effects (font (size 1 1) (thickness 0.15)))
+  )
+  (gr_poly (pts (xy 81.915 57.785) (xy 82.2325 58.42) (xy 81.915 59.055) (xy 81.28 59.3725) (xy 80.645 59.055) (xy 80.3275 58.42) (xy 80.645 57.785) (xy 81.28 57.4675)) (layer F.Mask) (width 0.1))
+  (gr_poly (pts (xy 81.915 57.785) (xy 82.2325 58.42) (xy 81.915 59.055) (xy 81.28 59.3725) (xy 80.645 59.055) (xy 80.3275 58.42) (xy 80.645 57.785) (xy 81.28 57.4675)) (layer B.Mask) (width 0.1))
   (gr_line (start 76.2 53.34) (end 76.2 58.42) (layer F.SilkS) (width 0.12))
   (gr_line (start 78.74 53.34) (end 78.74 58.42) (layer F.SilkS) (width 0.12))
@@
   (segment (start 30.48 20.32) (end 30.48 22.86) (width 1.2) (layer B.Cu) (net 0))
   (segment (start 30.48 22.86) (end 30.48 25.4) (width 1.2) (layer B.Cu) (net 0))
-  (via (at 27.94 35.56) (size 1.6) (drill 0.9) (layers F.Cu B.Cu) (net 49))
-  (via (at 25.4 35.56) (size 1.6) (drill 0.9) (layers F.Cu B.Cu) (net 49))
   (via (at 25.4 38.1) (size 1.6) (drill 0.9) (layers F.Cu B.Cu) (net 0))
   (via (at 27.94 38.1) (size 1.6) (drill 0.9) (layers F.Cu B.Cu) (net 0))
@@
   (segment (start 25.4 22.86) (end 27.94 22.86) (width 1.2) (layer B.Cu) (net 0))
   (segment (start 25.4 25.4) (end 27.94 25.4) (width 1.2) (layer B.Cu) (net 0))
-  (segment (start 25.4 35.56) (end 27.94 35.56) (width 1.2) (layer B.Cu) (net 49))
   (segment (start 25.4 38.1) (end 27.94 38.1) (width 1.2) (layer B.Cu) (net 0))
   (segment (start 23.495 31.115) (end 23.495 31.75) (width 0.25) (layer B.Cu) (net 0))
@@
   (segment (start 83.82 40.64) (end 83.82 40.64) (width 1.2) (layer B.Cu) (net 35))
   (via (at 83.82 40.64) (size 1.6) (drill 0.9) (layers F.Cu B.Cu) (net 35))
-  (segment (start 81.28 53.34) (end 81.28 66.04) (width 0.6) (layer B.Cu) (net 36))
+  (segment (start 81.28 53.34) (end 81.28 58.42) (width 0.6) (layer B.Cu) (net 36))
   (segment (start 81.28 66.04) (end 81.915 66.675) (width 0.6) (layer B.Cu) (net 36))
   (segment (start 81.915 66.675) (end 106.045 66.675) (width 0.6) (layer B.Cu) (net 36))
   (segment (start 106.045 66.675) (end 106.68 66.04) (width 0.6) (layer B.Cu) (net 36))
   (segment (start 106.68 66.04) (end 106.68 64.135) (width 0.6) (layer B.Cu) (net 36))
+  (segment (start 81.28 58.42) (end 81.28 66.04) (width 0.6) (layer B.Cu) (net 36))
+  (via (at 81.28 58.42) (size 1.6) (drill 0.9) (layers F.Cu B.Cu) (net 36))
   (segment (start 104.2925 45.8725) (end 104.14 45.72) (width 0.5) (layer B.Cu) (net 37))
   (segment (start 109.915 45.8725) (end 104.2925 45.8725) (width 0.5) (layer B.Cu) (net 37))
@@
   (segment (start 96.2625 28) (end 96.2025 27.94) (width 0.4) (layer B.Cu) (net 48))
   (segment (start 98.2725 28) (end 96.2625 28) (width 0.4) (layer B.Cu) (net 48))
+  (via (at 27.94 35.56) (size 1.6) (drill 0.9) (layers F.Cu B.Cu) (net 49))
+  (via (at 25.4 35.56) (size 1.6) (drill 0.9) (layers F.Cu B.Cu) (net 49))
+  (segment (start 25.4 35.56) (end 27.94 35.56) (width 1.2) (layer B.Cu) (net 49))
   (segment (start 27.94 34.02) (end 27.94 35.56) (width 0.5) (layer B.Cu) (net 49))
 )
