File: Regs-v2/Regs-v2.sch (KiCad schematic (older format))
At the start: 44 parts, among them J1 Conn_01x08_Male, U1 REG, U10 REG, U11 REG, U12 REG, U13 REG, U14 REG, U15 REG, U16 REG, U17 REG, U18 REG, U19 REG, U2 REG, U20 REG, U21 REG, U22 REG, U23 REG, U24 REG, U25 REG, U26 REG, U27 REG, U28 REG, U29 REG, U3 REG, U30 REG, U31 REG, U32 REG, U33 REG, U34 REG, U4 REG, U5 REG, U6 REG, U7 REG, U8 REG, U9 REG

Commit message: Regs v2 in work
Parts:
- removed U17, U18, U19, U20, U21, U22, U23, U24, U25, U26, U27, U28, U29, U30, U31, U32, U33, U34, U8, U9: REG, CommonLibrary:REG, symbol CommonLibrary:REG
- added D10, D11, D12, D13, D14, D15, D16, D17, D18, D19, D20, D21, D22, D23, D24, D25, D26, D27, D28, D29, D30, D31, D32, D33, D34, D35, D36, D37, D38, D39, D40, D41, D42, D43, D44, D45, D46, D47, D48, D49, D50, D51, D52, D53, D54, D55, D56, D57, D58, D59, D60, D61, D62, D63, D64, D9: LED, LED_THT:LED_Rectangular_W5.0mm_H2.0mm, symbol Device:LED
- added J2, J3, J4, J5, J6, J7, J8: Conn_01x08_Male, Connector_PinHeader_2.54mm:PinHeader_1x08_P2.54mm_Vertical, symbol Connector:Conn_01x08_Male
- added RN2, RN3, RN4, RN5, RN6, RN7, RN8: R_Network08, Resistor_THT:R_Array_SIP9, symbol Device:R_Network08
- renumbered U12 to U10, U13 to U11, U14 to U12, U15 to U13, U16 to U14, U10 to U8, U11 to U9
Connections:
- net DL0: now reaches U1.1 (D0)
- net DL0: now also U2.1 (D0), U3.1 (D0), U4.1 (D0), U5.1 (D0), U6.1 (D0), U7.1 (D0)
- net VCC: now reaches U1.10 (Vcc)
- net VCC: now also U10.10 (Vcc), U11.10 (Vcc), U12.10 (Vcc), U13.10 (Vcc), U14.10 (Vcc), U2.10 (Vcc), U3.10 (Vcc), U4.10 (Vcc), U5.10 (Vcc), U6.10 (Vcc), U7.10 (Vcc), U8.10 (Vcc), U9.10 (Vcc)
- net DL1: now reaches U1.2 (D1)
- net DL1: now also U2.2 (D1), U3.2 (D1), U4.2 (D1), U5.2 (D1), U6.2 (D1), U7.2 (D1)
- net DL2: now reaches U1.3 (D2)
- net DL2: now also U2.3 (D2), U3.3 (D2), U4.3 (D2), U5.3 (D2), U6.3 (D2), U7.3 (D2)
- net DL3: now reaches U1.4 (D3)
- net DL3: now also U2.4 (D3), U3.4 (D3), U4.4 (D3), U5.4 (D3), U6.4 (D3), U7.4 (D3)
- net DL4: now reaches U1.5 (D4)
- net DL4: now also U2.5 (D4), U3.5 (D4), U4.5 (D4), U5.5 (D4), U6.5 (D4), U7.5 (D4)
- net DL5: now reaches U1.6 (D5)
- net DL5: now also U2.6 (D5), U3.6 (D5), U4.6 (D5), U5.6 (D5), U6.6 (D5), U7.6 (D5)
- net DL6: now reaches U1.7 (D6)
- net DL6: now also U2.7 (D6), U3.7 (D6), U4.7 (D6), U5.7 (D6), U6.7 (D6), U7.7 (D6)
- net DL7: now reaches U1.8 (D7)
- net DL7: now also U2.8 (D7), U3.8 (D7), U4.8 (D7), U5.8 (D7), U6.8 (D7), U7.8 (D7)
- net GND: now reaches U1.9 (Gnd)
- net GND: now also RN1.1 (common), U10.9 (Gnd), U11.9 (Gnd), U12.9 (Gnd), U13.9 (Gnd), U14.9 (Gnd), U2.9 (Gnd), U3.9 (Gnd), U4.9 (Gnd), U5.9 (Gnd), U6.9 (Gnd), U7.9 (Gnd), U8.9 (Gnd), U9.9 (Gnd), RN2.1 (common), RN3.1 (common), RN4.1 (common), RN5.1 (common), RN6.1 (common), RN7.1 (common), RN8.1 (common)
- net at RN1.3 (R2): now also D2.1 (K)
- net at RN1.4 (R3): now also D3.1 (K)
- net at RN1.5 (R4): now also D4.1 (K)
- net at RN1.6 (R5): now also D5.1 (K)
- net at RN1.7 (R6): now also D6.1 (K)
- net at RN1.8 (R7): now also D7.1 (K)
- net at RN1.9 (R8): now also D8.1 (K)
- net DH0: now reaches U8.1 (D0)
- net DH0: now also U10.1 (D0), U11.1 (D0), U12.1 (D0), U13.1 (D0), U14.1 (D0), U9.1 (D0)
- net R1.7: now reaches U8.11 (Q7)
- net R1.7: now also D40.2 (A), J5.8 (Pin_8)
- net R1.6: now reaches U8.12 (Q6)
- net R1.6: now also D39.2 (A), J5.7 (Pin_7)
- net R1.5: now reaches U8.13 (Q5)
- net R1.5: now also D38.2 (A), J5.6 (Pin_6)
- net R1.4: now reaches U8.14 (Q4)
- net R1.4: now also D37.2 (A), J5.5 (Pin_5)
- net R1.3: now reaches U8.15 (Q3)
- net R1.3: now also D36.2 (A), J5.4 (Pin_4)
- net R1.2: now reaches U8.16 (Q2)
- net R1.2: now also D35.2 (A), J5.3 (Pin_3)
- net R1.1: now reaches U8.17 (Q1)
- net R1.1: now also D34.2 (A), J5.2 (Pin_2)
- net R1.0: now reaches U8.18 (Q0)
- net R1.0: now also D33.2 (A), J5.1 (Pin_1)
- net DH1: now reaches U8.2 (D1)
- net DH1: now also U10.2 (D1), U11.2 (D1), U12.2 (D1), U13.2 (D1), U14.2 (D1), U9.2 (D1)
- net DH2: now reaches U8.3 (D2)
- net DH2: now also U10.3 (D2), U11.3 (D2), U12.3 (D2), U13.3 (D2), U14.3 (D2), U9.3 (D2)
- net DH3: now reaches U8.4 (D3)
- net DH3: now also U10.4 (D3), U11.4 (D3), U12.4 (D3), U13.4 (D3), U14.4 (D3), U9.4 (D3)
- net DH4: now reaches U8.5 (D4)
- net DH4: now also U10.5 (D4), U11.5 (D4), U12.5 (D4), U13.5 (D4), U14.5 (D4), U9.5 (D4)
- net DH5: now reaches U8.6 (D5)
- net DH5: now also U10.6 (D5), U11.6 (D5), U12.6 (D5), U13.6 (D5), U14.6 (D5), U9.6 (D5)
- net DH6: now reaches U8.7 (D6)
- net DH6: now also U10.7 (D6), U11.7 (D6), U12.7 (D6), U13.7 (D6), U14.7 (D6), U9.7 (D6)
- net DH7: now reaches U8.8 (D7)
- net DH7: now also U10.8 (D7), U11.8 (D7), U12.8 (D7), U13.8 (D7), U14.8 (D7), U9.8 (D7)
- net R2.7: now reaches U2.11 (Q7)
- net R2.7: now also U3.11 (Q7), D16.2 (A), J2.8 (Pin_8)
- net R2.6: now reaches U2.12 (Q6)
- net R2.6: now also U3.12 (Q6), D15.2 (A), J2.7 (Pin_7)
- net R2.5: now reaches U2.13 (Q5)
- net R2.5: now also U3.13 (Q5), D14.2 (A), J2.6 (Pin_6)
- net R2.4: now reaches U2.14 (Q4)
- net R2.4: now also U3.14 (Q4), D13.2 (A), J2.5 (Pin_5)
- net R2.3: now reaches U2.15 (Q3)
- net R2.3: now also U3.15 (Q3), D12.2 (A), J2.4 (Pin_4)
- net R2.2: now reaches U2.16 (Q2)
- net R2.2: now also U3.16 (Q2), D11.2 (A), J2.3 (Pin_3)
- net R2.1: now reaches U2.17 (Q1)
- net R2.1: now also U3.17 (Q1), D10.2 (A), J2.2 (Pin_2)
- net R2.0: now reaches U2.18 (Q0)
- net R2.0: now also U3.18 (Q0), D9.2 (A), J2.1 (Pin_1)
- net R3.7: now reaches U9.11 (Q7)
- net R3.7: now also U10.11 (Q7), D48.2 (A), J6.8 (Pin_8)
- net R3.6: now reaches U9.12 (Q6)
- net R3.6: now also U10.12 (Q6), D47.2 (A), J6.7 (Pin_7)
- net R3.5: now reaches U9.13 (Q5)
- net R3.5: now also U10.13 (Q5), D46.2 (A), J6.6 (Pin_6)
- net R3.4: now reaches U9.14 (Q4)
- net R3.4: now also U10.14 (Q4), D45.2 (A), J6.5 (Pin_5)
- net R3.3: now reaches U9.15 (Q3)
- net R3.3: now also U10.15 (Q3), D44.2 (A), J6.4 (Pin_4)
- net R3.2: now reaches U9.16 (Q2)
- net R3.2: now also U10.16 (Q2), D43.2 (A), J6.3 (Pin_3)
- net R3.1: now reaches U9.17 (Q1)
- net R3.1: now also U10.17 (Q1), D42.2 (A), J6.2 (Pin_2)
- net R3.0: now reaches U9.18 (Q0)
- net R3.0: now also U10.18 (Q0), D41.2 (A), J6.1 (Pin_1)
- net R4.7: now reaches U4.11 (Q7)
- net R4.7: now also U5.11 (Q7), D24.2 (A), J3.8 (Pin_8)
- net R4.6: now reaches U4.12 (Q6)
- net R4.6: now also U5.12 (Q6), D23.2 (A), J3.7 (Pin_7)
- net R4.5: now reaches U4.13 (Q5)
- net R4.5: now also U5.13 (Q5), D22.2 (A), J3.6 (Pin_6)
- net R4.4: now reaches U4.14 (Q4)
- net R4.4: now also U5.14 (Q4), D21.2 (A), J3.5 (Pin_5)
- net R4.3: now reaches U4.15 (Q3)
- net R4.3: now also U5.15 (Q3), D20.2 (A), J3.4 (Pin_4)
- net R4.2: now reaches U4.16 (Q2)
- net R4.2: now also U5.16 (Q2), D19.2 (A), J3.3 (Pin_3)
- net R4.1: now reaches U4.17 (Q1)
- net R4.1: now also U5.17 (Q1), D18.2 (A), J3.2 (Pin_2)
- net R4.0: now reaches U4.18 (Q0)
- net R4.0: now also U5.18 (Q0), D17.2 (A), J3.1 (Pin_1)
- net R5.7: now reaches U11.11 (Q7)
- net R5.7: now also U12.11 (Q7), D56.2 (A), J7.8 (Pin_8)
- net R5.6: now reaches U11.12 (Q6)
- net R5.6: now also U12.12 (Q6), D55.2 (A), J7.7 (Pin_7)
- net R5.5: now reaches U11.13 (Q5)
- net R5.5: now also U12.13 (Q5), D54.2 (A), J7.6 (Pin_6)
- net R5.4: now reaches U11.14 (Q4)
- net R5.4: now also U12.14 (Q4), D53.2 (A), J7.5 (Pin_5)
- net R5.3: now reaches U11.15 (Q3)
- net R5.3: now also U12.15 (Q3), D52.2 (A), J7.4 (Pin_4)
- net R5.2: now reaches U11.16 (Q2)
- net R5.2: now also U12.16 (Q2), D51.2 (A), J7.3 (Pin_3)
- net R5.1: now reaches U11.17 (Q1)
- net R5.1: now also U12.17 (Q1), D50.2 (A), J7.2 (Pin_2)
- net R5.0: now reaches U11.18 (Q0)
- net R5.0: now also U12.18 (Q0), D49.2 (A), J7.1 (Pin_1)
- net R6.7: now reaches U6.11 (Q7)
- net R6.7: now also U7.11 (Q7), D32.2 (A), J4.8 (Pin_8)
- net R6.6: now reaches U6.12 (Q6)
- net R6.6: now also U7.12 (Q6), D31.2 (A), J4.7 (Pin_7)
- net R6.5: now reaches U6.13 (Q5)
- net R6.5: now also U7.13 (Q5), D30.2 (A), J4.6 (Pin_6)
- net R6.4: now reaches U6.14 (Q4)
- net R6.4: now also U7.14 (Q4), D29.2 (A), J4.5 (Pin_5)
- net R6.3: now reaches U6.15 (Q3)
- net R6.3: now also U7.15 (Q3), D28.2 (A), J4.4 (Pin_4)
- net R6.2: now reaches U6.16 (Q2)
- net R6.2: now also U7.16 (Q2), D27.2 (A), J4.3 (Pin_3)
- net R6.1: now reaches U6.17 (Q1)
- net R6.1: now also U7.17 (Q1), D26.2 (A), J4.2 (Pin_2)
- net R6.0: now reaches U6.18 (Q0)
- net R6.0: now also U7.18 (Q0), D25.2 (A), J4.1 (Pin_1)
- net R7.7: now reaches U13.11 (Q7)
- net R7.7: now also U14.11 (Q7), D64.2 (A), J8.8 (Pin_8)
- net R7.6: now reaches U13.12 (Q6)
- net R7.6: now also U14.12 (Q6), D63.2 (A), J8.7 (Pin_7)
- net R7.5: now reaches U13.13 (Q5)
- net R7.5: now also U14.13 (Q5), D62.2 (A), J8.6 (Pin_6)
- net R7.4: now reaches U13.14 (Q4)
- net R7.4: now also U14.14 (Q4), D61.2 (A), J8.5 (Pin_5)
- net R7.3: now reaches U13.15 (Q3)
- net R7.3: now also U14.15 (Q3), D60.2 (A), J8.4 (Pin_4)
- net R7.2: now reaches U13.16 (Q2)
- net R7.2: now also U14.16 (Q2), D59.2 (A), J8.3 (Pin_3)
- net R7.1: now reaches U13.17 (Q1)
- net R7.1: now also U14.17 (Q1), D58.2 (A), J8.2 (Pin_2)
- net R7.0: now reaches U13.18 (Q0)
- net R7.0: now also U14.18 (Q0), D57.2 (A), J8.1 (Pin_1)
- new net: D9.1 (K), RN2.2 (R1)
- new net: D10.1 (K), RN2.3 (R2)
- new net: D11.1 (K), RN2.4 (R3)
- new net: D12.1 (K), RN2.5 (R4)
- new net: D13.1 (K), RN2.6 (R5)
- new net: D14.1 (K), RN2.7 (R6)
- new net: D15.1 (K), RN2.8 (R7)
- new net: D16.1 (K), RN2.9 (R8)
- new net: D17.1 (K), RN3.2 (R1)
- new net: D18.1 (K), RN3.3 (R2)
- new net: D19.1 (K), RN3.4 (R3)
- new net: D20.1 (K), RN3.5 (R4)
- new net: D21.1 (K), RN3.6 (R5)
- new net: D22.1 (K), RN3.7 (R6)
- new net: D23.1 (K), RN3.8 (R7)
- new net: D24.1 (K), RN3.9 (R8)
- new net: D25.1 (K), RN4.2 (R1)
- new net: D26.1 (K), RN4.3 (R2)
- new net: D27.1 (K), RN4.4 (R3)
- new net: D28.1 (K), RN4.5 (R4)
- new net: D29.1 (K), RN4.6 (R5)
- new net: D30.1 (K), RN4.7 (R6)
- new net: D31.1 (K), RN4.8 (R7)
- new net: D32.1 (K), RN4.9 (R8)
- new net: D33.1 (K), RN5.2 (R1)
- new net: D34.1 (K), RN5.3 (R2)
- new net: D35.1 (K), RN5.4 (R3)
- new net: D36.1 (K), RN5.5 (R4)
- new net: D37.1 (K), RN5.6 (R5)
- new net: D38.1 (K), RN5.7 (R6)
- new net: D39.1 (K), RN5.8 (R7)
- new net: D40.1 (K), RN5.9 (R8)
- new net: D41.1 (K), RN6.2 (R1)
- new net: D42.1 (K), RN6.3 (R2)
- new net: D43.1 (K), RN6.4 (R3)
- new net: D44.1 (K), RN6.5 (R4)
- new net: D45.1 (K), RN6.6 (R5)
- new net: D46.1 (K), RN6.7 (R6)
- new net: D47.1 (K), RN6.8 (R7)
- new net: D48.1 (K), RN6.9 (R8)
- new net: D49.1 (K), RN7.2 (R1)
- new net: D50.1 (K), RN7.3 (R2)
- new net: D51.1 (K), RN7.4 (R3)
- new net: D52.1 (K), RN7.5 (R4)
- new net: D53.1 (K), RN7.6 (R5)
- new net: D54.1 (K), RN7.7 (R6)
- new net: D55.1 (K), RN7.8 (R7)
- new net: D56.1 (K), RN7.9 (R8)
- new net: D57.1 (K), RN8.2 (R1)
- new net: D58.1 (K), RN8.3 (R2)
- new net: D59.1 (K), RN8.4 (R3)
- new net: D60.1 (K), RN8.5 (R4)
- new net: D61.1 (K), RN8.6 (R5)
- new net: D62.1 (K), RN8.7 (R6)
- new net: D63.1 (K), RN8.8 (R7)
- new net: D64.1 (K), RN8.9 (R8)
Other:
- note added: "Bank0"
- note added: "Bank1"
- note added: "R0"
- note added: "R1"
- note added: "R2"
- note added: "R3"
- note added: "R4"
- note added: "R5"
- note added: "R6"
- note added: "R7"
- moved on the sheet: D1, D2, D3, D4, D5, D6, D7, D8, J1, RN1, U10, U11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

Commit message: Regs v2 in work
Parts:
- added C1: 1uF, Capacitor_THT:C_Disc_D5.0mm_W2.5mm_P5.00mm, symbol Device:C
- added D65, D66: LED, LED_THT:LED_Rectangular_W5.0mm_H2.0mm, symbol Device:LED
- added H1, H2, H3, H4, H5, H6: MountingHole, MountingHole:MountingHole_3.2mm_M3, symbol Mechanical:MountingHole
- added J10, J13: Conn_01x08_Male, Connector_PinHeader_2.54mm:PinHeader_1x08_P2.54mm_Vertical, symbol Connector:Conn_01x08_Male
- added J11, J12: Conn_01x01_Male, Connector_PinHeader_2.54mm:PinHeader_1x01_P2.54mm_Vertical, symbol Connector:Conn_01x01_Male
- added J14: Conn_01x02_Male, Connector_PinHeader_2.54mm:PinHeader_1x02_P2.54mm_Vertical, symbol Connector:Conn_01x02_Male
- added J9: Conn_01x03_Male, Connector_PinHeader_2.54mm:PinHeader_1x03_P2.54mm_Vertical, symbol Connector:Conn_01x03_Male
- added R1, R2, R3, R5, R7: 10k, Resistor_THT:R_Axial_DIN0207_L6.3mm_D2.5mm_P7.62mm_Horizontal, symbol Device:R
- added R4, R6: 1k, Resistor_THT:R_Axial_DIN0207_L6.3mm_D2.5mm_P7.62mm_Horizontal, symbol Device:R
- added SW1, SW2: SW_Push, Button_Switch_THT:SW_PUSH_6mm_H5mm, symbol Switch:SW_Push
- added U15, U17: 74HC00, Package_DIP:DIP-14_W7.62mm_Socket, symbol 74xx:74HC00
- added U16: 74HC238, Package_DIP:DIP-16_W7.62mm_Socket, symbol 74xx_IEEE:74HC238
- added U18: 74LS10, Package_DIP:DIP-14_W7.62mm_Socket, symbol 74xx:74LS10
Connections:
- net DH0: now also J13.1 (Pin_1)
- net DH1: now also J13.2 (Pin_2)
- net DH2: now also J13.3 (Pin_3)
- net DH3: now also J13.4 (Pin_4)
- net DH4: now also J13.5 (Pin_5)
- net DH5: now also J13.6 (Pin_6)
- net DH6: now also J13.7 (Pin_7)
- net DH7: now also J13.8 (Pin_8)
- net DL0: now also J10.1 (Pin_1)
- net DL1: now also J10.2 (Pin_2)
- net DL2: now also J10.3 (Pin_3)
- net DL3: now also J10.4 (Pin_4)
- net DL4: now also J10.5 (Pin_5)
- net DL5: now also J10.6 (Pin_6)
- net DL6: now also J10.7 (Pin_7)
- net DL7: now also J10.8 (Pin_8)
- net GND: now also C1.2, SW1.1, SW2.1, U15.7 (GND), U16.3 (A2), U16.4 (~G2A), U16.5 (~G2B), U16.8 (GND), U17.7 (GND), U18.7 (GND)
- net VCC: now also R1.2, R2.2, R3.2, R4.1, R5.1, R6.1, R7.1, U15.14 (VCC), U16.16 (VCC), U17.14 (VCC), U18.14 (VCC)
- net at U1.19 (~CS): now also R1.1
- net Col0: now reaches U1.20 (~Col)
- net Col0: now also U8.20 (~Col), U16.15 (Y0)
- net RowL: now reaches U1.21 (~Row)
- net RowL: now also U2.21 (~Row), U3.21 (~Row), U4.21 (~Row), U5.21 (~Row), U6.21 (~Row), U7.21 (~Row), U15.8
- net at U8.19 (~CS): now also R2.1
- net RowH: now reaches U8.21 (~Row)
- net RowH: now also U10.21 (~Row), U11.21 (~Row), U12.21 (~Row), U13.21 (~Row), U14.21 (~Row), U9.21 (~Row), U15.11
- net Bank0: now reaches U2.19 (~CS)
- net Bank0: now also U11.19 (~CS), U13.19 (~CS), U4.19 (~CS), U6.19 (~CS), U9.19 (~CS), U17.6
- net Col1: now reaches U2.20 (~Col)
- net Col1: now also U10.20 (~Col), U3.20 (~Col), U9.20 (~Col), U16.14 (Y1)
- net Bank1: now reaches U3.19 (~CS)
- net Bank1: now also U10.19 (~CS), U12.19 (~CS), U14.19 (~CS), U5.19 (~CS), U7.19 (~CS), U17.3
- net Col2: now reaches U4.20 (~Col)
- net Col2: now also U11.20 (~Col), U12.20 (~Col), U5.20 (~Col), U16.13 (Y2)
- net Col3: now reaches U6.20 (~Col)
- net Col3: now also U13.20 (~Col), U14.20 (~Col), U7.20 (~Col), U16.12 (Y3)
- new net: U15.10, U15.12, U15.3
- new net: U15.6, U15.9
- new net: R3.1, U16.6 (G1)
- new net: D65.1 (K), U17.1, U17.2, U18.12, U18.3
- new net: C1.1, R7.2, SW2.2, U18.4
- new net: U17.8, U18.5
- new net: D66.1 (K), U17.4, U17.5, U18.13, U18.6
- new net: U17.11, U18.1
- new net: R5.2, SW1.2, U18.2
- new net: D65.2 (A), R4.2
- new net: D66.2 (A), R6.2
- new net 8\16: J11.1 (Pin_1), U15.1, U15.2
- new net Bank0-cmd: J14.1 (Pin_1), U17.10
- new net Bank1-cmd: J14.2 (Pin_2), U17.12
- new net C2: J12.1 (Pin_1), U17.13, U17.9
- new net Reg[0]: J9.1 (Pin_1), U15.13, U15.4, U15.5
- new net Reg[1]: J9.2 (Pin_2), U16.1 (A0)
- new net Reg[2]: J9.3 (Pin_3), U16.2 (A1)
- no-connect marks 0 -> 4

Commit message: Regs pcb is ready
Parts:
- removed R2, R3: 10k, Resistor_THT:R_Axial_DIN0207_L6.3mm_D2.5mm_P7.62mm_Horizontal, symbol Device:R
- removed U15: 74HC00, Package_DIP:DIP-14_W7.62mm_Socket, symbol 74xx:74HC00
- removed U16: 74HC238, Package_DIP:DIP-16_W7.62mm_Socket, symbol 74xx_IEEE:74HC238
- removed unit 1 of U17
- removed unit 2 of U17
- removed unit 2 of U18
- added J15: Screw_Terminal_01x02, TerminalBlock_Phoenix:TerminalBlock_Phoenix_MKDS-1,5-2_1x02_P5.00mm_Horizontal, symbol Connector:Screw_Terminal_01x02
- added J16: Conn_01x01_Male, Connector_PinHeader_2.54mm:PinHeader_1x01_P2.54mm_Vertical, symbol Connector:Conn_01x01_Male
- added U15: 74HC02, Package_DIP:DIP-14_W7.62mm_Socket, symbol 74xx:74HC02
- added U16: 74LS139, Package_DIP:DIP-16_W7.62mm_Socket, symbol 74xx:74LS139
- added unit 3 of U18
Connections:
- net Bank0 is gone; now on net ~Bank0: U11.19 (~CS), U13.19 (~CS), U2.19 (~CS), U4.19 (~CS), U6.19 (~CS), U9.19 (~CS)
- net Bank1 is gone; now on net ~Bank1: U10.19 (~CS), U12.19 (~CS), U14.19 (~CS), U3.19 (~CS), U5.19 (~CS), U7.19 (~CS)
- net 8\16: now also R1.1, U15.12, U15.8
- net GND: now also R1.2, U1.19 (~CS), U8.19 (~CS), J15.2 (Pin_2), U15.7 (GND), U16.8 (GND)
- net Reg[0]: now also U15.5, U15.6, U15.9
- net Reg[1]: now also U16.2 (A0)
- net Reg[2]: now also U16.3 (A1)
- net VCC: now also J15.1 (Pin_1), U15.14 (VCC), U16.16 (VCC); no longer R1.2
- net at D1.1 (K): now also RN1.9 (R8); no longer RN1.2 (R1)
- net at RN1.3 (R2): now also D7.1 (K); no longer D2.1 (K)
- net at RN1.4 (R3): now also D6.1 (K); no longer D3.1 (K)
- net at RN1.5 (R4): now also D5.1 (K); no longer D4.1 (K)
- net at RN1.6 (R5): now also D4.1 (K); no longer D5.1 (K)
- net at RN1.7 (R6): now also D3.1 (K); no longer D6.1 (K)
- net at RN1.8 (R7): now also D2.1 (K); no longer D7.1 (K)
- net at D8.1 (K): now also RN1.2 (R1); no longer RN1.9 (R8)
- net at D9.1 (K): now also RN2.9 (R8); no longer RN2.2 (R1)
- net at RN2.3 (R2): now also D15.1 (K); no longer D10.1 (K)
- net at RN2.4 (R3): now also D14.1 (K); no longer D11.1 (K)
- net at RN2.5 (R4): now also D13.1 (K); no longer D12.1 (K)
- net at RN2.6 (R5): now also D12.1 (K); no longer D13.1 (K)
- net at RN2.7 (R6): now also D11.1 (K); no longer D14.1 (K)
- net at RN2.8 (R7): now also D10.1 (K); no longer D15.1 (K)
- net at D16.1 (K): now also RN2.2 (R1); no longer RN2.9 (R8)
- net at D17.1 (K): now also RN3.9 (R8); no longer RN3.2 (R1)
- net at RN3.3 (R2): now also D23.1 (K); no longer D18.1 (K)
- net at RN3.4 (R3): now also D22.1 (K); no longer D19.1 (K)
- net at RN3.5 (R4): now also D21.1 (K); no longer D20.1 (K)
- net at RN3.6 (R5): now also D20.1 (K); no longer D21.1 (K)
- net at RN3.7 (R6): now also D19.1 (K); no longer D22.1 (K)
- net at RN3.8 (R7): now also D18.1 (K); no longer D23.1 (K)
- net at D24.1 (K): now also RN3.2 (R1); no longer RN3.9 (R8)
- net at D25.1 (K): now also RN4.9 (R8); no longer RN4.2 (R1)
- net at RN4.3 (R2): now also D31.1 (K); no longer D26.1 (K)
- net at RN4.4 (R3): now also D30.1 (K); no longer D27.1 (K)
- net at RN4.5 (R4): now also D29.1 (K); no longer D28.1 (K)
- net at RN4.6 (R5): now also D28.1 (K); no longer D29.1 (K)
- net at RN4.7 (R6): now also D27.1 (K); no longer D30.1 (K)
- net at RN4.8 (R7): now also D26.1 (K); no longer D31.1 (K)
- net at D32.1 (K): now also RN4.2 (R1); no longer RN4.9 (R8)
- net at D33.1 (K): now also RN5.9 (R8); no longer RN5.2 (R1)
- net at RN5.3 (R2): now also D39.1 (K); no longer D34.1 (K)
- net at RN5.4 (R3): now also D38.1 (K); no longer D35.1 (K)
- net at RN5.5 (R4): now also D37.1 (K); no longer D36.1 (K)
- net at RN5.6 (R5): now also D36.1 (K); no longer D37.1 (K)
- net at RN5.7 (R6): now also D35.1 (K); no longer D38.1 (K)
- net at RN5.8 (R7): now also D34.1 (K); no longer D39.1 (K)
- net at D40.1 (K): now also RN5.2 (R1); no longer RN5.9 (R8)
- net at D41.1 (K): now also RN6.9 (R8); no longer RN6.2 (R1)
- net at RN6.3 (R2): now also D47.1 (K); no longer D42.1 (K)
- net at RN6.4 (R3): now also D46.1 (K); no longer D43.1 (K)
- net at RN6.5 (R4): now also D45.1 (K); no longer D44.1 (K)
- net at RN6.6 (R5): now also D44.1 (K); no longer D45.1 (K)
- net at RN6.7 (R6): now also D43.1 (K); no longer D46.1 (K)
- net at RN6.8 (R7): now also D42.1 (K); no longer D47.1 (K)
- net at D48.1 (K): now also RN6.2 (R1); no longer RN6.9 (R8)
- net at D49.1 (K): now also RN7.9 (R8); no longer RN7.2 (R1)
- net at RN7.3 (R2): now also D55.1 (K); no longer D50.1 (K)
- net at RN7.4 (R3): now also D54.1 (K); no longer D51.1 (K)
- net at RN7.5 (R4): now also D53.1 (K); no longer D52.1 (K)
- net at RN7.6 (R5): now also D52.1 (K); no longer D53.1 (K)
- net at RN7.7 (R6): now also D51.1 (K); no longer D54.1 (K)
- net at RN7.8 (R7): now also D50.1 (K); no longer D55.1 (K)
- net at D56.1 (K): now also RN7.2 (R1); no longer RN7.9 (R8)
- net at D57.1 (K): now also RN8.9 (R8); no longer RN8.2 (R1)
- net at RN8.3 (R2): now also D63.1 (K); no longer D58.1 (K)
- net at RN8.4 (R3): now also D62.1 (K); no longer D59.1 (K)
- net at RN8.5 (R4): now also D61.1 (K); no longer D60.1 (K)
- net at RN8.6 (R5): now also D60.1 (K); no longer D61.1 (K)
- net at RN8.7 (R6): now also D59.1 (K); no longer D62.1 (K)
- net at RN8.8 (R7): now also D58.1 (K); no longer D63.1 (K)
- net at D64.1 (K): now also RN8.2 (R1); no longer RN8.9 (R8)
- net ~Bank1: now reaches D65.1 (K), U18.12
- net ~Bank1: now also U18.11
- net at C1.1, R7.2, SW2.2: now also U18.10
- net at U17.8: now also U18.9
- net ~Bank0: now reaches D66.1 (K), U18.13
- net ~Bank0: now also U18.8
- net at U17.11: now also U18.2; no longer U18.1
- net at R5.2, SW1.2: now also U18.1; no longer U18.2
- net Col0 renamed ~Col0
- net ~Col0: now also U16.4 (O0)
- net Col1 renamed ~Col1
- net ~Col1: now also U16.5 (O1)
- net Col2 renamed ~Col2
- net ~Col2: now also U16.6 (O2)
- net Col3 renamed ~Col3
- net ~Col3: now also U16.7 (O3)
- net RowH renamed ~RowH
- net ~RowH: now also U15.10
- net RowL renamed ~RowL
- net ~RowL: now also U15.13
- new net: U15.11, U15.4
- new net ~Latch: J16.1 (Pin_1), U16.1 (E)
- no-connect marks 4 -> 0
Other:
- moved on the sheet: H1, H2, H3, H4, H5, H6, R5, U17E, U18D
