File: Regs-v2/Regs-v2.sch (KiCad schematic (older format))
At the start: 122 parts, among them J1 Conn_01x08_Male, J10 Conn_01x08_Male, J11 Conn_01x01_Male, J12 Conn_01x01_Male, J13 Conn_01x08_Male, J14 Conn_01x02_Male, J15 Screw_Terminal_01x02, J16 Conn_01x01_Male, J2 Conn_01x08_Male, J3 Conn_01x08_Male, J4 Conn_01x08_Male, J5 Conn_01x08_Male, J6 Conn_01x08_Male, J7 Conn_01x08_Male, J8 Conn_01x08_Male, J9 Conn_01x03_Male, SW1 SW_Push, SW2 SW_Push, U1 REG, U10 REG, U11 REG, U12 REG, U13 REG, U14 REG, U15 74HC02, U16 74LS139, U17 74HC00, U18 74LS10, U2 REG, U3 REG, U4 REG, U5 REG, U6 REG, U7 REG, U8 REG, U9 REG

Commit message: Polishing Regs pcb
Parts:
- removed H6: MountingHole, MountingHole:MountingHole_3.2mm_M3, symbol Mechanical:MountingHole
- added C2, C3, C4: 1uF, Capacitor_SMD:C_0805_2012Metric_Pad1.18x1.45mm_HandSolder, symbol Device:C
- added unit 1 of U15
Connections:
- net GND: now also C2.2, C3.2, C4.2
- net VCC: now also C2.1, C3.1, C4.1
- net ~Latch: no longer names the net of U16.1 (E)
- net ~Latch: now also U15.1; no longer J16.1 (Pin_1)
- new net Latch: J16.1 (Pin_1), U15.2, U15.3
Other:
- moved on the sheet: H1, H2, H3, H4, H5
Changed lines of the file:
@@
 L Mechanical:MountingHole H1
 U 1 1 63C65500
-P 5750 9000
-F 0 "H1" H 5850 9046 50  0000 L CNN
-F 1 "MountingHole" H 5850 8955 50  0000 L CNN
-F 2 "MountingHole:MountingHole_3.2mm_M3" H 5750 9000 50  0001 C CNN
-F 3 "~" H 5750 9000 50  0001 C CNN
-	1    5750 9000
+P 5500 9000
+F 0 "H1" H 5600 9046 50  0000 L CNN
+F 1 "MountingHole" H 5600 8955 50  0000 L CNN
+F 2 "MountingHole:MountingHole_3.2mm_M3" H 5500 9000 50  0001 C CNN
+F 3 "~" H 5500 9000 50  0001 C CNN
+	1    5500 9000
 	1    0    0    -1
 $EndComp
@@
 L Mechanical:MountingHole H3
 U 1 1 63C65EAE
-P 5750 9250
-F 0 "H3" H 5850 9296 50  0000 L CNN
-F 1 "MountingHole" H 5850 9205 50  0000 L CNN
-F 2 "MountingHole:MountingHole_3.2mm_M3" H 5750 9250 50  0001 C CNN
-F 3 "~" H 5750 9250 50  0001 C CNN
-	1    5750 9250
+P 5500 9250
+F 0 "H3" H 5600 9296 50  0000 L CNN
+F 1 "MountingHole" H 5600 9205 50  0000 L CNN
+F 2 "MountingHole:MountingHole_3.2mm_M3" H 5500 9250 50  0001 C CNN
+F 3 "~" H 5500 9250 50  0001 C CNN
+	1    5500 9250
 	1    0    0    -1
 $EndComp
@@
 L Mechanical:MountingHole H5
 U 1 1 63C66157
-P 5750 9500
-F 0 "H5" H 5850 9546 50  0000 L CNN
-F 1 "MountingHole" H 5850 9455 50  0000 L CNN
-F 2 "MountingHole:MountingHole_3.2mm_M3" H 5750 9500 50  0001 C CNN
-F 3 "~" H 5750 9500 50  0001 C CNN
-	1    5750 9500
+P 5500 9500
+F 0 "H5" H 5600 9546 50  0000 L CNN
+F 1 "MountingHole" H 5600 9455 50  0000 L CNN
+F 2 "MountingHole:MountingHole_3.2mm_M3" H 5500 9500 50  0001 C CNN
+F 3 "~" H 5500 9500 50  0001 C CNN
+	1    5500 9500
 	1    0    0    -1
 $EndComp
@@
 L Mechanical:MountingHole H2
 U 1 1 63C66406
-P 6750 9000
-F 0 "H2" H 6850 9046 50  0000 L CNN
-F 1 "MountingHole" H 6850 8955 50  0000 L CNN
-F 2 "MountingHole:MountingHole_3.2mm_M3" H 6750 9000 50  0001 C CNN
-F 3 "~" H 6750 9000 50  0001 C CNN
-	1    6750 9000
+P 6500 9000
+F 0 "H2" H 6600 9046 50  0000 L CNN
+F 1 "MountingHole" H 6600 8955 50  0000 L CNN
+F 2 "MountingHole:MountingHole_3.2mm_M3" H 6500 9000 50  0001 C CNN
+F 3 "~" H 6500 9000 50  0001 C CNN
+	1    6500 9000
 	1    0    0    -1
 $EndComp
@@
 L Mechanical:MountingHole H4
 U 1 1 63C66876
-P 6750 9250
-F 0 "H4" H 6850 9296 50  0000 L CNN
-F 1 "MountingHole" H 6850 9205 50  0000 L CNN
-F 2 "MountingHole:MountingHole_3.2mm_M3" H 6750 9250 50  0001 C CNN
-F 3 "~" H 6750 9250 50  0001 C CNN
-	1    6750 9250
-	1    0    0    -1
-$EndComp
-$Comp
-L Mechanical:MountingHole H6
-U 1 1 63C66AC4
-P 6750 9500
-F 0 "H6" H 6850 9546 50  0000 L CNN
-F 1 "MountingHole" H 6850 9455 50  0000 L CNN
-F 2 "MountingHole:MountingHole_3.2mm_M3" H 6750 9500 50  0001 C CNN
-F 3 "~" H 6750 9500 50  0001 C CNN
-	1    6750 9500
+P 6500 9250
+F 0 "H4" H 6600 9296 50  0000 L CNN
+F 1 "MountingHole" H 6600 9205 50  0000 L CNN
+F 2 "MountingHole:MountingHole_3.2mm_M3" H 6500 9250 50  0001 C CNN
+F 3 "~" H 6500 9250 50  0001 C CNN
+	1    6500 9250
 	1    0    0    -1
 $EndComp
@@
 L power:PWR_FLAG #FLG02
 U 1 1 648C1C04
-P 8000 9500
-F 0 "#FLG02" H 8000 9575 50  0001 C CNN
-F 1 "PWR_FLAG" H 8000 9673 50  0000 C CNN
-F 2 "" H 8000 9500 50  0001 C CNN
-F 3 "~" H 8000 9500 50  0001 C CNN
-	1    8000 9500
+P 7500 9425
+F 0 "#FLG02" H 7500 9500 50  0001 C CNN
+F 1 "PWR_FLAG" H 7500 9598 50  0000 C CNN
+F 2 "" H 7500 9425 50  0001 C CNN
+F 3 "~" H 7500 9425 50  0001 C CNN
+	1    7500 9425
 	1    0    0    -1
 $EndComp
@@
 L power:PWR_FLAG #FLG01
 U 1 1 648C207F
-P 8000 9000
-F 0 "#FLG01" H 8000 9075 50  0001 C CNN
-F 1 "PWR_FLAG" H 8000 9173 50  0000 C CNN
-F 2 "" H 8000 9000 50  0001 C CNN
-F 3 "~" H 8000 9000 50  0001 C CNN
-	1    8000 9000
+P 7500 8925
+F 0 "#FLG01" H 7500 9000 50  0001 C CNN
+F 1 "PWR_FLAG" H 7500 9098 50  0000 C CNN
+F 2 "" H 7500 8925 50  0001 C CNN
+F 3 "~" H 7500 8925 50  0001 C CNN
+	1    7500 8925
 	-1   0    0    1
 $EndComp
@@
 L power:VCC #PWR056
 U 1 1 64969903
-P 8000 9000
-F 0 "#PWR056" H 8000 8850 50  0001 C CNN
-F 1 "VCC" H 8015 9173 50  0000 C CNN
-F 2 "" H 8000 9000 50  0001 C CNN
-F 3 "" H 8000 9000 50  0001 C CNN
-	1    8000 9000
+P 7500 8925
+F 0 "#PWR056" H 7500 8775 50  0001 C CNN
+F 1 "VCC" H 7515 9098 50  0000 C CNN
+F 2 "" H 7500 8925 50  0001 C CNN
+F 3 "" H 7500 8925 50  0001 C CNN
+	1    7500 8925
 	1    0    0    -1
 $EndComp
@@
 L power:GND #PWR057
 U 1 1 64969CA8
-P 8000 9500
-F 0 "#PWR057" H 8000 9250 50  0001 C CNN
-F 1 "GND" H 8005 9327 50  0000 C CNN
-F 2 "" H 8000 9500 50  0001 C CNN
-F 3 "" H 8000 9500 50  0001 C CNN
-	1    8000 9500
+P 7500 9425
+F 0 "#PWR057" H 7500 9175 50  0001 C CNN
+F 1 "GND" H 7505 9252 50  0000 C CNN
+F 2 "" H 7500 9425 50  0001 C CNN
+F 3 "" H 7500 9425 50  0001 C CNN
+	1    7500 9425
 	1    0    0    -1
 $EndComp
@@
 Connection ~ 11100 8500
 Wire Wire Line
-	5550 7400 5800 7400
-Text Label 5550 7400 0    50   ~ 0
-~Latch
+	4950 7300 5200 7300
+Text Label 4950 7300 0    50   ~ 0
+Latch
 $Comp
 L Connector:Conn_01x01_Male J16
@@
 $EndComp
 Text Label 15500 9000 0    50   ~ 0
-~Latch
+Latch
+$Comp
+L 74xx:74HC02 U15
+U 1 1 629E5478
+P 5500 7400
+F 0 "U15" H 5425 7600 50  0000 C CNN
+F 1 "74HC02" H 5500 7200 50  0000 C CNN
+F 2 "Package_DIP:DIP-14_W7.62mm_Socket" H 5500 7400 50  0001 C CNN
+F 3 "http://www.ti.com/lit/gpn/sn74hc02" H 5500 7400 50  0001 C CNN
+	1    5500 7400
+	1    0    0    -1
+$EndComp
+Wire Wire Line
+	5200 7300 5200 7500
+Connection ~ 5200 7300
+$Comp
+L Device:C C2
+U 1 1 62C23C18
+P 8000 9150
+F 0 "C2" H 8115 9196 50  0000 L CNN
+F 1 "1uF" H 8115 9105 50  0000 L CNN
+F 2 "Capacitor_SMD:C_0805_2012Metric_Pad1.18x1.45mm_HandSolder" H 8038 9000 50  0001 C CNN
+F 3 "~" H 8000 9150 50  0001 C CNN
+	1    8000 9150
+	1    0    0    -1
+$EndComp
+$Comp
+L power:VCC #PWR042
+U 1 1 62C24293
+P 8000 9000
+F 0 "#PWR042" H 8000 8850 50  0001 C CNN
+F 1 "VCC" H 8015 9173 50  0000 C CNN
+F 2 "" H 8000 9000 50  0001 C CNN
+F 3 "" H 8000 9000 50  0001 C CNN
+	1    8000 9000
+	1    0    0    -1
+$EndComp
+$Comp
+L power:GND #PWR043
+U 1 1 62C24654
+P 8000 9300
+F 0 "#PWR043" H 8000 9050 50  0001 C CNN
+F 1 "GND" H 8005 9127 50  0000 C CNN
+F 2 "" H 8000 9300 50  0001 C CNN
+F 3 "" H 8000 9300 50  0001 C CNN
+	1    8000 9300
+	1    0    0    -1
+$EndComp
+$Comp
+L Device:C C3
+U 1 1 62CAD8F1
+P 8000 9975
+F 0 "C3" H 8115 10021 50  0000 L CNN
+F 1 "1uF" H 8115 9930 50  0000 L CNN
+F 2 "Capacitor_SMD:C_0805_2012Metric_Pad1.18x1.45mm_HandSolder" H 8038 9825 50  0001 C CNN
+F 3 "~" H 8000 9975 50  0001 C CNN
+	1    8000 9975
+	1    0    0    -1
+$EndComp
+$Comp
+L power:VCC #PWR058
+U 1 1 62CAD8F7
+P 8000 9825
+F 0 "#PWR058" H 8000 9675 50  0001 C CNN
+F 1 "VCC" H 8015 9998 50  0000 C CNN
+F 2 "" H 8000 9825 50  0001 C CNN
+F 3 "" H 8000 9825 50  0001 C CNN
+	1    8000 9825
+	1    0    0    -1
+$EndComp
+$Comp
+L power:GND #PWR060
+U 1 1 62CAD8FD
+P 8000 10125
+F 0 "#PWR060" H 8000 9875 50  0001 C CNN
+F 1 "GND" H 8005 9952 50  0000 C CNN
+F 2 "" H 8000 10125 50  0001 C CNN
+F 3 "" H 8000 10125 50  0001 C CNN
+	1    8000 10125
+	1    0    0    -1
+$EndComp
+$Comp
+L Device:C C4
+U 1 1 62D043B0
+P 8500 9975
+F 0 "C4" H 8615 10021 50  0000 L CNN
+F 1 "1uF" H 8615 9930 50  0000 L CNN
+F 2 "Capacitor_SMD:C_0805_2012Metric_Pad1.18x1.45mm_HandSolder" H 8538 9825 50  0001 C CNN
+F 3 "~" H 8500 9975 50  0001 C CNN
+	1    8500 9975
+	1    0    0    -1
+$EndComp
+$Comp
+L power:VCC #PWR059
+U 1 1 62D043B6
+P 8500 9825
+F 0 "#PWR059" H 8500 9675 50  0001 C CNN
+F 1 "VCC" H 8515 9998 50  0000 C CNN
+F 2 "" H 8500 9825 50  0001 C CNN
+F 3 "" H 8500 9825 50  0001 C CNN
+	1    8500 9825
+	1    0    0    -1
+$EndComp
+$Comp
+L power:GND #PWR061
+U 1 1 62D043BC
+P 8500 10125
+F 0 "#PWR061" H 8500 9875 50  0001 C CNN
+F 1 "GND" H 8505 9952 50  0000 C CNN
+F 2 "" H 8500 10125 50  0001 C CNN
+F 3 "" H 8500 10125 50  0001 C CNN
+	1    8500 10125
+	1    0    0    -1
+$EndComp
 $EndSCHEMATC

Commit message: Remove bank trigger
Parts:
- removed C1: 1uF, Capacitor_THT:C_Disc_D5.0mm_W2.5mm_P5.00mm, symbol Device:C
- removed D65, D66: LED, LED_THT:LED_Rectangular_W5.0mm_H2.0mm, symbol Device:LED
- removed J12: Conn_01x01_Male, Connector_PinHeader_2.54mm:PinHeader_1x01_P2.54mm_Vertical, symbol Connector:Conn_01x01_Male
- removed R4, R6: 1k, Resistor_THT:R_Axial_DIN0207_L6.3mm_D2.5mm_P7.62mm_Horizontal, symbol Device:R
- removed R5, R7: 10k, Resistor_THT:R_Axial_DIN0207_L6.3mm_D2.5mm_P7.62mm_Horizontal, symbol Device:R
- removed SW1, SW2: SW_Push, Button_Switch_THT:SW_PUSH_6mm_H5mm, symbol Switch:SW_Push
- removed U17: 74HC00, Package_DIP:DIP-14_W7.62mm_Socket, symbol 74xx:74HC00
- removed U18: 74LS10, Package_DIP:DIP-14_W7.62mm_Socket, symbol 74xx:74LS10
- added J12, J17: Conn_01x08_Male, Connector_PinHeader_2.54mm:PinHeader_1x08_P2.54mm_Vertical, symbol Connector:Conn_01x08_Male
- added R2, R3: 10k, Resistor_SMD:R_0805_2012Metric_Pad1.20x1.40mm_HandSolder, symbol Device:R
- R1: footprint Resistor_THT:R_Axial_DIN0207_L6.3mm_D2.5mm_P7.62mm_Horizontal -> Resistor_SMD:R_0805_2012Metric_Pad1.20x1.40mm_HandSolder
Connections:
- net Bank0-cmd is gone; now on net ~Bank0: J14.1 (Pin_1)
- net Bank1-cmd is gone; now on net ~Bank1: J14.2 (Pin_2)
- net DH0: now also J17.1 (Pin_1)
- net DH1: now also J17.2 (Pin_2)
- net DH2: now also J17.3 (Pin_3)
- net DH3: now also J17.4 (Pin_4)
- net DH4: now also J17.5 (Pin_5)
- net DH5: now also J17.6 (Pin_6)
- net DH6: now also J17.7 (Pin_7)
- net DH7: now also J17.8 (Pin_8)
- net DL0: now also J12.1 (Pin_1)
- net DL1: now also J12.2 (Pin_2)
- net DL2: now also J12.3 (Pin_3)
- net DL3: now also J12.4 (Pin_4)
- net DL4: now also J12.5 (Pin_5)
- net DL5: now also J12.6 (Pin_6)
- net DL6: now also J12.7 (Pin_7)
- net DL7: now also J12.8 (Pin_8)
- net GND: now also R3.2
- net VCC: now also R2.1
- net ~Bank0: now also R3.1
- net ~Bank1: now also R2.2
Other:
- moved on the sheet: U15E
