File: MUX8x1-v2/MUX.kicad_pcb (KiCad board)
At the start: 2 copper layers, 152.4 x 152.4 mm, 42 parts, among them J1 Conn_01x08_Male, J10 Conn_01x03_Male, J11 Conn_01x08_Male, J12 Conn_01x08_Male, J13 Conn_01x08_Male, J14 Conn_01x08_Male, J15 Conn_01x08_Male, J16 Conn_01x08_Male, J17 Conn_01x08_Male, J18 Conn_01x08_Male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

Commit message: Add date & gerber
Routing:
- net (no net): track 0.00 -> 5.08 mm
Other:
- board text added: "31.05.2022"
- board text added: "~En"

Commit message: Add second output
Parts:
- added J21: Conn_01x08_Male, Connector_PinHeader_2.54mm:PinHeader_1x08_P2.54mm_Vertical, F.Cu at (179.1, 88.9)
- moved J11 2.54 mm to (175.3, 88.9)
Routing:
- net /O7: track 101.7 -> 105.7 mm
- net /O6: track 132.9 -> 136.3 mm
- net /G7: track 196.8 -> 199.0 mm
- net /O0: track 125.5 -> 127.5 mm
- net /O1: track 108.8 -> 110.4 mm
- net /O5: track 70.6 -> 71.8 mm
- net /O4: track 99.0 -> 100.3 mm
- net /O3: track 76.2 -> 77.5 mm
- net /O2: track 97.5 -> 98.8 mm
- net /G6: track 219.7 -> 220.8 mm
