File: ALU/ALU.kicad_pcb (KiCad board)
At the start: 2 copper layers, 152.4 x 152.4 mm, 89 parts, among them J1 Conn_01x08_Male, J10 Conn_01x01_Male, J11 Conn_01x08_Male, J12 Conn_01x01_Male, J13 Conn_01x01_Male, J14 Conn_01x03_Male, J15 Conn_01x01_Male, J16 Conn_01x01_Male, J17 Conn_01x01_Male, J18 Conn_01x01_Male, J19 Conn_01x01_Male, J2 Conn_01x08_Male, J20 Conn_01x01_Male, J21 Conn_01x01_Male, J22 Conn_01x01_Male, J23 Conn_01x01_Male, J24 Conn_01x01_Male, J25 Conn_01x01_Male, J26 Conn_01x01_Male, J27 Conn_01x01_Male, J28 Conn_01x01_Male, J29 Conn_01x01_Male, J3 Conn_01x08_Male, J30 Conn_01x01_Male, J31 Conn_01x01_Male, J32 Conn_01x01_Male, J33 Conn_01x01_Male, J34 Conn_01x01_Male, J36 Conn_01x01_Male, J37 Conn_01x01_Male, J38 Conn_01x01_Male, J39 Conn_01x01_Male, J4 Conn_01x01_Male, J5 Conn_01x01_Male, J6 Conn_01x01_Male, J7 Screw_Terminal_01x02, J8 Conn_01x08_Male, J9 Conn_01x01_Male, U1 74HC245, U10 74HC245, U11 CMD, U12 CMD, U13 CMD, U14 CMD, U15 CMD, U16 74HC74, U17 74LS00, U18 74LS08, U19 74LS10, U2 CMD, U20 74LS257, U21 74LS138, U22 74LS10, U23 74HC74, U24 74HC245, U25 74LS138, U26 74LS27, U27 74LS08, U28 74LS257, U29 74LS175, U3 CMD, U4 CMD, U5 CMD, U6 CMD, U7 CMD, U8 74HC245, U9 74LS08

Commit message: Polishing ALU
Parts:
- added J35: Conn_01x01_Male, Connector_PinHeader_2.54mm:PinHeader_1x01_P2.54mm_Vertical, F.Cu at (47.0, 148.3)
- added J40: Conn_01x01_Male, Connector_PinHeader_2.54mm:PinHeader_1x01_P2.54mm_Vertical, F.Cu at (52.7, 150.2)
- moved D3 0.64 mm to (87.0, 154.3)
- moved D4 0.64 mm to (87.0, 164.5)
- moved J34 0.64 mm to (87.0, 151.8)
- moved J36 0.64 mm to (87.0, 167.0)
- moved J37 0.64 mm to (87.0, 158.1)
- moved R10 0.63 mm to (89.5, 157.5)
- moved R11 0.63 mm to (89.5, 161.3)
Connections:
- net Net-(U23-Pad9) renamed /~Bank0
- U23 pad 8: Net-(U23-Pad8) -> /~Bank1
Routing:
- net VCC: track 696.5 -> 704.6 mm
- net /~Bank1: track 0.00 -> 3.57 mm
- net /~Bank0: track 57.8 -> 60.1 mm
- net Net-(U23-Pad13): track 38.9 -> 40.4 mm
- net /~BANK1_CMD: track 95.9 -> 97.2 mm
- net Net-(U23-Pad5): track 76.6 -> 77.6 mm
- net /~EQ_OUT: track 79.5 -> 80.3 mm
- net Net-(U18-Pad3): track 58.0 -> 58.7 mm
- net /~POP_FL: track 81.3 -> 82.0 mm
- net /LT_OUT: track 88.1 -> 88.7 mm
- net /EQ_OUT: track 4.97 -> 5.61 mm
- net GND: track 657.7 -> 658.3 mm
Other:
- board text added: "~Bank0"
- board text added: "~Bank1"

Commit message: Polishing ALU
Parts:
- moved J5 2.22 mm to (95.2, 123.5)
Routing:
- net /COP[1]: track 72.2 -> 75.9 mm
- net /~ACT_BIN: track 72.8 -> 74.2 mm
- net /COP[2]: track 62.7 -> 63.9 mm
- net /~MOV: track 34.5 -> 35.6 mm
- net /COP[0]: track 60.7 -> 61.8 mm

Commit message: Add INC cmd
Parts:
- added J41: Conn_01x01_Male, Connector_PinHeader_2.54mm:PinHeader_1x01_P2.54mm_Vertical, F.Cu at (107.3, 152.4)
- added J42: Conn_01x01_Male, Connector_PinHeader_2.54mm:PinHeader_1x01_P2.54mm_Vertical, F.Cu at (109.9, 152.4)
- U19: value 74LS10 -> 74LS08
- moved J16 104.0 mm to (135.9, 135.9)
- moved U19 64.5 mm to (85.1, 114.9)
- moved U21 9.53 mm to (87.6, 127.6)
- moved R4 9.52 mm to (99.4, 124.5)
- moved J9 7.62 mm to (121.3, 132.7)
- moved J10 7.62 mm to (118.7, 132.7)
- moved J5 7.30 mm to (95.2, 130.8)
Connections:
- U16 pad 5: /ADD_CIN -> Net-(U16-Pad5)
- U17 pad 10: /~LSR_COUT -> Net-(U16-Pad6)
- U17 pad 11: (no net) -> Net-(U17-Pad11)
- U17 pad 12: (no net) -> /~LSL_COUT
- U17 pad 13: (no net) -> /~LSR_COUT
- U17 pad 4: (no net) -> /~ACT_BIN
- U17 pad 5: (no net) -> /~ACT_UNO
- U17 pad 6: (no net) -> Net-(U16-Pad6)
- U17 pad 8: Net-(U17-Pad8) -> /ADD_CIN
- U17 pad 9: /~LSL_COUT -> Net-(U16-Pad6)
- U18 pad 9: /Arithm -> Net-(U16-Pad6)
- U19 pad 1: Net-(U19-Pad1) -> /~ADDC
- U19 pad 10: /~ACT_BIN -> (no net)
- U19 pad 11: /~ACT_UNO -> (no net)
- U19 pad 12: Net-(U19-Pad12) -> (no net)
- U19 pad 13: /~CMPC -> (no net)
- U19 pad 2: /~CMP -> /~INCC
- U19 pad 3: Net-(U19-Pad12) -> Net-(U19-Pad3)
- U19 pad 4: Net-(U19-Pad12) -> Net-(U16-Pad6)
- U19 pad 5: Net-(U19-Pad12) -> /~ADD
- U19 pad 6: /Arithm -> Net-(U19-Pad6)
- U19 pad 8: Net-(U19-Pad1) -> (no net)
- U19 pad 9: /~ACT_BIN -> (no net)
- U20 pad 6: Net-(U17-Pad8) -> Net-(U17-Pad11)
- U21 pad 7: /~CMPC -> /~INCC
- U21 pad 9: /~CMP -> Net-(U16-Pad6)
- U22 pad 10: /~CMPC -> /~CMP
- U22 pad 9: /~CMP -> /~CMPC
- U24 pad 2: /ADD_CIN -> Net-(U16-Pad5)
- U26 pad 9: /Arithm -> Net-(U16-Pad6)
- U3 pad 28: /~ADD -> Net-(U19-Pad6)
- U3 pad 29: /~ADDC -> Net-(U19-Pad3)
Routing:
- net Net-(U16-Pad6): track 0.00 -> 458.7 mm, vias 0 -> 7
- net (no net): track 350.5 -> 0.00 mm, vias 180 -> 0
- net /Arithm: track 289.1 -> 0.00 mm
- net Net-(U17-Pad11): track 0.00 -> 171.2 mm, vias 0 -> 1
- net Net-(U17-Pad8): track 97.2 -> 0.00 mm
- net /~CMPC: track 109.1 -> 58.1 mm, vias 2 -> 0
- net Net-(U16-Pad5): track 0.00 -> 47.5 mm
- net /~CMP: track 107.1 -> 61.7 mm
- net /ADD_CIN: track 47.5 -> 4.44 mm
- net /~ACT_BIN: track 74.2 -> 40.3 mm
- net Net-(U19-Pad1): track 30.4 -> 0.00 mm
- net VCC: track 704.6 -> 676.4 mm, vias 7 -> 5
- net Net-(U19-Pad6): track 0.00 -> 26.8 mm
- net /~INCC: track 0.00 -> 24.2 mm, vias 0 -> 1
- net /~ACT_UNO: track 20.6 -> 43.6 mm
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Other:
- net class Default: trace_width 0.25 -> 0.5; via_dia 0.8 -> 1.5; via_drill 0.4 -> 0.5
- board text added: "CMPC"
