File: MUX4x1/MUX4x1.kicad_pcb (KiCad board)
At the start: 2 copper layers, 85.1 x 50.8 mm, 16 parts, among them J1 Screw_Terminal_01x02, J2 Conn_01x09_Male, J3 Conn_01x09_Male, J4 Conn_01x09_Male, J5 Conn_01x09_Male, J6 Conn_01x09_Male, J7 Conn_01x03_Male, U1 74LS153, U2 74LS153, U3 74LS153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

Commit message: MUX 4:1 ready?
Routing:
- net /C0: track 0.00 -> 165.1 mm
- net /B6: track 0.00 -> 123.4 mm
- net /B7: track 0.00 -> 118.8 mm
- net /A7: track 0.00 -> 107.7 mm
- net /D0: track 0.00 -> 99.6 mm
- net /D1: track 0.00 -> 98.1 mm, vias 0 -> 1
- net /C1: track 0.00 -> 80.4 mm
- net /A6: track 0.00 -> 79.2 mm, vias 0 -> 1
- net /~E: track 3.03 -> 74.9 mm
- net /S1: track 0.00 -> 71.0 mm
- net /S0: track 0.00 -> 67.3 mm
- net /A5: track 0.00 -> 64.3 mm
- net /B5: track 0.00 -> 62.6 mm
- net /C2: track 0.00 -> 58.6 mm
- net /D2: track 0.00 -> 56.0 mm
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