File: 273/273.kicad_pcb (KiCad board)
At the start: 2 copper layers, 22.9 x 27.9 mm, 3 parts, among them J1 Conn_01x10_Male, J2 Conn_01x10_Male, U1 74HC273

Commit message: Polishing 273 socket
Parts:
- moved J2 1.27 mm to (87.6, 33.0)
- moved J1 1.27 mm to (72.4, 33.0)
Routing:
- net /VCC: track 5.08 -> 3.81 mm
- net /Q7: track 5.08 -> 3.81 mm
- net /Q6: track 13.8 -> 12.5 mm
- net /Q5: track 13.8 -> 12.5 mm
- net /Q4: track 5.08 -> 3.81 mm
- net /Q3: track 5.08 -> 3.81 mm
- net /Q2: track 13.8 -> 12.5 mm
- net /Q1: track 13.8 -> 12.5 mm
- net /Q0: track 5.08 -> 3.81 mm
- net /CP: track 5.08 -> 3.81 mm
- net /D7: track 13.8 -> 12.5 mm
- net /D4: track 13.8 -> 12.5 mm
- net /D3: track 13.8 -> 12.5 mm
- net /D0: track 13.8 -> 12.5 mm
- net /~MR: track 5.08 -> 3.81 mm
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Other:
- board size 22.9 x 27.9 mm -> 20.3 x 27.9 mm
