File: MUX4x1-v2/MUX4x1.sch (KiCad schematic (older format))
At the start: 22 parts, among them J1 Screw_Terminal_01x02, J10 Conn_01x09_Male, J11 Conn_01x09_Male, J2 Conn_01x09_Male, J3 Conn_01x09_Male, J4 Conn_01x09_Male, J5 Conn_01x09_Male, J6 Conn_01x09_Male, J7 Conn_01x03_Male, J8 Conn_01x09_Male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

Commit message: Polishing MUX4:1
Parts:
- added J12: Conn_01x09_Male, Connector_PinHeader_2.54mm:PinHeader_1x09_P2.54mm_Vertical, symbol Connector:Conn_01x09_Male
Connections:
- net GND: now also J12.1 (Pin_1)
- net O0: now also J12.2 (Pin_2)
- net O1: now also J12.3 (Pin_3)
- net O2: now also J12.4 (Pin_4)
- net O3: now also J12.5 (Pin_5)
- net O4: now also J12.6 (Pin_6)
- net O5: now also J12.7 (Pin_7)
- net O6: now also J12.8 (Pin_8)
- net O7: now also J12.9 (Pin_9)
Changed lines of the file:
@@
 	1    0    0    -1
 $EndComp
+$Comp
+L Connector:Conn_01x09_Male J12
+U 1 1 6362CA47
+P 6000 6650
+F 0 "J12" H 6108 7231 50  0000 C CNN
+F 1 "Conn_01x09_Male" H 6000 6150 50  0000 C CNN
+F 2 "Connector_PinHeader_2.54mm:PinHeader_1x09_P2.54mm_Vertical" H 6000 6650 50  0001 C CNN
+F 3 "~" H 6000 6650 50  0001 C CNN
+	1    6000 6650
+	1    0    0    -1
+$EndComp
+$Comp
+L power:GND #PWR0107
+U 1 1 6362CA4D
+P 6200 6250
+F 0 "#PWR0107" H 6200 6000 50  0001 C CNN
+F 1 "GND" H 6205 6077 50  0000 C CNN
+F 2 "" H 6200 6250 50  0001 C CNN
+F 3 "" H 6200 6250 50  0001 C CNN
+	1    6200 6250
+	-1   0    0    1
+$EndComp
+Text Label 6200 6350 0    50   ~ 0
+O0
+Text Label 6200 6450 0    50   ~ 0
+O1
+Text Label 6200 6550 0    50   ~ 0
+O2
+Text Label 6200 6650 0    50   ~ 0
+O3
+Text Label 6200 6750 0    50   ~ 0
+O4
+Text Label 6200 6850 0    50   ~ 0
+O5
+Text Label 6200 6950 0    50   ~ 0
+O6
+Text Label 6200 7050 0    50   ~ 0
+O7
 $EndSCHEMATC
