File: MUX8x1-v4/MUX8x1-v4.kicad_pcb (KiCad board)
At the start: 4 copper layers, 99.1 x 99.1 mm, 38 parts, among them J1 Conn_01x09_Male, J10 Conn_01x03_Male, J11 Conn_01x09_Male, J12 Conn_01x09_Male, J14 Conn_01x09_Male, J15 Conn_01x09_Male, J16 Conn_01x09_Male, J18 Conn_01x09_Male, J19 Conn_01x09_Male, J2 Conn_01x09_Male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

Commit message: Add date
Other:
- board text added: "02.12.2022"
