File: RegLed/Reg.kicad_pcb (KiCad board)
At the start: 2 copper layers, 72.1 x 39.4 mm, 25 parts, among them J1 Conn_01x08_Male, J2 Conn_01x08_Male, J3 Conn_01x02_Male, J4 Conn_01x03_Male, U1 74LS573, U2 74HC245, U3 74LS27

Commit message: Polishing RegLED. Gerber.
Parts:
- added C2: 0.1uF, Capacitor_SMD:C_0805_2012Metric_Pad1.18x1.45mm_HandSolder, F.Cu at (86.0, 46.7)
Connections:
- U3 pad 1: (no net) -> GND
- U3 pad 10: (no net) -> GND
- U3 pad 11: (no net) -> GND
- U3 pad 12: (no net) -> Net-(U3-Pad12)
- U3 pad 13: (no net) -> GND
- U3 pad 2: (no net) -> GND
- U3 pad 3: /~Col -> /~CS
- U3 pad 4: /~Row -> /~Col
- U3 pad 5: /~CS -> /~Row
- U3 pad 8: (no net) -> Net-(U3-Pad8)
- U3 pad 9: (no net) -> GND
Routing:
- net GND: track 137.1 -> 178.6 mm
- net Net-(U1-Pad11): track 79.2 -> 70.6 mm
- net /~CS: track 45.6 -> 40.5 mm
- net VCC: track 83.3 -> 86.7 mm
- net /~Row: track 12.1 -> 11.5 mm
- net /~Col: track 11.5 -> 11.0 mm
Other:
- board text added: "11.11.2022"
- board text removed: "23.10.2022"
