File: SWAP/SWAP.sch (KiCad schematic (older format))
At the start: 7 parts, among them J2 Conn_01x08_Male, J3 Conn_01x08_Male, J4 Conn_01x04_Male, U1 74LS573

Commit message: Polishing SWAP cmd
Parts:
- J2, J3: footprint Connector_PinHeader_2.54mm:PinHeader_1x08_P2.54mm_Vertical -> Connector_PinHeader_2.54mm:PinHeader_1x08_P2.54mm_Horizontal
- J4: footprint Connector_PinHeader_2.54mm:PinHeader_1x04_P2.54mm_Vertical -> Connector_PinHeader_2.54mm:PinHeader_1x04_P2.54mm_Horizontal
Changed lines of the file:
@@
 F 0 "J2" H 4358 3431 50  0000 C CNN
 F 1 "Conn_01x08_Male" H 3975 2475 50  0000 C CNN
-F 2 "Connector_PinHeader_2.54mm:PinHeader_1x08_P2.54mm_Vertical" H 4250 2950 50  0001 C CNN
+F 2 "Connector_PinHeader_2.54mm:PinHeader_1x08_P2.54mm_Horizontal" H 4250 2950 50  0001 C CNN
 F 3 "~" H 4250 2950 50  0001 C CNN
 	1    4250 2950
@@
 F 0 "J3" H 7308 3831 50  0000 C CNN
 F 1 "Conn_01x08_Male" H 7300 2775 50  0000 C CNN
-F 2 "Connector_PinHeader_2.54mm:PinHeader_1x08_P2.54mm_Vertical" H 7200 3350 50  0001 C CNN
+F 2 "Connector_PinHeader_2.54mm:PinHeader_1x08_P2.54mm_Horizontal" H 7200 3350 50  0001 C CNN
 F 3 "~" H 7200 3350 50  0001 C CNN
 	1    7200 3350
@@
 F 0 "J4" H 1825 4775 50  0000 C CNN
 F 1 "Conn_01x04_Male" H 1625 5375 50  0000 C CNN
-F 2 "Connector_PinHeader_2.54mm:PinHeader_1x04_P2.54mm_Vertical" H 1750 5150 50  0001 C CNN
+F 2 "Connector_PinHeader_2.54mm:PinHeader_1x04_P2.54mm_Horizontal" H 1750 5150 50  0001 C CNN
 F 3 "~" H 1750 5150 50  0001 C CNN
 	1    1750 5150
