File: INV/INV.sch (KiCad schematic (older format))
At the start: 9 parts, among them J1 Conn_01x08_Male, J2 Conn_01x08_Male, J3 Conn_01x04_Male, U1 74HC00, U2 74LS573, U3 74HC00

Commit message: Polishing INV cmd
Parts:
- added C2, C3: 0.1uF, Capacitor_SMD:C_0805_2012Metric_Pad1.18x1.45mm_HandSolder, symbol Device:C
Connections:
- net GND: now also C2.2, C3.2
- net VCC: now also C2.1, C3.1
Other:
- moved on the sheet: U1E, U3E
Changed lines of the file:
@@
 L 74xx:74HC00 U1
 U 5 1 63830A5A
-P 5450 5300
-F 0 "U1" H 5680 5346 50  0000 L CNN
-F 1 "74HC00" H 5680 5255 50  0000 L CNN
-F 2 "Package_SO:SO-14_3.9x8.65mm_P1.27mm" H 5450 5300 50  0001 C CNN
-F 3 "http://www.ti.com/lit/gpn/sn74hc00" H 5450 5300 50  0001 C CNN
-	5    5450 5300
+P 6450 5300
+F 0 "U1" H 6680 5346 50  0000 L CNN
+F 1 "74HC00" H 6680 5255 50  0000 L CNN
+F 2 "Package_SO:SO-14_3.9x8.65mm_P1.27mm" H 6450 5300 50  0001 C CNN
+F 3 "http://www.ti.com/lit/gpn/sn74hc00" H 6450 5300 50  0001 C CNN
+	5    6450 5300
 	1    0    0    -1
 $EndComp
@@
 L 74xx:74HC00 U3
 U 5 1 638454CE
-P 6450 5300
-F 0 "U3" H 6680 5346 50  0000 L CNN
-F 1 "74HC00" H 6680 5255 50  0000 L CNN
-F 2 "Package_SO:SO-14_3.9x8.65mm_P1.27mm" H 6450 5300 50  0001 C CNN
-F 3 "http://www.ti.com/lit/gpn/sn74hc00" H 6450 5300 50  0001 C CNN
-	5    6450 5300
+P 7200 5300
+F 0 "U3" H 7430 5346 50  0000 L CNN
+F 1 "74HC00" H 7430 5255 50  0000 L CNN
+F 2 "Package_SO:SO-14_3.9x8.65mm_P1.27mm" H 7200 5300 50  0001 C CNN
+F 3 "http://www.ti.com/lit/gpn/sn74hc00" H 7200 5300 50  0001 C CNN
+	5    7200 5300
 	1    0    0    -1
 $EndComp
@@
 L power:GND #PWR09
 U 1 1 6385FD3E
-P 5450 5800
-F 0 "#PWR09" H 5450 5550 50  0001 C CNN
-F 1 "GND" H 5455 5627 50  0000 C CNN
-F 2 "" H 5450 5800 50  0001 C CNN
-F 3 "" H 5450 5800 50  0001 C CNN
-	1    5450 5800
-	1    0    0    -1
-$EndComp
-$Comp
-L power:GND #PWR010
-U 1 1 63860936
 P 6450 5800
-F 0 "#PWR010" H 6450 5550 50  0001 C CNN
+F 0 "#PWR09" H 6450 5550 50  0001 C CNN
 F 1 "GND" H 6455 5627 50  0000 C CNN
 F 2 "" H 6450 5800 50  0001 C CNN
@@
 $EndComp
 $Comp
+L power:GND #PWR010
+U 1 1 63860936
+P 7200 5800
+F 0 "#PWR010" H 7200 5550 50  0001 C CNN
+F 1 "GND" H 7205 5627 50  0000 C CNN
+F 2 "" H 7200 5800 50  0001 C CNN
+F 3 "" H 7200 5800 50  0001 C CNN
+	1    7200 5800
+	1    0    0    -1
+$EndComp
+$Comp
 L power:VCC #PWR03
 U 1 1 63861494
-P 5450 4800
-F 0 "#PWR03" H 5450 4650 50  0001 C CNN
-F 1 "VCC" H 5465 4973 50  0000 C CNN
-F 2 "" H 5450 4800 50  0001 C CNN
-F 3 "" H 5450 4800 50  0001 C CNN
-	1    5450 4800
-	1    0    0    -1
-$EndComp
-$Comp
-L power:VCC #PWR04
-U 1 1 63862208
 P 6450 4800
-F 0 "#PWR04" H 6450 4650 50  0001 C CNN
+F 0 "#PWR03" H 6450 4650 50  0001 C CNN
 F 1 "VCC" H 6465 4973 50  0000 C CNN
 F 2 "" H 6450 4800 50  0001 C CNN
 F 3 "" H 6450 4800 50  0001 C CNN
 	1    6450 4800
+	1    0    0    -1
+$EndComp
+$Comp
+L power:VCC #PWR04
+U 1 1 63862208
+P 7200 4800
+F 0 "#PWR04" H 7200 4650 50  0001 C CNN
+F 1 "VCC" H 7215 4973 50  0000 C CNN
+F 2 "" H 7200 4800 50  0001 C CNN
+F 3 "" H 7200 4800 50  0001 C CNN
+	1    7200 4800
 	1    0    0    -1
 $EndComp
@@
 Text Label 3500 5750 0    50   ~ 0
 ~OE
+$Comp
+L Device:C C2
+U 1 1 63A83AF0
+P 5250 5275
+F 0 "C2" H 5365 5321 50  0000 L CNN
+F 1 "0.1uF" H 5365 5230 50  0000 L CNN
+F 2 "Capacitor_SMD:C_0805_2012Metric_Pad1.18x1.45mm_HandSolder" H 5288 5125 50  0001 C CNN
+F 3 "~" H 5250 5275 50  0001 C CNN
+	1    5250 5275
+	1    0    0    -1
+$EndComp
+$Comp
+L power:VCC #PWR012
+U 1 1 63A83AF6
+P 5250 5125
+F 0 "#PWR012" H 5250 4975 50  0001 C CNN
+F 1 "VCC" H 5265 5298 50  0000 C CNN
+F 2 "" H 5250 5125 50  0001 C CNN
+F 3 "" H 5250 5125 50  0001 C CNN
+	1    5250 5125
+	1    0    0    -1
+$EndComp
+$Comp
+L power:GND #PWR014
+U 1 1 63A83AFC
+P 5250 5425
+F 0 "#PWR014" H 5250 5175 50  0001 C CNN
+F 1 "GND" H 5255 5252 50  0000 C CNN
+F 2 "" H 5250 5425 50  0001 C CNN
+F 3 "" H 5250 5425 50  0001 C CNN
+	1    5250 5425
+	1    0    0    -1
+$EndComp
+$Comp
+L Device:C C3
+U 1 1 63A85FB7
+P 5750 5275
+F 0 "C3" H 5865 5321 50  0000 L CNN
+F 1 "0.1uF" H 5865 5230 50  0000 L CNN
+F 2 "Capacitor_SMD:C_0805_2012Metric_Pad1.18x1.45mm_HandSolder" H 5788 5125 50  0001 C CNN
+F 3 "~" H 5750 5275 50  0001 C CNN
+	1    5750 5275
+	1    0    0    -1
+$EndComp
+$Comp
+L power:VCC #PWR013
+U 1 1 63A85FBD
+P 5750 5125
+F 0 "#PWR013" H 5750 4975 50  0001 C CNN
+F 1 "VCC" H 5765 5298 50  0000 C CNN
+F 2 "" H 5750 5125 50  0001 C CNN
+F 3 "" H 5750 5125 50  0001 C CNN
+	1    5750 5125
+	1    0    0    -1
+$EndComp
+$Comp
+L power:GND #PWR015
+U 1 1 63A85FC3
+P 5750 5425
+F 0 "#PWR015" H 5750 5175 50  0001 C CNN
+F 1 "GND" H 5755 5252 50  0000 C CNN
+F 2 "" H 5750 5425 50  0001 C CNN
+F 3 "" H 5750 5425 50  0001 C CNN
+	1    5750 5425
+	1    0    0    -1
+$EndComp
 $EndSCHEMATC
