File: STACK1/STACK1.kicad_pcb (KiCad board)
At the start: 2 copper layers, 34.3 x 25.4 mm, 23 parts, among them J1 Conn_01x09_Male, J2 Conn_01x09_Male, J3 Conn_01x01_Male, J4 Conn_01x01_Male, U1 74LS574

Commit message: Stack is ready!
Connections:
- net Net-(J2-Pad8) renamed /D7
- net Net-(J3-Pad1) renamed /CP
- net Net-(J4-Pad1) renamed /~OE
Routing:
- net GND: track 0.00 -> 76.2 mm
- net VCC: track 0.00 -> 15.3 mm
- net /Q7: track 0.00 -> 12.7 mm
- net /Q6: track 0.00 -> 11.6 mm
- net /~OE: track 0.00 -> 10.5 mm
- net /Q0: track 0.00 -> 9.81 mm
- net /Q5: track 0.00 -> 9.81 mm
- net /D0: track 0.00 -> 9.43 mm
- net /Q1: track 0.00 -> 9.37 mm
- net /Q4: track 0.00 -> 9.28 mm
- net /Q3: track 0.00 -> 8.85 mm
- net /Q2: track 0.00 -> 8.85 mm
- net Net-(J2-Pad2): track 0.00 -> 8.16 mm
- net Net-(J2-Pad3): track 0.00 -> 6.73 mm
- net /D7: track 0.00 -> 6.73 mm
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Other:
- board text added: "0"
- board text added: "574"
- board text added: "7"
- board text added: "CP"
- board text added: "Data In"
- board text added: "Data Out"
- board text added: "Gnd"
- board text added: "Vcc"
- board text added: "~OE"
