File: MUX4x1-v4/MUX4x1.kicad_pcb (KiCad board)
At the start: 2 copper layers, 87.6 x 65.4 mm, 32 parts, among them J1 Screw_Terminal_01x02, J10 Conn_01x09_Male, J11 Conn_01x09_Male, J12 Conn_01x09_Male, J13 Conn_01x01_Male, J2 Conn_01x09_Male, J3 Conn_01x09_Male, J4 Conn_01x09_Male, J5 Conn_01x09_Male, J6 Conn_01x09_Male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

Commit message: Polishing MUX4:1
Parts:
- added J14: Conn_01x03_Male, Connector_PinHeader_2.54mm:PinHeader_1x03_P2.54mm_Vertical, F.Cu at (139.7, 114.3)
- moved R2 10.9 mm to (152.4, 111.1)
- moved R3 10.9 mm to (154.9, 111.1)
- moved D1 10.2 mm to (152.4, 115.3)
- moved D2 10.2 mm to (154.9, 115.3)
- moved J7 0.95 mm to (145.7, 79.4)
Routing:
- net /~E: track 78.2 -> 125.9 mm
- net /S1: track 88.9 -> 119.0 mm, vias 0 -> 2
- net /S0: track 77.5 -> 101.5 mm
- net GND: track 407.1 -> 416.0 mm, vias 3 -> 2
- net Net-(D2-Pad2): track 3.06 -> 2.10 mm
- net Net-(D1-Pad2): track 3.06 -> 2.10 mm
- net /O7: track 36.8 -> 36.0 mm
- net /D0: vias 2 -> 1
- net /C0: vias 2 -> 1
Other:
- outline, holes or cut-outs redrawn
- board text added: "23.01.2023"
- board text removed: "22.01.2023"

Commit message: Polishing MUX4:1
Routing:
- net /A6: track 81.9 -> 82.7 mm, vias 2 -> 1
- net /D1: track 92.9 -> 92.4 mm
- net /C1: track 50.7 -> 50.1 mm, vias 2 -> 1
- net /A7: track 87.9 -> 87.5 mm, vias 2 -> 1
- net /O4: vias 1 -> 0
- net /O6: vias 1 -> 0
- net /O2: vias 1 -> 0
- net /D6: vias 2 -> 1
- net /D5: vias 2 -> 1
- net /D4: vias 2 -> 1
- net /D3: vias 2 -> 1
- net /D2: vias 2 -> 1
- net /C6: vias 2 -> 1
- net /C5: vias 2 -> 1
- net /C4: vias 2 -> 1
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
Commit message: Fix some silk & power tracks
Routing:
- net GND: track 416.0 -> 410.1 mm, vias 2 -> 1
Other:
- board text added: "18.02.2023"
- board text removed: "23.01.2023"
