File: MUL1/MUL1.kicad_pcb (KiCad board)
At the start: 2 copper layers, 83.8 x 38.1 mm, 11 parts, among them J1 Conn_01x08_Male, J2 Conn_01x09_Male, J3 Conn_01x08_Male, J4 Conn_01x01_Male, J5 Conn_01x02_Male, U1 74LS08, U2 74LS283, U3 74LS08, U4 74LS283

Commit message: Polishing MUL. Add gerber.
Parts:
- C1, C2: footprint Capacitor_SMD:C_0805_2012Metric_Pad1.18x1.45mm_HandSolder -> Capacitor_THT:C_Disc_D7.5mm_W5.0mm_P10.00mm
- moved C1 8.37 mm to (151.8, 58.4)
- moved C2 7.65 mm to (115.6, 59.1)
Routing:
- net Net-(U3-Pad8): track 95.0 -> 65.5 mm, vias 0 -> 2
- net VCC: track 92.9 -> 121.2 mm
- net Net-(U1-Pad8): track 51.9 -> 69.8 mm
- net GND: track 125.3 -> 114.3 mm
- net Net-(U1-Pad6): track 44.8 -> 53.3 mm
- net /P2: track 52.1 -> 58.8 mm
- net /Bi: track 71.9 -> 78.0 mm
- net /P6: track 59.2 -> 65.3 mm
- net /P5: track 29.3 -> 35.1 mm
- net /A6: track 18.8 -> 23.2 mm
- net /P7: track 49.9 -> 54.2 mm
- net /S1: track 36.4 -> 40.5 mm
- net /S2: track 27.7 -> 31.6 mm
- net /P3: track 27.0 -> 30.7 mm
- net /A0: track 28.1 -> 31.5 mm
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Other:
- board size 83.8 x 38.1 mm -> 83.8 x 36.2 mm
- board text added: "0"
- board text added: "7"
- board text added: "8"
- board text added: "A"
- board text added: "Bi"
- board text added: "Gnd"
- board text added: "P"
- board text added: "S"
- board text added: "Vcc"

Commit message: Add jumper to MUL1
Parts:
- added J6: Conn_01x02_Male, Connector_PinHeader_2.54mm:PinHeader_1x02_P2.54mm_Vertical, F.Cu at (116.5, 74.3)
Connections:
- U2 pad 7: GND -> Net-(J6-Pad2)
Routing:
- net Net-(J6-Pad2): track 0.00 -> 3.12 mm
Other:
- board text added: "MUL1"

Commit message: Polishing MUL1
Parts:
- added R1: 10k, Resistor_SMD:R_0805_2012Metric_Pad1.20x1.40mm_HandSolder, F.Cu at (122.6, 71.1)
- J6: value Conn_01x02_Male -> Conn_01x01_Male; footprint Connector_PinHeader_2.54mm:PinHeader_1x02_P2.54mm_Vertical -> Connector_PinHeader_2.54mm:PinHeader_1x01_P2.54mm_Vertical
- moved J6 2.54 mm to (116.5, 71.8), turned to 270 degrees
Connections:
- J6 pad 1: GND -> Net-(J6-Pad1)
- U2 pad 7: Net-(J6-Pad2) -> Net-(J6-Pad1)
Routing:
- net Net-(J6-Pad1): track 0.00 -> 6.71 mm
- net GND: track 114.8 -> 118.3 mm
- net Net-(J6-Pad2): track 3.12 -> 0.00 mm
Other:
- board text added: "+5V"
- board text added: "08"
- board text added: "18.02.2023"
- board text added: "283"
- board text added: "74HCPU"
- board text added: "Cin"

Commit message: Polishing MUL1
Parts:
- moved R1 0.63 mm to (123.2, 71.1)
Routing:
- net GND: track 118.3 -> 140.1 mm
- net VCC: track 121.2 -> 111.1 mm
- net Net-(J6-Pad1): track 6.71 -> 7.34 mm
Other:
- board text added: "13.05.2023"
- board text removed: "18.02.2023"
