File: AND/AND.sch (KiCad schematic (older format))
At the start: 8 parts, among them J1 Conn_01x08_Male, J2 Conn_01x08_Male, J3 Conn_01x08_Male, J4 Conn_01x04_Male, U1 74LS08, U2 74LS08, U3 74LS573

Commit message: New template + 74HC573
Parts:
- removed U1, U2: 74LS08, Package_DIP:DIP-14_W7.62mm, symbol 74xx:74LS08
- removed U3: 74LS573, Package_DIP:DIP-20_W7.62mm, symbol 74xx:74LS573
- added U1: 74LS573, Package_DIP:DIP-20_W7.62mm, symbol 74xx:74LS573
Connections:
- net GND: now also J4.2 (Pin_2), U1.10 (GND); no longer J4.3 (Pin_3)
- net VCC: now also J4.3 (Pin_3), U1.20 (VCC); no longer J4.2 (Pin_2)
- net at J3.1 (Pin_1): now also U1.19 (Q0)
- net at J3.2 (Pin_2): now also U1.18 (Q1)
- net at J3.3 (Pin_3): now also U1.17 (Q2)
- net at J3.4 (Pin_4): now also U1.16 (Q3)
- net at J3.5 (Pin_5): now also U1.15 (Q4)
- net at J3.6 (Pin_6): now also U1.14 (Q5)
- net at J3.7 (Pin_7): now also U1.13 (Q6)
- net at J3.8 (Pin_8): now also U1.12 (Q7)
- net at J4.1 (Pin_1): now also U1.1 (OE)
- net at J4.4 (Pin_4): now also U1.11 (Load)
Other:
- moved on the sheet: C1, J3, J4

Commit message: pcb is ready
Parts:
- added U2, U3: 74LS08, Package_DIP:DIP-14_W7.62mm, symbol 74xx:74LS08
Connections:
- net GND: now also U2.7 (GND), U3.7 (GND)
- net VCC: now also U2.14 (VCC), U3.14 (VCC)
- net at J1.1 (Pin_1): now also U3.9
- net at J1.2 (Pin_2): now also U3.12
- net at J1.3 (Pin_3): now also U3.4
- net at J1.4 (Pin_4): now also U3.1
- net at J1.5 (Pin_5): now also U2.9
- net at J1.6 (Pin_6): now also U2.12
- net at J1.7 (Pin_7): now also U2.4
- net at J1.8 (Pin_8): now also U2.1
- net at J2.1 (Pin_1): now also U3.10
- net at J2.2 (Pin_2): now also U3.13
- net at J2.3 (Pin_3): now also U3.5
- net at J2.4 (Pin_4): now also U3.2
- net at J2.5 (Pin_5): now also U2.10
- net at J2.6 (Pin_6): now also U2.13
- net at J2.7 (Pin_7): now also U2.5
- net at J2.8 (Pin_8): now also U2.2
- net at U1.2 (D0): now also U3.8
- net at U1.3 (D1): now also U3.11
- net at U1.4 (D2): now also U3.6
- net at U1.5 (D3): now also U3.3
- net at U1.6 (D4): now also U2.8
- net at U1.7 (D5): now also U2.11
- net at U1.8 (D6): now also U2.6
- net at U1.9 (D7): now also U2.3
Other:
- moved on the sheet: C1, J1, J2, J3, J4, U1

Commit message: Polishing AND cmd Add date & label
Parts:
- added D1: LED, LED_SMD:LED_0805_2012Metric_Pad1.15x1.40mm_HandSolder, symbol Device:LED
- added R1: 1k, Resistor_SMD:R_0805_2012Metric_Pad1.20x1.40mm_HandSolder, symbol Device:R
Connections:
- net GND: now also D1.1 (K)
- net A7: now reaches J1.1 (Pin_1), U3.9
- net A0: now reaches J1.8 (Pin_8), U2.1
- net B7: now reaches J2.1 (Pin_1), U3.10
- net B0: now reaches J2.8 (Pin_8), U2.2
- net O7: now reaches J3.1 (Pin_1), U1.19 (Q0)
- net O0: now reaches J3.8 (Pin_8), U1.12 (Q7)
- net ~OE: now reaches J4.1 (Pin_1), U1.1 (OE)
- net ~OE: now also R1.1
- net Latch: now reaches J4.4 (Pin_4), U1.11 (Load)
- new net: D1.2 (A), R1.2
Changed lines of the file:
@@
 U 1 1 5F5004CF
 P 1750 3100
-F 0 "J1" H 1858 3581 50  0000 C CNN
-F 1 "Conn_01x08_Male" H 1858 3490 50  0000 C CNN
+F 0 "J1" H 1800 3500 50  0000 C CNN
+F 1 "Conn_01x08_Male" H 1700 2650 50  0000 C CNN
 F 2 "Connector_PinHeader_2.54mm:PinHeader_1x08_P2.54mm_Horizontal" H 1750 3100 50  0001 C CNN
 F 3 "~" H 1750 3100 50  0001 C CNN
@@
 U 1 1 5F5016B1
 P 1750 4100
-F 0 "J2" H 1858 4581 50  0000 C CNN
-F 1 "Conn_01x08_Male" H 1858 4490 50  0000 C CNN
+F 0 "J2" H 1800 4500 50  0000 C CNN
+F 1 "Conn_01x08_Male" H 1700 3650 50  0000 C CNN
 F 2 "Connector_PinHeader_2.54mm:PinHeader_1x08_P2.54mm_Horizontal" H 1750 4100 50  0001 C CNN
 F 3 "~" H 1750 4100 50  0001 C CNN
@@
 U 1 1 5F50268E
 P 1750 5150
-F 0 "J4" H 1825 4775 50  0000 C CNN
-F 1 "Conn_01x04_Male" H 1625 5375 50  0000 C CNN
+F 0 "J4" H 1775 4875 50  0000 C CNN
+F 1 "Conn_01x04_Male" H 1650 5325 50  0000 C CNN
 F 2 "Connector_PinHeader_2.54mm:PinHeader_1x04_P2.54mm_Horizontal" H 1750 5150 50  0001 C CNN
 F 3 "~" H 1750 5150 50  0001 C CNN
@@
 	2025 5250 2025 5675
 Wire Wire Line
-	2025 5675 5750 5675
+	2025 5675 3550 5675
 Wire Wire Line
 	5750 5675 5750 4050
@@
 	5250 3050 5750 3050
 $Comp
-L power:GND #PWR?
+L power:GND #PWR05
 U 1 1 5F5F285E
 P 6475 5900
-F 0 "#PWR?" H 6475 5650 50  0001 C CNN
+F 0 "#PWR05" H 6475 5650 50  0001 C CNN
 F 1 "GND" H 6480 5727 50  0000 C CNN
 F 2 "" H 6475 5900 50  0001 C CNN
@@
 $EndComp
 $Comp
-L power:GND #PWR?
+L power:GND #PWR06
 U 1 1 5F5F35E6
 P 7325 5900
-F 0 "#PWR?" H 7325 5650 50  0001 C CNN
+F 0 "#PWR06" H 7325 5650 50  0001 C CNN
 F 1 "GND" H 7330 5727 50  0000 C CNN
 F 2 "" H 7325 5900 50  0001 C CNN
@@
 $EndComp
 $Comp
-L power:VCC #PWR?
+L power:VCC #PWR03
 U 1 1 5F5F429B
 P 6475 4900
-F 0 "#PWR?" H 6475 4750 50  0001 C CNN
+F 0 "#PWR03" H 6475 4750 50  0001 C CNN
 F 1 "VCC" H 6492 5073 50  0000 C CNN
 F 2 "" H 6475 4900 50  0001 C CNN
@@
 $EndComp
 $Comp
-L power:VCC #PWR?
+L power:VCC #PWR04
 U 1 1 5F5F500E
 P 7325 4900
-F 0 "#PWR?" H 7325 4750 50  0001 C CNN
+F 0 "#PWR04" H 7325 4750 50  0001 C CNN
 F 1 "VCC" H 7342 5073 50  0000 C CNN
 F 2 "" H 7325 4900 50  0001 C CNN
@@
 	1    0    0    -1
 $EndComp
+$Comp
+L Device:R R1
+U 1 1 635F51D3
+P 3550 5825
+F 0 "R1" H 3600 5875 50  0000 L CNN
+F 1 "1k" V 3550 5775 50  0000 L CNN
+F 2 "Resistor_SMD:R_0805_2012Metric_Pad1.20x1.40mm_HandSolder" V 3480 5825 50  0001 C CNN
+F 3 "~" H 3550 5825 50  0001 C CNN
+	1    3550 5825
+	1    0    0    -1
+$EndComp
+$Comp
+L Device:LED D1
+U 1 1 635F5DFD
+P 3550 6125
+F 0 "D1" H 3550 6225 50  0000 C CNN
+F 1 "LED" H 3575 6025 50  0000 C CNN
+F 2 "LED_SMD:LED_0805_2012Metric_Pad1.15x1.40mm_HandSolder" H 3550 6125 50  0001 C CNN
+F 3 "~" H 3550 6125 50  0001 C CNN
+	1    3550 6125
+	0    -1   -1   0
+$EndComp
+Connection ~ 3550 5675
+Wire Wire Line
+	3550 5675 5750 5675
+$Comp
+L power:GND #PWR07
+U 1 1 6360635D
+P 3550 6275
+F 0 "#PWR07" H 3550 6025 50  0001 C CNN
+F 1 "GND" H 3555 6102 50  0000 C CNN
+F 2 "" H 3550 6275 50  0001 C CNN
+F 3 "" H 3550 6275 50  0001 C CNN
+	1    3550 6275
+	1    0    0    -1
+$EndComp
+Text Label 2200 5675 0    50   ~ 0
+~OE
+Text Label 2250 4625 0    50   ~ 0
+Latch
+Text Label 1975 2800 0    50   ~ 0
+A7
+Text Label 1975 3500 0    50   ~ 0
+A0
+Text Label 1975 3800 0    50   ~ 0
+B7
+Text Label 2000 4500 0    50   ~ 0
+B0
+Text Label 6875 3050 0    50   ~ 0
+O7
+Text Label 6875 3750 0    50   ~ 0
+O0
 $EndSCHEMATC

Commit message: AND cmd. Swap SRC & DST busses
Connections:
- net A0: now also J2.8 (Pin_8), U2.2; no longer J1.8 (Pin_8), U2.1
- net A7: now also J2.1 (Pin_1), U3.10; no longer J1.1 (Pin_1), U3.9
- net B0: now also J1.8 (Pin_8), U2.1; no longer J2.8 (Pin_8), U2.2
- net B7: now also J1.1 (Pin_1), U3.9; no longer J2.1 (Pin_1), U3.10
Changed lines of the file:
@@
 	1    0    0    1
 $EndComp
-Text Notes 1400 3150 0    50   ~ 0
+Text Notes 1525 4150 0    50   ~ 0
 A
-Text Notes 1425 4125 0    50   ~ 0
+Text Notes 1525 3150 0    50   ~ 0
 B
 Text Notes 7375 3425 0    50   ~ 0
@@
 Latch
 Text Label 1975 2800 0    50   ~ 0
+B7
+Text Label 1975 3500 0    50   ~ 0
+B0
+Text Label 1975 3800 0    50   ~ 0
 A7
-Text Label 1975 3500 0    50   ~ 0
+Text Label 2000 4500 0    50   ~ 0
 A0
-Text Label 1975 3800 0    50   ~ 0
-B7
-Text Label 2000 4500 0    50   ~ 0
-B0
 Text Label 6875 3050 0    50   ~ 0
 O7
