File: MUX4x1-v5/MUX4x1.sch (KiCad schematic (older format))
At the start: 28 parts, among them J1 Screw_Terminal_01x02, J12 Conn_01x09_Male, J13 Conn_01x01_Male, J2 Conn_01x09_Male, J3 Conn_01x09_Male, J4 Conn_01x09_Male, J5 Conn_01x09_Male, J6 Conn_01x09_Male, J7 Conn_01x03_Male, U1 74LS153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

Commit message: MUX4:1 v5 in work
Parts:
- added C4, C5: 0.1uF, Capacitor_SMD:C_0805_2012Metric_Pad1.18x1.45mm_HandSolder, symbol Device:C
Connections:
- net GND: now also C4.2, C5.2
- net S0: now also J7.2 (Pin_2), R3.2; no longer J7.1 (Pin_1), R2.2
- net S1: now also J7.1 (Pin_1), R2.2; no longer J7.2 (Pin_2), R3.2
- net VCC: now also C4.1, C5.1
Other:
- moved on the sheet: C1, C2
Changed lines of the file:
@@
 	1    0    0    -1
 $EndComp
+Text Label 6950 5100 0    50   ~ 0
+S0
 Text Label 6950 5000 0    50   ~ 0
-S0
-Text Label 6950 5100 0    50   ~ 0
 S1
 Text Label 6950 5200 0    50   ~ 0
@@
 L Device:C C1
 U 1 1 6366F825
-P 8500 5750
-F 0 "C1" H 8615 5796 50  0000 L CNN
-F 1 "0.1uF" H 8615 5705 50  0000 L CNN
-F 2 "Capacitor_SMD:C_0805_2012Metric_Pad1.18x1.45mm_HandSolder" H 8538 5600 50  0001 C CNN
-F 3 "~" H 8500 5750 50  0001 C CNN
-	1    8500 5750
+P 7750 6250
+F 0 "C1" H 7865 6296 50  0000 L CNN
+F 1 "0.1uF" H 7865 6205 50  0000 L CNN
+F 2 "Capacitor_SMD:C_0805_2012Metric_Pad1.18x1.45mm_HandSolder" H 7788 6100 50  0001 C CNN
+F 3 "~" H 7750 6250 50  0001 C CNN
+	1    7750 6250
 	1    0    0    -1
 $EndComp
@@
 L power:VCC #PWR019
 U 1 1 6366FC74
-P 8500 5600
-F 0 "#PWR019" H 8500 5450 50  0001 C CNN
-F 1 "VCC" H 8515 5773 50  0000 C CNN
-F 2 "" H 8500 5600 50  0001 C CNN
-F 3 "" H 8500 5600 50  0001 C CNN
-	1    8500 5600
+P 7750 6100
+F 0 "#PWR019" H 7750 5950 50  0001 C CNN
+F 1 "VCC" H 7765 6273 50  0000 C CNN
+F 2 "" H 7750 6100 50  0001 C CNN
+F 3 "" H 7750 6100 50  0001 C CNN
+	1    7750 6100
 	1    0    0    -1
 $EndComp
@@
 L power:GND #PWR020
 U 1 1 636700DF
-P 8500 5900
-F 0 "#PWR020" H 8500 5650 50  0001 C CNN
-F 1 "GND" H 8505 5727 50  0000 C CNN
-F 2 "" H 8500 5900 50  0001 C CNN
-F 3 "" H 8500 5900 50  0001 C CNN
-	1    8500 5900
+P 7750 6400
+F 0 "#PWR020" H 7750 6150 50  0001 C CNN
+F 1 "GND" H 7755 6227 50  0000 C CNN
+F 2 "" H 7750 6400 50  0001 C CNN
+F 3 "" H 7750 6400 50  0001 C CNN
+	1    7750 6400
 	1    0    0    -1
 $EndComp
@@
 L Device:C C2
 U 1 1 636F284C
-P 9000 5750
-F 0 "C2" H 9115 5796 50  0000 L CNN
-F 1 "0.1uF" H 9115 5705 50  0000 L CNN
-F 2 "Capacitor_SMD:C_0805_2012Metric_Pad1.18x1.45mm_HandSolder" H 9038 5600 50  0001 C CNN
-F 3 "~" H 9000 5750 50  0001 C CNN
-	1    9000 5750
+P 8250 6250
+F 0 "C2" H 8365 6296 50  0000 L CNN
+F 1 "0.1uF" H 8365 6205 50  0000 L CNN
+F 2 "Capacitor_SMD:C_0805_2012Metric_Pad1.18x1.45mm_HandSolder" H 8288 6100 50  0001 C CNN
+F 3 "~" H 8250 6250 50  0001 C CNN
+	1    8250 6250
 	1    0    0    -1
 $EndComp
@@
 L power:VCC #PWR021
 U 1 1 636F2852
-P 9000 5600
-F 0 "#PWR021" H 9000 5450 50  0001 C CNN
-F 1 "VCC" H 9015 5773 50  0000 C CNN
-F 2 "" H 9000 5600 50  0001 C CNN
-F 3 "" H 9000 5600 50  0001 C CNN
-	1    9000 5600
+P 8250 6100
+F 0 "#PWR021" H 8250 5950 50  0001 C CNN
+F 1 "VCC" H 8265 6273 50  0000 C CNN
+F 2 "" H 8250 6100 50  0001 C CNN
+F 3 "" H 8250 6100 50  0001 C CNN
+	1    8250 6100
 	1    0    0    -1
 $EndComp
@@
 L power:GND #PWR022
 U 1 1 636F2858
-P 9000 5900
-F 0 "#PWR022" H 9000 5650 50  0001 C CNN
-F 1 "GND" H 9005 5727 50  0000 C CNN
-F 2 "" H 9000 5900 50  0001 C CNN
-F 3 "" H 9000 5900 50  0001 C CNN
-	1    9000 5900
+P 8250 6400
+F 0 "#PWR022" H 8250 6150 50  0001 C CNN
+F 1 "GND" H 8255 6227 50  0000 C CNN
+F 2 "" H 8250 6400 50  0001 C CNN
+F 3 "" H 8250 6400 50  0001 C CNN
+	1    8250 6400
 	1    0    0    -1
 $EndComp
@@
 	1    0    0    -1
 $EndComp
+$Comp
+L Device:C C4
+U 1 1 6487349D
+P 8750 6250
+F 0 "C4" H 8865 6296 50  0000 L CNN
+F 1 "0.1uF" H 8865 6205 50  0000 L CNN
+F 2 "Capacitor_SMD:C_0805_2012Metric_Pad1.18x1.45mm_HandSolder" H 8788 6100 50  0001 C CNN
+F 3 "~" H 8750 6250 50  0001 C CNN
+	1    8750 6250
+	1    0    0    -1
+$EndComp
+$Comp
+L power:VCC #PWR025
+U 1 1 648734A3
+P 8750 6100
+F 0 "#PWR025" H 8750 5950 50  0001 C CNN
+F 1 "VCC" H 8765 6273 50  0000 C CNN
+F 2 "" H 8750 6100 50  0001 C CNN
+F 3 "" H 8750 6100 50  0001 C CNN
+	1    8750 6100
+	1    0    0    -1
+$EndComp
+$Comp
+L power:GND #PWR027
+U 1 1 648734A9
+P 8750 6400
+F 0 "#PWR027" H 8750 6150 50  0001 C CNN
+F 1 "GND" H 8755 6227 50  0000 C CNN
+F 2 "" H 8750 6400 50  0001 C CNN
+F 3 "" H 8750 6400 50  0001 C CNN
+	1    8750 6400
+	1    0    0    -1
+$EndComp
+$Comp
+L Device:C C5
+U 1 1 648734AF
+P 9250 6250
+F 0 "C5" H 9365 6296 50  0000 L CNN
+F 1 "0.1uF" H 9365 6205 50  0000 L CNN
+F 2 "Capacitor_SMD:C_0805_2012Metric_Pad1.18x1.45mm_HandSolder" H 9288 6100 50  0001 C CNN
+F 3 "~" H 9250 6250 50  0001 C CNN
+	1    9250 6250
+	1    0    0    -1
+$EndComp
+$Comp
+L power:VCC #PWR026
+U 1 1 648734B5
+P 9250 6100
+F 0 "#PWR026" H 9250 5950 50  0001 C CNN
+F 1 "VCC" H 9265 6273 50  0000 C CNN
+F 2 "" H 9250 6100 50  0001 C CNN
+F 3 "" H 9250 6100 50  0001 C CNN
+	1    9250 6100
+	1    0    0    -1
+$EndComp
+$Comp
+L power:GND #PWR028
+U 1 1 648734BB
+P 9250 6400
+F 0 "#PWR028" H 9250 6150 50  0001 C CNN
+F 1 "GND" H 9255 6227 50  0000 C CNN
+F 2 "" H 9250 6400 50  0001 C CNN
+F 3 "" H 9250 6400 50  0001 C CNN
+	1    9250 6400
+	1    0    0    -1
+$EndComp
