File: CMP/CMP.sch (KiCad schematic (older format))
At the start: 12 parts, among them J1 Conn_01x04_Male, J2 Conn_01x08_Male, J3 Conn_01x08_Male, J4 Conn_01x08_Male, J5 Conn_01x03_Male, J6 Conn_01x03_Male, J7 Conn_01x01_Male, U1 74LS85, U2 74HC4078, U3 74LS85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

Commit message: CMP cmd is ready
Parts:
- added R1: 10k, Resistor_SMD:R_0805_2012Metric_Pad1.20x1.40mm_HandSolder, symbol Device:R
Connections:
- net EQ: now also J5.2 (Pin_2); no longer J5.3 (Pin_3)
- net EQ(I): now also U5.8; no longer U4.8
- net EQ_IN: now also J6.1 (Pin_1), U5.12, U5.13; no longer J6.3 (Pin_3), U5.1, U5.2
- net Expand: now also U4.12, U5.9, R1.1; no longer U4.2, U5.5
- net GND: now also U4.1, U4.2, U4.4, U4.5, U5.1, U5.2, U5.4, U5.5, R1.2
- net GT: now also J5.3 (Pin_3); no longer J5.1 (Pin_1)
- net GT(I): now also U4.8; no longer U4.3
- net GT_IN: now also J6.3 (Pin_3), U4.9; no longer J6.1 (Pin_1), U4.1
- net LT: now also J5.1 (Pin_1); no longer J5.2 (Pin_2)
- net LT(I): now also U4.11; no longer U5.6
- net LT_IN: now also U4.13; no longer U5.4
- net O0: now also U2.2 (A); no longer U2.5 (D)
- net O1: now also U2.3 (B); no longer U2.4 (C)
- net O2: now also U2.4 (C); no longer U2.9 (E)
- net O3: now also U2.5 (D); no longer U2.10 (F)
- net O4: now also U2.9 (E); no longer U2.11 (G)
- net O5: now also U2.10 (F); no longer U2.12 (H)
- net O6: now also U2.11 (G); no longer U2.3 (B)
- net O7: now also U2.12 (H); no longer U2.2 (A)
- net at U5.3: no longer U4.9
- net at U5.10: now also U5.11
- no-connect marks 14 -> 6
Other:
- moved on the sheet: U4A, U4C, U4D, U5A, U5B, U5C, U5D
Changed lines of the file:
@@
 Text Label 1950 1800 0    50   ~ 0
 Latch
+Text Label 2500 6250 0    50   ~ 0
+O0
+Text Label 2500 6300 0    50   ~ 0
+O1
+Text Label 2500 6350 0    50   ~ 0
+O2
 Text Label 2500 6400 0    50   ~ 0
-O0
-Text Label 2500 6350 0    50   ~ 0
-O1
+O3
 Text Label 2500 6450 0    50   ~ 0
-O2
+O4
 Text Label 2500 6500 0    50   ~ 0
-O3
-Text Label 2500 6550 0    50   ~ 0
-O4
+O5
 Text Label 2500 6600 0    50   ~ 0
-O5
-Text Label 2500 6250 0    50   ~ 0
 O7
 $Comp
@@
 U 1 1 6363769E
 P 5200 1100
-F 0 "J6" H 5200 1300 50  0000 C CNN
-F 1 "Conn_01x03_Male" H 5200 925 50  0000 C CNN
+F 0 "J6" H 5225 925 50  0000 C CNN
+F 1 "Conn_01x03_Male" H 5200 1300 50  0000 C CNN
 F 2 "Connector_PinHeader_2.54mm:PinHeader_1x03_P2.54mm_Horizontal" H 5200 1100 50  0001 C CNN
 F 3 "~" H 5200 1100 50  0001 C CNN
 	1    5200 1100
-	1    0    0    -1
-$EndComp
+	1    0    0    1
+$EndComp
+Text Label 3850 1200 0    50   ~ 0
+GT
 Text Label 3850 1000 0    50   ~ 0
-GT
+LT
 Text Label 3850 1100 0    50   ~ 0
-LT
-Text Label 3850 1200 0    50   ~ 0
 EQ
-Text Label 2500 6300 0    50   ~ 0
+Text Label 2500 6550 0    50   ~ 0
 O6
 Wire Wire Line
@@
 L 74xx:74LS08 U4
 U 1 1 63674782
-P 6950 850
-F 0 "U4" H 6825 1050 50  0000 C CNN
-F 1 "74LS08" H 7075 1050 50  0000 C CNN
-F 2 "Package_SO:SO-14_3.9x8.65mm_P1.27mm" H 6950 850 50  0001 C CNN
-F 3 "http://www.ti.com/lit/gpn/sn74LS08" H 6950 850 50  0001 C CNN
-	1    6950 850
+P 10300 1350
+F 0 "U4" H 10175 1550 50  0000 C CNN
+F 1 "74LS08" H 10425 1550 50  0000 C CNN
+F 2 "Package_SO:SO-14_3.9x8.65mm_P1.27mm" H 10300 1350 50  0001 C CNN
+F 3 "http://www.ti.com/lit/gpn/sn74LS08" H 10300 1350 50  0001 C CNN
+	1    10300 1350
 	1    0    0    -1
 $EndComp
@@
 L 74xx:74LS08 U4
 U 3 1 636776F1
-P 6950 1850
-F 0 "U4" H 6825 2050 50  0000 C CNN
-F 1 "74LS08" H 7075 2050 50  0000 C CNN
-F 2 "Package_SO:SO-14_3.9x8.65mm_P1.27mm" H 6950 1850 50  0001 C CNN
-F 3 "http://www.ti.com/lit/gpn/sn74LS08" H 6950 1850 50  0001 C CNN
-	3    6950 1850
+P 6950 850
+F 0 "U4" H 6825 1050 50  0000 C CNN
+F 1 "74LS08" H 7075 1050 50  0000 C CNN
+F 2 "Package_SO:SO-14_3.9x8.65mm_P1.27mm" H 6950 850 50  0001 C CNN
+F 3 "http://www.ti.com/lit/gpn/sn74LS08" H 6950 850 50  0001 C CNN
+	3    6950 850
 	1    0    0    -1
 $EndComp
@@
 L 74xx:74LS08 U4
 U 4 1 63679175
-P 10300 1350
-F 0 "U4" H 10300 1675 50  0000 C CNN
-F 1 "74LS08" H 10300 1584 50  0000 C CNN
-F 2 "Package_SO:SO-14_3.9x8.65mm_P1.27mm" H 10300 1350 50  0001 C CNN
-F 3 "http://www.ti.com/lit/gpn/sn74LS08" H 10300 1350 50  0001 C CNN
-	4    10300 1350
-	1    0    0    -1
+P 6950 1350
+F 0 "U4" H 6950 1675 50  0000 C CNN
+F 1 "74LS08" H 6950 1584 50  0000 C CNN
+F 2 "Package_SO:SO-14_3.9x8.65mm_P1.27mm" H 6950 1350 50  0001 C CNN
+F 3 "http://www.ti.com/lit/gpn/sn74LS08" H 6950 1350 50  0001 C CNN
+	4    6950 1350
+	1    0    0    1
 $EndComp
 $Comp
@@
 L 74xx:74LS00 U5
 U 1 1 6369DF1D
+P 9300 1850
+F 0 "U5" H 9175 2050 50  0000 C CNN
+F 1 "74LS00" H 9425 2050 50  0000 C CNN
+F 2 "Package_SO:SO-14_3.9x8.65mm_P1.27mm" H 9300 1850 50  0001 C CNN
+F 3 "http://www.ti.com/lit/gpn/sn74ls00" H 9300 1850 50  0001 C CNN
+	1    9300 1850
+	1    0    0    -1
+$EndComp
+$Comp
+L 74xx:74LS00 U5
+U 2 1 636A1716
+P 9300 1350
+F 0 "U5" H 9175 1550 50  0000 C CNN
+F 1 "74LS00" H 9450 1550 50  0000 C CNN
+F 2 "Package_SO:SO-14_3.9x8.65mm_P1.27mm" H 9300 1350 50  0001 C CNN
+F 3 "http://www.ti.com/lit/gpn/sn74ls00" H 9300 1350 50  0001 C CNN
+	2    9300 1350
+	1    0    0    -1
+$EndComp
+$Comp
+L 74xx:74LS00 U5
+U 3 1 636A34E9
+P 6950 1850
+F 0 "U5" H 6950 2175 50  0000 C CNN
+F 1 "74LS00" H 6950 2084 50  0000 C CNN
+F 2 "Package_SO:SO-14_3.9x8.65mm_P1.27mm" H 6950 1850 50  0001 C CNN
+F 3 "http://www.ti.com/lit/gpn/sn74ls00" H 6950 1850 50  0001 C CNN
+	3    6950 1850
+	1    0    0    1
+$EndComp
+$Comp
+L 74xx:74LS00 U5
+U 4 1 636A5509
 P 6050 1750
-F 0 "U5" H 5925 1950 50  0000 C CNN
-F 1 "74LS00" H 6175 1950 50  0000 C CNN
+F 0 "U5" H 6050 2075 50  0000 C CNN
+F 1 "74LS00" H 6050 1984 50  0000 C CNN
 F 2 "Package_SO:SO-14_3.9x8.65mm_P1.27mm" H 6050 1750 50  0001 C CNN
 F 3 "http://www.ti.com/lit/gpn/sn74ls00" H 6050 1750 50  0001 C CNN
-	1    6050 1750
-	1    0    0    -1
-$EndComp
-$Comp
-L 74xx:74LS00 U5
-U 2 1 636A1716
-P 6950 1350
-F 0 "U5" H 6825 1550 50  0000 C CNN
-F 1 "74LS00" H 7100 1550 50  0000 C CNN
-F 2 "Package_SO:SO-14_3.9x8.65mm_P1.27mm" H 6950 1350 50  0001 C CNN
-F 3 "http://www.ti.com/lit/gpn/sn74ls00" H 6950 1350 50  0001 C CNN
-	2    6950 1350
-	1    0    0    -1
-$EndComp
-$Comp
-L 74xx:74LS00 U5
-U 3 1 636A34E9
-P 9300 1350
-F 0 "U5" H 9300 1675 50  0000 C CNN
-F 1 "74LS00" H 9300 1584 50  0000 C CNN
-F 2 "Package_SO:SO-14_3.9x8.65mm_P1.27mm" H 9300 1350 50  0001 C CNN
-F 3 "http://www.ti.com/lit/gpn/sn74ls00" H 9300 1350 50  0001 C CNN
-	3    9300 1350
-	1    0    0    -1
-$EndComp
-$Comp
-L 74xx:74LS00 U5
-U 4 1 636A5509
-P 9300 1850
-F 0 "U5" H 9300 2175 50  0000 C CNN
-F 1 "74LS00" H 9300 2084 50  0000 C CNN
-F 2 "Package_SO:SO-14_3.9x8.65mm_P1.27mm" H 9300 1850 50  0001 C CNN
-F 3 "http://www.ti.com/lit/gpn/sn74ls00" H 9300 1850 50  0001 C CNN
-	4    9300 1850
+	4    6050 1750
 	1    0    0    -1
 $EndComp
@@
 EQ(I)
 Connection ~ 6400 950
-Text Label 5500 1000 0    50   ~ 0
+Text Label 5475 1000 0    50   ~ 0
 GT_IN
-Text Label 5500 1100 0    50   ~ 0
+Text Label 5475 1100 0    50   ~ 0
 LT_IN
-Text Label 5500 1200 0    50   ~ 0
+Text Label 5475 1200 0    50   ~ 0
 EQ_IN
-Text Notes 5975 2275 0    50   ~ 0
+Text Notes 5825 675  0    50   ~ 0
 Expand == 0: CMP\nExpand == 1: CMPC
-NoConn ~ 9000 1250
-NoConn ~ 9000 1450
-NoConn ~ 9000 1750
-NoConn ~ 9000 1950
 NoConn ~ 9600 1350
 NoConn ~ 9600 1850
-NoConn ~ 10000 1250
-NoConn ~ 10000 1450
-NoConn ~ 10000 1750
-NoConn ~ 10000 1950
 NoConn ~ 10600 1350
 NoConn ~ 10600 1850
@@
 NoConn ~ 1950 1800
 NoConn ~ 3025 6375
+$Comp
+L Device:R R1
+U 1 1 63668488
+P 6400 2100
+F 0 "R1" H 6450 2150 50  0000 L CNN
+F 1 "10k" V 6400 2025 50  0000 L CNN
+F 2 "Resistor_SMD:R_0805_2012Metric_Pad1.20x1.40mm_HandSolder" V 6330 2100 50  0001 C CNN
+F 3 "~" H 6400 2100 50  0001 C CNN
+	1    6400 2100
+	1    0    0    -1
+$EndComp
+Connection ~ 6400 1950
+$Comp
+L power:GND #PWR0107
+U 1 1 6366A6F1
+P 6400 2250
+F 0 "#PWR0107" H 6400 2000 50  0001 C CNN
+F 1 "GND" H 6405 2077 50  0000 C CNN
+F 2 "" H 6400 2250 50  0001 C CNN
+F 3 "" H 6400 2250 50  0001 C CNN
+	1    6400 2250
+	1    0    0    -1
+$EndComp
+$Comp
+L power:GND #PWR?
+U 1 1 636D17CE
+P 9000 1250
+F 0 "#PWR?" H 9000 1000 50  0001 C CNN
+F 1 "GND" V 9005 1122 50  0000 R CNN
+F 2 "" H 9000 1250 50  0001 C CNN
+F 3 "" H 9000 1250 50  0001 C CNN
+	1    9000 1250
+	0    1    1    0
+$EndComp
+$Comp
+L power:GND #PWR?
+U 1 1 636D1D8D
+P 9000 1450
+F 0 "#PWR?" H 9000 1200 50  0001 C CNN
+F 1 "GND" V 9005 1322 50  0000 R CNN
+F 2 "" H 9000 1450 50  0001 C CNN
+F 3 "" H 9000 1450 50  0001 C CNN
+	1    9000 1450
+	0    1    1    0
+$EndComp
+$Comp
+L power:GND #PWR?
+U 1 1 636D2127
+P 9000 1750
+F 0 "#PWR?" H 9000 1500 50  0001 C CNN
+F 1 "GND" V 9005 1622 50  0000 R CNN
+F 2 "" H 9000 1750 50  0001 C CNN
+F 3 "" H 9000 1750 50  0001 C CNN
+	1    9000 1750
+	0    1    1    0
+$EndComp
+$Comp
+L power:GND #PWR?
+U 1 1 636D23FB
+P 9000 1950
+F 0 "#PWR?" H 9000 1700 50  0001 C CNN
+F 1 "GND" V 9005 1822 50  0000 R CNN
+F 2 "" H 9000 1950 50  0001 C CNN
+F 3 "" H 9000 1950 50  0001 C CNN
+	1    9000 1950
+	0    1    1    0
+$EndComp
+$Comp
+L power:GND #PWR?
+U 1 1 636D26AD
+P 10000 1250
+F 0 "#PWR?" H 10000 1000 50  0001 C CNN
+F 1 "GND" V 10005 1122 50  0000 R CNN
+F 2 "" H 10000 1250 50  0001 C CNN
+F 3 "" H 10000 1250 50  0001 C CNN
+	1    10000 1250
+	0    1    1    0
+$EndComp
+$Comp
+L power:GND #PWR?
+U 1 1 636D2A90
+P 10000 1450
+F 0 "#PWR?" H 10000 1200 50  0001 C CNN
+F 1 "GND" V 10005 1322 50  0000 R CNN
+F 2 "" H 10000 1450 50  0001 C CNN
+F 3 "" H 10000 1450 50  0001 C CNN
+	1    10000 1450
+	0    1    1    0
+$EndComp
+$Comp
+L power:GND #PWR?
+U 1 1 636D2D3F
+P 10000 1750
+F 0 "#PWR?" H 10000 1500 50  0001 C CNN
+F 1 "GND" V 10005 1622 50  0000 R CNN
+F 2 "" H 10000 1750 50  0001 C CNN
+F 3 "" H 10000 1750 50  0001 C CNN
+	1    10000 1750
+	0    1    1    0
+$EndComp
+$Comp
+L power:GND #PWR?
+U 1 1 636D301A
+P 10000 1950
+F 0 "#PWR?" H 10000 1700 50  0001 C CNN
+F 1 "GND" V 10005 1822 50  0000 R CNN
+F 2 "" H 10000 1950 50  0001 C CNN
+F 3 "" H 10000 1950 50  0001 C CNN
+	1    10000 1950
+	0    1    1    0
+$EndComp
 $EndSCHEMATC

Commit message: Add lost invertor and caps
Parts:
- added C1, C2: 0.1uF, Capacitor_THT:C_Axial_L3.8mm_D2.6mm_P12.50mm_Horizontal, symbol Device:C
Connections:
- net EQ: now also J5.1 (Pin_1), U5.3; no longer J5.2 (Pin_2), U1.6 (Oa=b)
- net GND: now also C1.2, C2.2; no longer U5.1, U5.2
- net LT: now also J5.2 (Pin_2); no longer J5.1 (Pin_1)
- net VCC: now also C1.1, C2.1
- new net: U1.6 (Oa=b), U5.1, U5.2
- no-connect marks 6 -> 5
Other:
- moved on the sheet: U5A
Changed lines of the file:
@@
 Text Label 4750 3200 0    50   ~ 0
 LT
-Text Label 4750 3300 0    50   ~ 0
+Text Label 6350 3400 0    50   ~ 0
 EQ
 $Comp
@@
 Text Label 3850 1200 0    50   ~ 0
 GT
+Text Label 3850 1100 0    50   ~ 0
+LT
 Text Label 3850 1000 0    50   ~ 0
-LT
-Text Label 3850 1100 0    50   ~ 0
 EQ
 Text Label 2500 6550 0    50   ~ 0
@@
 L 74xx:74LS00 U5
 U 1 1 6369DF1D
-P 9300 1850
-F 0 "U5" H 9175 2050 50  0000 C CNN
-F 1 "74LS00" H 9425 2050 50  0000 C CNN
-F 2 "Package_SO:SO-14_3.9x8.65mm_P1.27mm" H 9300 1850 50  0001 C CNN
-F 3 "http://www.ti.com/lit/gpn/sn74ls00" H 9300 1850 50  0001 C CNN
-	1    9300 1850
+P 6050 3400
+F 0 "U5" H 5925 3600 50  0000 C CNN
+F 1 "74LS00" H 6175 3600 50  0000 C CNN
+F 2 "Package_SO:SO-14_3.9x8.65mm_P1.27mm" H 6050 3400 50  0001 C CNN
+F 3 "http://www.ti.com/lit/gpn/sn74ls00" H 6050 3400 50  0001 C CNN
+	1    6050 3400
 	1    0    0    -1
 $EndComp
@@
 Expand == 0: CMP\nExpand == 1: CMPC
 NoConn ~ 9600 1350
-NoConn ~ 9600 1850
 NoConn ~ 10600 1350
 NoConn ~ 10600 1850
@@
 $EndComp
 $Comp
-L power:GND #PWR?
+L power:GND #PWR0108
 U 1 1 636D17CE
 P 9000 1250
-F 0 "#PWR?" H 9000 1000 50  0001 C CNN
+F 0 "#PWR0108" H 9000 1000 50  0001 C CNN
 F 1 "GND" V 9005 1122 50  0000 R CNN
 F 2 "" H 9000 1250 50  0001 C CNN
@@
 $EndComp
 $Comp
-L power:GND #PWR?
+L power:GND #PWR0109
 U 1 1 636D1D8D
 P 9000 1450
-F 0 "#PWR?" H 9000 1200 50  0001 C CNN
+F 0 "#PWR0109" H 9000 1200 50  0001 C CNN
 F 1 "GND" V 9005 1322 50  0000 R CNN
 F 2 "" H 9000 1450 50  0001 C CNN
@@
 $EndComp
 $Comp
-L power:GND #PWR?
-U 1 1 636D2127
-P 9000 1750
-F 0 "#PWR?" H 9000 1500 50  0001 C CNN
-F 1 "GND" V 9005 1622 50  0000 R CNN
-F 2 "" H 9000 1750 50  0001 C CNN
-F 3 "" H 9000 1750 50  0001 C CNN
-	1    9000 1750
-	0    1    1    0
-$EndComp
-$Comp
-L power:GND #PWR?
-U 1 1 636D23FB
-P 9000 1950
-F 0 "#PWR?" H 9000 1700 50  0001 C CNN
-F 1 "GND" V 9005 1822 50  0000 R CNN
-F 2 "" H 9000 1950 50  0001 C CNN
-F 3 "" H 9000 1950 50  0001 C CNN
-	1    9000 1950
-	0    1    1    0
-$EndComp
-$Comp
-L power:GND #PWR?
+L power:GND #PWR0110
 U 1 1 636D26AD
 P 10000 1250
-F 0 "#PWR?" H 10000 1000 50  0001 C CNN
+F 0 "#PWR0110" H 10000 1000 50  0001 C CNN
 F 1 "GND" V 10005 1122 50  0000 R CNN
 F 2 "" H 10000 1250 50  0001 C CNN
@@
 $EndComp
 $Comp
-L power:GND #PWR?
+L power:GND #PWR0111
 U 1 1 636D2A90
 P 10000 1450
-F 0 "#PWR?" H 10000 1200 50  0001 C CNN
+F 0 "#PWR0111" H 10000 1200 50  0001 C CNN
 F 1 "GND" V 10005 1322 50  0000 R CNN
 F 2 "" H 10000 1450 50  0001 C CNN
@@
 $EndComp
 $Comp
-L power:GND #PWR?
+L power:GND #PWR0112
 U 1 1 636D2D3F
 P 10000 1750
-F 0 "#PWR?" H 10000 1500 50  0001 C CNN
+F 0 "#PWR0112" H 10000 1500 50  0001 C CNN
 F 1 "GND" V 10005 1622 50  0000 R CNN
 F 2 "" H 10000 1750 50  0001 C CNN
@@
 $EndComp
 $Comp
-L power:GND #PWR?
+L power:GND #PWR0113
 U 1 1 636D301A
 P 10000 1950
-F 0 "#PWR?" H 10000 1700 50  0001 C CNN
+F 0 "#PWR0113" H 10000 1700 50  0001 C CNN
 F 1 "GND" V 10005 1822 50  0000 R CNN
 F 2 "" H 10000 1950 50  0001 C CNN
@@
 	0    1    1    0
 $EndComp
+Wire Wire Line
+	4750 3300 5750 3300
+Wire Wire Line
+	5750 3300 5750 3500
+Connection ~ 5750 3300
+$Comp
+L Device:C C2
+U 1 1 63A9EAB0
+P 8250 3250
+F 0 "C2" H 8365 3296 50  0000 L CNN
+F 1 "0.1uF" H 8365 3205 50  0000 L CNN
+F 2 "Capacitor_THT:C_Axial_L3.8mm_D2.6mm_P12.50mm_Horizontal" H 8288 3100 50  0001 C CNN
+F 3 "~" H 8250 3250 50  0001 C CNN
+	1    8250 3250
+	1    0    0    -1
+$EndComp
+$Comp
+L Device:C C1
+U 1 1 63AA00B9
+P 7750 3250
+F 0 "C1" H 7865 3296 50  0000 L CNN
+F 1 "0.1uF" H 7865 3205 50  0000 L CNN
+F 2 "Capacitor_THT:C_Axial_L3.8mm_D2.6mm_P12.50mm_Horizontal" H 7788 3100 50  0001 C CNN
+F 3 "~" H 7750 3250 50  0001 C CNN
+	1    7750 3250
+	1    0    0    -1
+$EndComp
+$Comp
+L power:GND #PWR09
+U 1 1 63AA0DFD
+P 7750 3400
+F 0 "#PWR09" H 7750 3150 50  0001 C CNN
+F 1 "GND" H 7755 3227 50  0000 C CNN
+F 2 "" H 7750 3400 50  0001 C CNN
+F 3 "" H 7750 3400 50  0001 C CNN
+	1    7750 3400
+	1    0    0    -1
+$EndComp
+$Comp
+L power:GND #PWR010
+U 1 1 63AA15D4
+P 8250 3400
+F 0 "#PWR010" H 8250 3150 50  0001 C CNN
+F 1 "GND" H 8255 3227 50  0000 C CNN
+F 2 "" H 8250 3400 50  0001 C CNN
+F 3 "" H 8250 3400 50  0001 C CNN
+	1    8250 3400
+	1    0    0    -1
+$EndComp
+$Comp
+L power:VCC #PWR07
+U 1 1 63AA215C
+P 7750 3100
+F 0 "#PWR07" H 7750 2950 50  0001 C CNN
+F 1 "VCC" H 7765 3273 50  0000 C CNN
+F 2 "" H 7750 3100 50  0001 C CNN
+F 3 "" H 7750 3100 50  0001 C CNN
+	1    7750 3100
+	1    0    0    -1
+$EndComp
+$Comp
+L power:VCC #PWR08
+U 1 1 63AA2A09
+P 8250 3100
+F 0 "#PWR08" H 8250 2950 50  0001 C CNN
+F 1 "VCC" H 8265 3273 50  0000 C CNN
+F 2 "" H 8250 3100 50  0001 C CNN
+F 3 "" H 8250 3100 50  0001 C CNN
+	1    8250 3100
+	1    0    0    -1
+$EndComp
 $EndSCHEMATC

Commit message: fix CMP pcb
Other:
- note added: "DST(A)"
- note added: "SRC(B)"
- note added: "SRC(B) < DST(A)"
- note added: "SRC(B) > DST(A)"
- note added: "~SRC(B) == DST(A)"
Changed lines of the file:
@@
 	1    0    0    -1
 $EndComp
+Text Notes 1350 2825 0    50   ~ 0
+DST(A)
+Text Notes 1375 4125 0    50   ~ 0
+SRC(B)
+Text Notes 4875 3200 0    50   ~ 0
+SRC(B) < DST(A)
+Text Notes 4875 3100 0    50   ~ 0
+SRC(B) > DST(A)
+Text Notes 6550 3400 0    50   ~ 0
+~SRC(B) == DST(A)
 $EndSCHEMATC
