File: Toggle/Toggle.kicad_pcb (KiCad board)
At the start: 2 copper layers, 58.4 x 26.7 mm, 5 parts, among them J1 Conn_01x07_Male, J2 Conn_01x07_Male, U1 74LS08, U2 74LS86, U3 74LS175

Commit message: Polishing Toggle pcb
Parts:
- J1, J2: moved to B.Cu
- moved J2 11.4 mm to (61.0, 29.2), turned to 0 degrees
- moved J1 7.18 mm to (12.7, 14.0), turned to 180 degrees
- moved U3 5.68 mm to (48.3, 14.0)
- moved U1 5.68 mm to (33.0, 16.5)
- moved U2 5.68 mm to (17.8, 16.5)
Routing:
- net VCC: track 52.6 -> 39.5 mm
- net /M0: track 31.5 -> 39.3 mm, vias 0 -> 2
- net /Q2: track 36.2 -> 41.7 mm, vias 0 -> 2
- net /Q3: track 26.5 -> 31.7 mm, vias 0 -> 2
- net /Q0: track 37.2 -> 32.2 mm
- net /C: track 10.2 -> 6.13 mm
- net /Q1: track 29.6 -> 25.6 mm
- net GND: track 51.3 -> 48.9 mm
- net /Toggle: track 61.0 -> 63.3 mm, vias 0 -> 3
- net /D2: track 5.08 -> 6.13 mm
- net /~MR: track 37.1 -> 36.1 mm
- net /D0: track 6.13 -> 5.08 mm
- net /M2: track 48.5 -> 49.3 mm
- net /M3: track 27.5 -> 28.2 mm
- net /M1: vias 2 -> 0
Other:
- board size 58.4 x 26.7 mm -> 53.3 x 26.7 mm

Commit message: Polishing Toggle pcb
Parts:
- moved U1 1.91 mm to (33.0, 14.6)
- moved U2 1.91 mm to (17.8, 14.6)
- moved U3 1.91 mm to (48.3, 12.1)
- moved J2 0.64 mm to (61.0, 28.6)
- moved J1 0.63 mm to (12.7, 13.3)
Connections:
- J1 pad 2: Net-(J1-Pad2) -> /D0
- J1 pad 3: /D0 -> /D1
- J1 pad 4: /D1 -> Net-(J1-Pad4)
- J2 pad 4: /Q1 -> /Toggle
- J2 pad 5: /Q0 -> /Q1
- J2 pad 6: /Toggle -> /Q0
Routing:
- net /Toggle: track 63.3 -> 48.3 mm, vias 3 -> 2
- net VCC: track 39.5 -> 46.1 mm
- net Net-(U1-Pad8): track 24.4 -> 18.6 mm
- net /M3: track 28.2 -> 33.1 mm
- net /M2: track 49.3 -> 47.0 mm
- net /M0: track 39.3 -> 37.2 mm
- net /Q1: track 25.6 -> 23.6 mm
- net /Q3: track 31.7 -> 30.0 mm
- net /Q0: track 32.2 -> 30.5 mm
- net GND: track 48.9 -> 50.1 mm
- net /D2: track 6.13 -> 5.61 mm
- net /C: track 6.13 -> 5.61 mm
- net /~MR: track 36.1 -> 36.6 mm
- net /D1: track 13.8 -> 13.2 mm
- net /D0: track 5.08 -> 5.61 mm
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Other:
- board size 53.3 x 26.7 mm -> 53.3 x 24.1 mm
- board text added: "+5V"
- board text added: "08"
- board text added: "15.07.2023"
- board text added: "175"
- board text added: "74HCPU"
- board text added: "86"
- board text added: "C"
- board text added: "D0"
- board text added: "D1"
- board text added: "D2"
- board text added: "D3"
- board text added: "Gnd"
- board text added: "Q0"
- board text added: "Q1"
- board text added: "Q2"
- board text added: "Q3"
- board text added: "Tog"
- board text added: "Toggler"
- board text added: "Vcc"
- board text added: "~MR"
