File: Regs-v3/Regs-v3.kicad_pcb (KiCad board)
At the start: 2 copper layers, 149.9 x 99.1 mm, 41 parts, among them J1 Conn_01x09_Male, J10 Conn_01x09_Male, J11 Conn_01x03_Male, J12 Conn_01x01_Male, J13 Conn_01x01_Male, J14 Conn_01x01_Male, J15 Conn_01x01_Male, J16 Screw_Terminal_01x02, J2 Conn_01x09_Male, J3 Conn_01x09_Male, J4 Conn_01x09_Male, J5 Conn_01x09_Male, J6 Conn_01x09_Male, J7 Conn_01x09_Male, J8 Conn_01x09_Male, J9 Conn_01x09_Male, U1 REG_CNT, U10 REG_CNT, U11 74HC245, U12 74HC245, U13 74LS139, U14 74HC00, U15 MUX2-1, U2 REG_CNT, U3 REG_CNT, U4 REG_CNT, U5 REG_CNT, U6 REG_CNT, U7 REG_CNT, U8 REG_CNT, U9 REG_CNT

Commit message: Regs pcb in work
Parts:
- added J17: Conn_01x09_Male, Connector_PinHeader_2.54mm:PinHeader_1x09_P2.54mm_Vertical, F.Cu at (116.8, 109.2)
- added J18: Conn_01x09_Male, Connector_PinHeader_2.54mm:PinHeader_1x09_P2.54mm_Vertical, F.Cu at (83.8, 109.2)
- added R5: 10k, Resistor_SMD:R_0805_2012Metric_Pad1.20x1.40mm_HandSolder, B.Cu at (39.3, 105.1)
- added R6: 10k, Resistor_SMD:R_0805_2012Metric_Pad1.20x1.40mm_HandSolder, B.Cu at (121.6, 101.6)
- moved J16 89.0 mm to (109.2, 20.3), turned to 180 degrees
- moved U15 15.3 mm to (109.2, 102.9)
- moved J3 10.2 mm to (127.0, 78.7)
- moved J1 10.2 mm to (127.0, 91.4)
- moved J5 10.2 mm to (127.0, 66.0)
- moved J7 10.2 mm to (127.0, 53.3)
Connections:
- U15 pad 1: Net-(U15-Pad1) -> /L0
- U15 pad 16: Net-(U15-Pad16) -> /ALU_H7
- U15 pad 17: Net-(U15-Pad17) -> /H0
- U15 pad 18: Net-(U15-Pad18) -> /H1
- U15 pad 19: Net-(U15-Pad19) -> /H2
- U15 pad 2: Net-(U15-Pad2) -> /L1
- U15 pad 20: Net-(U15-Pad20) -> /H3
- U15 pad 21: Net-(U15-Pad21) -> /H4
- U15 pad 22: Net-(U15-Pad22) -> /H5
- U15 pad 23: Net-(U15-Pad23) -> /H6
- U15 pad 24: Net-(U15-Pad24) -> /H7
- U15 pad 25: Net-(U15-Pad25) -> /~MUL
- U15 pad 26: Net-(U15-Pad26) -> VCC
- U15 pad 27: Net-(U15-Pad27) -> GND
- U15 pad 28: Net-(U15-Pad28) -> GND
- U15 pad 3: Net-(U15-Pad3) -> /L2
- U15 pad 4: Net-(U15-Pad4) -> /L3
- U15 pad 5: Net-(U15-Pad5) -> /L4
- U15 pad 6: Net-(U15-Pad6) -> /L5
- U15 pad 7: Net-(U15-Pad7) -> /L6
- U15 pad 8: Net-(U15-Pad8) -> /L7
- U15 pad 9: Net-(U15-Pad9) -> /ALU_H0
Routing:
- net /H7: track 38.1 -> 82.6 mm, vias 0 -> 1
- net /H6: track 38.1 -> 80.8 mm, vias 0 -> 1
- net /H5: track 38.1 -> 79.0 mm, vias 0 -> 1
- net /H4: track 38.1 -> 77.2 mm, vias 0 -> 1
- net /H3: track 38.1 -> 75.0 mm
- net VCC: track 297.2 -> 265.5 mm
- net /H1: track 38.1 -> 68.4 mm
- net /H2: track 38.1 -> 68.0 mm
- net /H0: track 38.1 -> 68.0 mm
- net /L3: track 38.1 -> 54.0 mm
- net /L7: track 38.1 -> 54.0 mm
- net /L5: track 38.1 -> 54.0 mm
- net /L2: track 38.1 -> 54.0 mm
- net /L0: track 38.1 -> 54.0 mm
- net /L6: track 38.1 -> 54.0 mm
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
Commit message: Regs pcb is almost ready
Parts:
- added C1: 0.1uF, Capacitor_SMD:C_0805_2012Metric_Pad1.18x1.45mm_HandSolder, B.Cu at (138.4, 41.9)
- added C2: 0.1uF, Capacitor_SMD:C_0805_2012Metric_Pad1.18x1.45mm_HandSolder, B.Cu at (64.8, 41.9)
Routing:
- net GND: track 553.7 -> 800.6 mm, vias 16 -> 6
- net VCC: track 265.5 -> 402.4 mm, vias 6 -> 8
- net /~MUL: track 4.89 -> 113.2 mm
- net /H6: track 80.8 -> 82.9 mm
- net /H4: track 77.2 -> 79.4 mm
- net /H5: track 79.0 -> 81.2 mm
- net /H7: track 82.6 -> 84.2 mm
- net /H3: track 75.0 -> 75.9 mm
Other:
- board text added: "ALU High byte"
- board text added: "ALU Low byte"
- board text added: "MUX2:1"

Commit message: Polishing Regs
Parts:
- added C3: 0.1uF, Capacitor_SMD:C_0805_2012Metric_Pad1.18x1.45mm_HandSolder, B.Cu at (83.2, 40.6)
- added C4: 0.1uF, Capacitor_SMD:C_0805_2012Metric_Pad1.18x1.45mm_HandSolder, B.Cu at (111.4, 41.3)
- added Q1: IRLML5203, Package_TO_SOT_SMD:SOT-23, B.Cu at (113.3, 19.4)
- added R7: 10k, Resistor_SMD:R_0805_2012Metric_Pad1.20x1.40mm_HandSolder, B.Cu at (109.2, 33.3)
- moved J12 88.9 mm to (116.8, 33.0)
- moved R5 82.0 mm to (82.8, 35.6)
- moved J11 61.0 mm to (81.3, 48.3)
- moved U13 61.0 mm to (81.3, 45.7)
- moved J14 10.2 mm to (106.7, 35.6)
- moved J15 10.2 mm to (106.7, 48.3)
- moved U14 10.2 mm to (104.1, 45.7)
- moved R2 5.40 mm to (82.8, 33.0), turned to 180 degrees
Connections:
- J16 pad 1: VCC -> Net-(J16-Pad1)
- U14 pad 10: GND -> /~MUL
- U14 pad 9: GND -> /~MUL
- U15 pad 25: /~MUL -> Net-(U14-Pad8)
Routing:
- net Net-(U14-Pad8): track 0.00 -> 183.5 mm, vias 0 -> 1
- net /~MUL: track 113.2 -> 45.7 mm, vias 0 -> 1
- net /~Res: track 214.5 -> 272.5 mm, vias 2 -> 4
- net /~R0: track 187.7 -> 133.5 mm
- net Net-(U13-Pad10): track 66.7 -> 13.0 mm, vias 2 -> 1
- net Net-(U13-Pad9): track 74.3 -> 21.4 mm
- net /~R1: track 170.7 -> 118.9 mm
- net /~R3: track 142.4 -> 95.9 mm, vias 3 -> 4
- net /~R2: track 153.2 -> 108.8 mm, vias 3 -> 4
- net VCC: track 402.4 -> 385.5 mm
- net GND: track 800.6 -> 811.1 mm, vias 6 -> 4
- net /~L: track 109.2 -> 99.1 mm
- net /~H: track 73.7 -> 83.8 mm
- net Net-(U10-Pad20): track 83.8 -> 91.4 mm, vias 4 -> 3
- net Net-(J16-Pad1): track 0.00 -> 3.52 mm
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Other:
- board text added: "+5V"
- board text added: "I0"
- board text added: "I1"
- board text added: "I2"
- board text added: "I3"
- board text added: "I4"
- board text added: "I5"
- board text added: "I6"
- board text added: "I7"
- board text added: "O0"
- board text added: "O1"
- board text added: "O2"
- board text added: "O3"
- board text added: "O4"
- board text added: "O5"
- board text added: "O6"
- board text added: "O7"
- board text added: "~CS"
- board text added: "~Col"
- board text added: "~Row"
