File: MUX8x1-100x150-reverted/MUX8x1-v5.kicad_pcb (KiCad board)
At the start: 2 copper layers, 149.9 x 99.1 mm, 49 parts, among them J1 Conn_01x09_Male, J10 Conn_01x03_Male, J11 Conn_01x09_Male, J12 Conn_01x09_Male, J13 Conn_01x01_Male, J15 Conn_01x09_Male, J16 Conn_01x09_Male, J2 Conn_01x09_Male, J20 Conn_01x01_Male, J21 Conn_01x09_Male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

Commit message: MUX8:1 polishing
Parts:
- added Q1: IRLML5203, Package_TO_SOT_SMD:SOT-23, F.Cu at (165.1, 85.7)
Connections:
- J9 pad 1: VCC -> Net-(J9-Pad1)
Routing:
- net VCC: track 259.5 -> 250.7 mm
- net Net-(J9-Pad1): track 0.00 -> 7.77 mm
- net /H7: track 72.0 -> 76.8 mm
- net GND: track 520.8 -> 525.3 mm
Other:
- board text added: "+5V"
- board text added: "13.01.24"
- board text added: "74HCPU"
- board text added: "MUX 8:1"
- board text added: "S0"
- board text added: "S1"
- board text added: "S2"
- board text added: "~EH"
- board text added: "~EL"
- board text added: "~OE"
