File: RegCntLed/Reg.sch (KiCad schematic (older format))
At the start: 31 parts, among them J1 Conn_01x08_Male, J2 Conn_01x08_Male, J3 Conn_01x02_Male, J4 Conn_01x03_Male, J5 Conn_01x02_Male, J6 Conn_01x02_Male, J7 Conn_01x01_Male, U1 74LS193, U2 74HC245, U3 74LS27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

Commit message: RegLed: Add pull-ups, align LEDs
Parts:
- added R10, R11: 10k, Resistor_SMD:R_0805_2012Metric_Pad1.20x1.40mm_HandSolder, symbol Device:R
Connections:
- net Down: now also R10.1
- net Up: now also R11.1
- net VCC: now also R10.2, R11.2
Changed lines of the file:
@@
 	1    0    0    -1
 $EndComp
+$Comp
+L Device:R R10
+U 1 1 65A34615
+P 10150 5600
+F 0 "R10" V 10225 5550 50  0000 L CNN
+F 1 "10k" V 10150 5550 50  0000 L CNN
+F 2 "Resistor_SMD:R_0805_2012Metric_Pad1.20x1.40mm_HandSolder" V 10080 5600 50  0001 C CNN
+F 3 "~" H 10150 5600 50  0001 C CNN
+	1    10150 5600
+	0    -1   -1   0
+$EndComp
+$Comp
+L Device:R R11
+U 1 1 65A363AC
+P 10150 5800
+F 0 "R11" V 10225 5750 50  0000 L CNN
+F 1 "10k" V 10150 5750 50  0000 L CNN
+F 2 "Resistor_SMD:R_0805_2012Metric_Pad1.20x1.40mm_HandSolder" V 10080 5800 50  0001 C CNN
+F 3 "~" H 10150 5800 50  0001 C CNN
+	1    10150 5800
+	0    -1   -1   0
+$EndComp
+Wire Wire Line
+	9700 5650 9950 5650
+Wire Wire Line
+	9950 5650 9950 5600
+Wire Wire Line
+	9950 5600 10000 5600
+Wire Wire Line
+	9700 5750 9950 5750
+Wire Wire Line
+	9950 5750 9950 5800
+Wire Wire Line
+	9950 5800 10000 5800
+$Comp
+L power:VCC #PWR0102
+U 1 1 65A3E22D
+P 10300 5450
+F 0 "#PWR0102" H 10300 5300 50  0001 C CNN
+F 1 "VCC" H 10315 5623 50  0000 C CNN
+F 2 "" H 10300 5450 50  0001 C CNN
+F 3 "" H 10300 5450 50  0001 C CNN
+	1    10300 5450
+	1    0    0    -1
+$EndComp
+Wire Wire Line
+	10300 5450 10300 5600
+Wire Wire Line
+	10300 5600 10300 5800
+Connection ~ 10300 5600
 $EndSCHEMATC

Commit message: Add unconditional load input
Parts:
- added J10, J8, J9: Conn_01x01_Male, Connector_PinHeader_2.54mm:PinHeader_1x01_P2.54mm_Horizontal, symbol Connector:Conn_01x01_Male
- added R12, R13: 10k, Resistor_SMD:R_0805_2012Metric_Pad1.20x1.40mm_HandSolder, symbol Device:R
Connections:
- net GND: now also R12.1; no longer U3.13
- net VCC: now also R13.1
- net at U3.10, U3.6, U3.9: no longer U3.11
- net at U3.12: now also J10.1 (Pin_1)
- new net MLOAD: J8.1 (Pin_1), R12.2, U3.11
- new net ~MLOAD: J9.1 (Pin_1), R13.2, U3.13
- no-connect marks 1 -> 0
Other:
- note added: "Unconditional\nload"
- moved on the sheet: U3A
Changed lines of the file:
@@
 L 74xx:74LS27 U3
 U 1 1 636F573A
-P 2050 4850
-F 0 "U3" H 2050 5175 50  0000 C CNN
-F 1 "74LS27" H 2050 5084 50  0000 C CNN
-F 2 "Package_SO:SO-14_3.9x8.65mm_P1.27mm" H 2050 4850 50  0001 C CNN
-F 3 "http://www.ti.com/lit/gpn/sn74LS27" H 2050 4850 50  0001 C CNN
-	1    2050 4850
+P 1650 4150
+F 0 "U3" H 1650 4475 50  0000 C CNN
+F 1 "74LS27" H 1650 4384 50  0000 C CNN
+F 2 "Package_SO:SO-14_3.9x8.65mm_P1.27mm" H 1650 4150 50  0001 C CNN
+F 3 "http://www.ti.com/lit/gpn/sn74LS27" H 1650 4150 50  0001 C CNN
+	1    1650 4150
 	1    0    0    -1
 $EndComp
@@
 $EndComp
 Wire Wire Line
-	1750 4750 1750 4850
-Connection ~ 1750 4850
-Wire Wire Line
-	1750 4850 1750 4950
+	1350 4050 1350 4150
 Wire Wire Line
 	2400 2525 2400 2625
 Connection ~ 2400 2625
-Wire Wire Line
-	2400 2625 2400 2725
 Wire Wire Line
 	2275 2625 2400 2625
@@
 Text Label 8275 5750 0    50   ~ 0
 DownOut
-NoConn ~ 2350 4850
 $Comp
 L power:GND #PWR024
 U 1 1 64AF5786
-P 1750 4850
-F 0 "#PWR024" H 1750 4600 50  0001 C CNN
-F 1 "GND" V 1755 4722 50  0000 R CNN
-F 2 "" H 1750 4850 50  0001 C CNN
-F 3 "" H 1750 4850 50  0001 C CNN
-	1    1750 4850
+P 1350 4050
+F 0 "#PWR024" H 1350 3800 50  0001 C CNN
+F 1 "GND" V 1355 3922 50  0000 R CNN
+F 2 "" H 1350 4050 50  0001 C CNN
+F 3 "" H 1350 4050 50  0001 C CNN
+	1    1350 4050
 	0    1    1    0
 $EndComp
@@
 	10300 5600 10300 5800
 Connection ~ 10300 5600
+$Comp
+L Connector:Conn_01x01_Male J8
+U 1 1 65AD21B9
+P 2200 3175
+F 0 "J8" H 2200 3100 50  0000 C CNN
+F 1 "Conn_01x01_Male" H 1800 3175 50  0000 C CNN
+F 2 "Connector_PinHeader_2.54mm:PinHeader_1x01_P2.54mm_Horizontal" H 2200 3175 50  0001 C CNN
+F 3 "~" H 2200 3175 50  0001 C CNN
+	1    2200 3175
+	1    0    0    -1
+$EndComp
+Wire Wire Line
+	2400 2725 2400 3175
+$Comp
+L Device:R R12
+U 1 1 65AD4FBF
+P 2400 3325
+F 0 "R12" V 2300 3250 50  0000 C CNN
+F 1 "10k" V 2400 3325 50  0000 C CNN
+F 2 "Resistor_SMD:R_0805_2012Metric_Pad1.20x1.40mm_HandSolder" V 2330 3325 50  0001 C CNN
+F 3 "~" H 2400 3325 50  0001 C CNN
+	1    2400 3325
+	-1   0    0    1
+$EndComp
+Connection ~ 2400 3175
+$Comp
+L power:GND #PWR028
+U 1 1 65AD5DA6
+P 2400 3475
+F 0 "#PWR028" H 2400 3225 50  0001 C CNN
+F 1 "GND" H 2550 3400 50  0000 C CNN
+F 2 "" H 2400 3475 50  0001 C CNN
+F 3 "" H 2400 3475 50  0001 C CNN
+	1    2400 3475
+	1    0    0    -1
+$EndComp
+Text Label 2400 2925 0    50   ~ 0
+MLOAD
+Text Notes 2425 3100 0    50   ~ 0
+Unconditional\nload
+Connection ~ 1350 4050
+$Comp
+L Connector:Conn_01x01_Male J9
+U 1 1 65AF4013
+P 1150 4550
+F 0 "J9" H 1125 4500 50  0000 C CNN
+F 1 "Conn_01x01_Male" H 1575 4500 50  0000 C CNN
+F 2 "Connector_PinHeader_2.54mm:PinHeader_1x01_P2.54mm_Horizontal" H 1150 4550 50  0001 C CNN
+F 3 "~" H 1150 4550 50  0001 C CNN
+	1    1150 4550
+	1    0    0    -1
+$EndComp
+$Comp
+L Device:R R13
+U 1 1 65AF401A
+P 1200 4250
+F 0 "R13" V 1100 4175 50  0000 C CNN
+F 1 "10k" V 1200 4250 50  0000 C CNN
+F 2 "Resistor_SMD:R_0805_2012Metric_Pad1.20x1.40mm_HandSolder" V 1130 4250 50  0001 C CNN
+F 3 "~" H 1200 4250 50  0001 C CNN
+	1    1200 4250
+	0    -1   -1   0
+$EndComp
+$Comp
+L Connector:Conn_01x01_Male J10
+U 1 1 65AF9C4B
+P 2150 4150
+F 0 "J10" H 2200 4225 50  0000 C CNN
+F 1 "Conn_01x01_Male" H 2100 4100 50  0000 C CNN
+F 2 "Connector_PinHeader_2.54mm:PinHeader_1x01_P2.54mm_Horizontal" H 2150 4150 50  0001 C CNN
+F 3 "~" H 2150 4150 50  0001 C CNN
+	1    2150 4150
+	-1   0    0    -1
+$EndComp
+$Comp
+L power:VCC #PWR029
+U 1 1 65B09055
+P 1050 4250
+F 0 "#PWR029" H 1050 4100 50  0001 C CNN
+F 1 "VCC" V 1065 4377 50  0000 L CNN
+F 2 "" H 1050 4250 50  0001 C CNN
+F 3 "" H 1050 4250 50  0001 C CNN
+	1    1050 4250
+	0    -1   -1   0
+$EndComp
+Wire Wire Line
+	1350 4250 1350 4550
+Connection ~ 1350 4250
+Text Label 1350 4550 0    50   ~ 0
+~MLOAD
 $EndSCHEMATC
