File: Regs-v4/Regs-v4.kicad_pcb (KiCad board)
At the start: 2 copper layers, 149.9 x 99.1 mm, 51 parts, among them J1 Conn_01x09_Male, J11 Conn_01x03_Male, J12 Conn_01x01_Male, J13 Conn_01x01_Male, J14 Conn_01x01_Male, J15 Conn_01x01_Male, J16 Screw_Terminal_01x02, J17 Conn_01x09_Male, J18 Conn_01x09_Male, J19 Conn_01x01_Male, J2 Conn_01x09_Male, J20 Conn_01x01_Male, J3 Conn_01x09_Male, J4 Conn_01x09_Male, J5 Conn_01x09_Male, J6 Conn_01x09_Male, J7 Conn_01x09_Male, J8 Conn_01x09_Male, Q1 IRLML5203, U1 REG_CNT, U10 REG_CNT, U11 REG_CNT, U12 REG_CNT, U13 74LS139, U14 74HC00, U15 MUX2-1, U16 REG_CNT, U17 REG_CNT, U18 REG_CNT, U19 REG_CNT, U2 REG_CNT, U3 REG_CNT, U4 REG_CNT, U5 REG_CNT, U6 REG_CNT, U7 REG_CNT, U8 REG_CNT, U9 REG_CNT

Commit message: Regs v4: is ready
Parts:
- moved J20 104.7 mm to (124.5, 104.1)
- moved J19 103.9 mm to (120.7, 104.1)
- moved R7 41.7 mm to (81.3, 18.4), turned to 0 degrees
- moved J14 39.8 mm to (78.1, 18.4)
- moved C2 36.4 mm to (49.5, 40.0), turned to 180 degrees
- moved R5 36.3 mm to (36.2, 22.9), turned to 270 degrees
- moved J12 36.1 mm to (50.2, 17.8)
- moved J11 30.5 mm to (28.6, 30.5)
- moved J15 25.5 mm to (55.2, 25.4)
- moved C1 9.12 mm to (123.2, 29.2), turned to 180 degrees
- moved U14 5.08 mm to (58.4, 25.4)
- moved C3 3.82 mm to (28.6, 22.9), turned to 270 degrees
- moved U13 2.69 mm to (28.6, 27.3)
- moved J13 2.54 mm to (116.8, 104.1)
- moved C4 2.14 mm to (58.4, 21.0), turned to 270 degrees
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Routing:
- net Net-(U14-Pad8): track 3.81 -> 165.6 mm
- net GND: track 411.9 -> 562.1 mm, vias 4 -> 8
- net /~R0: track 91.4 -> 201.9 mm, vias 0 -> 1
- net VCC: track 188.5 -> 293.7 mm, vias 0 -> 3
- net /~L: track 59.7 -> 161.4 mm, vias 0 -> 2
- net /~R1: track 91.4 -> 180.1 mm, vias 0 -> 1
- net /~R2: track 91.4 -> 163.4 mm, vias 0 -> 1
- net /~R3: track 91.4 -> 140.2 mm, vias 0 -> 2
- net /~H: track 59.7 -> 90.5 mm
- net /~Bank0: track 282.5 -> 311.4 mm, vias 16 -> 17
- net /~Bank1: track 211.9 -> 231.2 mm, vias 2 -> 3
- net /DST[0]: track 12.5 -> 27.8 mm
- net /~Res: track 206.9 -> 216.2 mm
- net Net-(U13-Pad10): track 11.9 -> 18.8 mm
- net Net-(U13-Pad9): track 20.3 -> 25.3 mm
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
Commit message: Regs v4: polishing
Routing:
- net /~Bank0: track 311.4 -> 296.2 mm
Other:
- board text added: "05.02.24"
- board text added: "SP"
- board text added: "Z"
- board text removed: "04.02.24"

Commit message: Regs v4: polishing
Parts:
- moved R7 1.67 mm to (82.8, 17.8)
Connections:
- U14 pad 10: /~MUL -> /~Bank0
- U14 pad 11: /~Bank1 -> Net-(U14-Pad11)
- U14 pad 12: /~Bank0 -> /~MUL
- U14 pad 13: /~Bank0 -> /~MUL
- U14 pad 8: Net-(U14-Pad8) -> /~Bank1
- U14 pad 9: /~MUL -> /~Bank0
- U15 pad 25: Net-(U14-Pad8) -> Net-(U14-Pad11)
Routing:
- net Net-(U14-Pad8): track 165.6 -> 0.00 mm
- net Net-(U14-Pad11): track 0.00 -> 156.5 mm, vias 0 -> 1
- net /~MUL: track 45.0 -> 34.7 mm
- net VCC: track 293.7 -> 302.0 mm, vias 3 -> 4
- net /~Bank0: track 296.2 -> 290.4 mm, vias 17 -> 13
- net /~R2: track 163.4 -> 158.3 mm, vias 1 -> 3
- net /~Res: track 216.2 -> 211.1 mm, vias 0 -> 2
- net /~Bank1: track 231.2 -> 227.0 mm, vias 3 -> 4
- net GND: track 562.1 -> 566.1 mm, vias 8 -> 9
- net /~R1: track 180.1 -> 177.5 mm, vias 1 -> 3
- net /~R0: track 201.9 -> 199.3 mm, vias 1 -> 3
- net /H3: track 96.8 -> 97.5 mm, vias 1 -> 2
- net /H6: track 106.2 -> 106.9 mm
- net Net-(U13-Pad10): track 18.8 -> 19.4 mm
- net /H7: track 108.8 -> 108.9 mm, vias 2 -> 0
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Other:
- board text added: "24.02.24"
- board text removed: "05.02.24"
