File: Regs-v4/Regs-v4.sch (KiCad schematic (older format))
At the start: 51 parts, among them J1 Conn_01x09_Male, J11 Conn_01x03_Male, J12 Conn_01x01_Male, J13 Conn_01x01_Male, J14 Conn_01x01_Male, J15 Conn_01x01_Male, J16 Screw_Terminal_01x02, J17 Conn_01x09_Male, J18 Conn_01x09_Male, J19 Conn_01x01_Male, J2 Conn_01x09_Male, J20 Conn_01x01_Male, J3 Conn_01x09_Male, J4 Conn_01x09_Male, J5 Conn_01x09_Male, J6 Conn_01x09_Male, J7 Conn_01x09_Male, J8 Conn_01x09_Male, Q1 IRLML5203, U1 REG_CNT, U10 REG_CNT, U11 REG_CNT, U12 REG_CNT, U13 74LS139, U14 74HC00, U15 MUX2-1, U16 REG_CNT, U17 REG_CNT, U18 REG_CNT, U19 REG_CNT, U2 REG_CNT, U3 REG_CNT, U4 REG_CNT, U5 REG_CNT, U6 REG_CNT, U7 REG_CNT, U8 REG_CNT, U9 REG_CNT

Commit message: Regs v4: polishing
Connections:
- net ~Bank0: now also U14.10, U14.9; no longer U14.12, U14.13
- net ~Bank1: now also U14.8; no longer U14.11
- net ~MUL: now also U14.12, U14.13; no longer U14.10, U14.9
- net at U15.25 (S): now also U14.11; no longer U14.8
Other:
- moved on the sheet: U14C, U14D
Changed lines of the file:
@@
 L 74xx:74HC00 U14
 U 3 1 659BB8BC
-P 3200 10450
-F 0 "U14" H 3200 10775 50  0000 C CNN
-F 1 "74HC00" H 3200 10684 50  0000 C CNN
-F 2 "Package_DIP:DIP-14_W7.62mm_Socket" H 3200 10450 50  0001 C CNN
-F 3 "http://www.ti.com/lit/gpn/sn74hc00" H 3200 10450 50  0001 C CNN
-	3    3200 10450
+P 10550 6850
+F 0 "U14" H 10550 7175 50  0000 C CNN
+F 1 "74HC00" H 10550 7084 50  0000 C CNN
+F 2 "Package_DIP:DIP-14_W7.62mm_Socket" H 10550 6850 50  0001 C CNN
+F 3 "http://www.ti.com/lit/gpn/sn74hc00" H 10550 6850 50  0001 C CNN
+	3    10550 6850
 	1    0    0    -1
 $EndComp
@@
 L 74xx:74HC00 U14
 U 4 1 659BD281
-P 10550 6850
-F 0 "U14" H 10500 7050 50  0000 C CNN
-F 1 "74HC00" H 10350 6650 50  0000 C CNN
-F 2 "Package_DIP:DIP-14_W7.62mm_Socket" H 10550 6850 50  0001 C CNN
-F 3 "http://www.ti.com/lit/gpn/sn74hc00" H 10550 6850 50  0001 C CNN
-	4    10550 6850
+P 3200 10450
+F 0 "U14" H 3150 10650 50  0000 C CNN
+F 1 "74HC00" H 3000 10250 50  0000 C CNN
+F 2 "Package_DIP:DIP-14_W7.62mm_Socket" H 3200 10450 50  0001 C CNN
+F 3 "http://www.ti.com/lit/gpn/sn74hc00" H 3200 10450 50  0001 C CNN
+	4    3200 10450
 	1    0    0    1
 $EndComp
