File: RegLed273/Reg.kicad_pcb (KiCad board)
At the start: 2 copper layers, 73.3 x 39.4 mm, 26 parts, among them J1 Conn_01x08_Male, J2 Conn_01x08_Male, J3 Conn_01x02_Male, J4 Conn_01x03_Male, J5 Conn_01x01_Male, U1 74HC273, U2 74HC245, U3 74LS27

Commit message: Polishing Reg 273
Connections:
- U1 pad 1: /Res -> Net-(U1-Pad1)
- U3 pad 1: GND -> /Res
- U3 pad 12: Net-(U3-Pad12) -> Net-(U1-Pad1)
- U3 pad 13: GND -> /Res
- U3 pad 2: GND -> /Res
Routing:
- net Net-(U1-Pad1): track 0.00 -> 84.6 mm
- net /Res: track 37.4 -> 57.5 mm
- net GND: track 129.8 -> 128.1 mm
- net /L0: track 45.3 -> 44.0 mm
- net VCC: track 96.8 -> 95.7 mm
Other:
- board text added: "IN"
- board text added: "OUT"
- board text added: "REG 273"
