File: !Perif/Kbd/Kbd.kicad_pcb (KiCad board)
At the start: 2 copper layers, 149.9 x 99.1 mm, 36 parts, among them SW1 SW_Push, SW10 SW_Push, SW11 SW_Push, SW12 SW_Push, SW13 SW_Push, SW14 SW_Push, SW15 SW_Push, SW16 SW_Push, SW17 SW_Push, SW18 SW_Push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

Commit message: Playing with keyboard
Parts:
- moved SW12 10.2 mm to (108.0, 100.3)
- moved SW15 10.2 mm to (123.2, 100.3)
- moved SW18 10.2 mm to (138.4, 100.3)
- moved SW21 10.2 mm to (153.7, 100.3)
- moved SW24 10.2 mm to (168.9, 100.3)
- moved SW27 10.2 mm to (184.2, 100.3)
- moved SW3 10.2 mm to (62.2, 100.3)
- moved SW30 10.2 mm to (199.4, 100.3)
- moved SW6 10.2 mm to (77.5, 100.3)
- moved SW9 10.2 mm to (92.7, 100.3)
- moved SW20 5.08 mm to (148.6, 81.3)
- moved SW23 5.08 mm to (163.8, 81.3)
- moved SW29 5.08 mm to (194.3, 81.3)
- moved SW11 5.08 mm to (102.9, 81.3)
- moved SW14 5.08 mm to (118.1, 81.3)
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Other:
- board text added: "A"
- board text added: "B"
- board text added: "C"
- board text added: "D"
- board text added: "F"
- board text added: "G"
- board text added: "H"
- board text added: "J"
- board text added: "K"
- board text added: "L"
- board text added: "M"
- board text added: "N"
- board text added: "S"
- board text added: "V"
- board text added: "X"
- board text added: "Z"

Commit message: Kbd in work
Parts:
- moved SW20 5.68 mm to (143.5, 78.7)
- moved SW23 5.68 mm to (158.8, 78.7)
- moved SW29 5.68 mm to (189.2, 78.7)
- moved SW10 5.68 mm to (92.7, 59.7)
- moved SW16 5.68 mm to (123.2, 59.7)
- moved SW22 5.68 mm to (153.7, 59.7)
- moved SW25 5.68 mm to (168.9, 59.7)
- moved SW18 5.68 mm to (133.3, 97.8)
- moved SW27 5.68 mm to (179.1, 97.8)
- moved SW4 5.68 mm to (62.2, 59.7)
- moved SW11 5.68 mm to (97.8, 78.7)
- moved SW14 5.68 mm to (113.0, 78.7)
- moved SW2 5.68 mm to (52.1, 78.7)
- moved SW5 5.68 mm to (67.3, 78.7)
- moved SW8 5.68 mm to (82.5, 78.7)
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Other:
- board size 149.9 x 99.1 mm -> 160 x 99.1 mm
- board text added: ";"
- board text added: "<"
- board text added: ">"
- board text added: "?"
