File: !REGS/Regs-v5/Regs-v5.sch (KiCad schematic (older format))
At the start: 51 parts, among them J1 Conn_01x09_Male, J11 Conn_01x03_Male, J12 Conn_01x01_Male, J13 Conn_01x01_Male, J14 Conn_01x01_Male, J15 Conn_01x01_Male, J16 Screw_Terminal_01x02, J17 Conn_01x09_Male, J18 Conn_01x09_Male, J19 Conn_01x01_Male, J2 Conn_01x09_Male, J20 Conn_01x01_Male, J3 Conn_01x09_Male, J4 Conn_01x09_Male, J5 Conn_01x09_Male, J6 Conn_01x09_Male, J7 Conn_01x09_Male, J8 Conn_01x09_Male, Q1 IRLML5203, U1 REG_CNT, U10 REG_CNT, U11 REG_CNT, U12 REG_CNT, U13 74LS139, U14 74HC00, U15 MUX2-1, U16 REG_CNT, U17 REG_CNT, U18 REG_CNT, U19 REG_CNT, U2 REG_CNT, U3 REG_CNT, U4 REG_CNT, U5 REG_CNT, U6 REG_CNT, U7 REG_CNT, U8 REG_CNT, U9 REG_CNT

Commit message: Regs v5 in work
Connections:
- net ALU_H0: now also U15.16 (B7); no longer U15.9 (B0)
- net ALU_H7: now also U15.9 (B0); no longer U15.16 (B7)
- net H0: now also U15.24 (O7); no longer U15.17 (O0)
- net H1: now also U15.23 (O6); no longer U15.18 (O1)
- net H2: now also U15.22 (O5); no longer U15.19 (O2)
- net H3: now also U15.21 (O4); no longer U15.20 (O3)
- net H4: now also U15.20 (O3); no longer U15.21 (O4)
- net H5: now also U15.19 (O2); no longer U15.22 (O5)
- net H6: now also U15.18 (O1); no longer U15.23 (O6)
- net H7: now also U15.17 (O0); no longer U15.24 (O7)
- net L0: now also U15.8 (A7); no longer U15.1 (A0)
- net L1: now also U15.7 (A6); no longer U15.2 (A1)
- net L2: now also U15.6 (A5); no longer U15.3 (A2)
- net L3: now also U15.5 (A4); no longer U15.4 (A3)
- net L4: now also U15.4 (A3); no longer U15.5 (A4)
- net L5: now also U15.3 (A2); no longer U15.6 (A5)
- net L6: now also U15.2 (A1); no longer U15.7 (A6)
- net L7: now also U15.1 (A0); no longer U15.8 (A7)
- net at U15.10 (B1): now also J18.8 (Pin_8); no longer J18.3 (Pin_3)
- net at U15.11 (B2): now also J18.7 (Pin_7); no longer J18.4 (Pin_4)
- net at U15.12 (B3): now also J18.6 (Pin_6); no longer J18.5 (Pin_5)
- net at U15.13 (B4): now also J18.5 (Pin_5); no longer J18.6 (Pin_6)
- net at U15.14 (B5): now also J18.4 (Pin_4); no longer J18.7 (Pin_7)
- net at U15.15 (B6): now also J18.3 (Pin_3); no longer J18.8 (Pin_8)
Other:
- moved on the sheet: J17, J18
Changed lines of the file:
@@
 L Connector:Conn_01x09_Male J17
 U 1 1 65A046FB
-P 3550 8050
-F 0 "J17" H 3625 8525 50  0000 R CNN
-F 1 "Conn_01x09_Male" V 3475 8350 50  0000 R CNN
-F 2 "Connector_PinHeader_2.54mm:PinHeader_1x09_P2.54mm_Vertical" H 3550 8050 50  0001 C CNN
-F 3 "~" H 3550 8050 50  0001 C CNN
-	1    3550 8050
-	1    0    0    -1
+P 3550 8150
+F 0 "J17" H 3625 8625 50  0000 R CNN
+F 1 "Conn_01x09_Male" V 3475 8450 50  0000 R CNN
+F 2 "Connector_PinHeader_2.54mm:PinHeader_1x09_P2.54mm_Vertical" H 3550 8150 50  0001 C CNN
+F 3 "~" H 3550 8150 50  0001 C CNN
+	1    3550 8150
+	1    0    0    1
 $EndComp
 Wire Wire Line
@@
 Wire Wire Line
 	3875 10250 4000 10250
+Text Label 3875 10250 0    50   ~ 0
+H0
+Text Label 3875 10150 0    50   ~ 0
+H1
+Text Label 3875 10050 0    50   ~ 0
+H2
+Text Label 3875 9950 0    50   ~ 0
+H3
+Text Label 3875 9850 0    50   ~ 0
+H4
+Text Label 3875 9750 0    50   ~ 0
+H5
+Text Label 3875 9650 0    50   ~ 0
+H6
 Text Label 3875 9550 0    50   ~ 0
-H0
-Text Label 3875 9650 0    50   ~ 0
-H1
-Text Label 3875 9750 0    50   ~ 0
-H2
-Text Label 3875 9850 0    50   ~ 0
-H3
-Text Label 3875 9950 0    50   ~ 0
-H4
-Text Label 3875 10050 0    50   ~ 0
-H5
-Text Label 3875 10150 0    50   ~ 0
-H6
-Text Label 3875 10250 0    50   ~ 0
 H7
 Wire Wire Line
@@
 L power:GND #PWR030
 U 1 1 65B84CC6
-P 3750 7650
-F 0 "#PWR030" H 3750 7400 50  0001 C CNN
-F 1 "GND" H 3725 7525 50  0000 C CNN
-F 2 "" H 3750 7650 50  0001 C CNN
-F 3 "" H 3750 7650 50  0001 C CNN
-	1    3750 7650
-	-1   0    0    1
+P 3750 8550
+F 0 "#PWR030" H 3750 8300 50  0001 C CNN
+F 1 "GND" V 3775 8375 50  0000 C CNN
+F 2 "" H 3750 8550 50  0001 C CNN
+F 3 "" H 3750 8550 50  0001 C CNN
+	1    3750 8550
+	0    -1   -1   0
 $EndComp
-Text Label 3825 7750 0    50   ~ 0
+Text Label 3800 8450 0    50   ~ 0
 L0
-Text Label 3825 7850 0    50   ~ 0
+Text Label 3800 8350 0    50   ~ 0
 L1
-Text Label 3825 7950 0    50   ~ 0
+Text Label 3800 8250 0    50   ~ 0
 L2
-Text Label 3825 8050 0    50   ~ 0
+Text Label 3800 8150 0    50   ~ 0
 L3
-Text Label 3825 8150 0    50   ~ 0
+Text Label 3800 8050 0    50   ~ 0
 L4
-Text Label 3825 8250 0    50   ~ 0
+Text Label 3800 7950 0    50   ~ 0
 L5
-Text Label 3825 8350 0    50   ~ 0
+Text Label 3800 7850 0    50   ~ 0
 L6
-Text Label 3825 8450 0    50   ~ 0
+Text Label 3800 7750 0    50   ~ 0
 L7
 Text Label 2650 10450 0    50   ~ 0
@@
 L Connector:Conn_01x09_Male J18
 U 1 1 65C3B36A
-P 3550 8950
-F 0 "J18" H 3525 9350 50  0000 R CNN
-F 1 "Conn_01x09_Male" V 3500 9275 50  0000 R CNN
-F 2 "Connector_PinHeader_2.54mm:PinHeader_1x09_P2.54mm_Vertical" H 3550 8950 50  0001 C CNN
-F 3 "~" H 3550 8950 50  0001 C CNN
-	1    3550 8950
-	1    0    0    -1
+P 3550 9050
+F 0 "J18" H 3525 9450 50  0000 R CNN
+F 1 "Conn_01x09_Male" V 3500 9375 50  0000 R CNN
+F 2 "Connector_PinHeader_2.54mm:PinHeader_1x09_P2.54mm_Vertical" H 3550 9050 50  0001 C CNN
+F 3 "~" H 3550 9050 50  0001 C CNN
+	1    3550 9050
+	1    0    0    1
 $EndComp
 $Comp
 L power:GND #PWR031
 U 1 1 65C40119
-P 3750 8550
-F 0 "#PWR031" H 3750 8300 50  0001 C CNN
-F 1 "GND" V 3750 8350 50  0000 C CNN
-F 2 "" H 3750 8550 50  0001 C CNN
-F 3 "" H 3750 8550 50  0001 C CNN
-	1    3750 8550
-	0    -1   -1   0
+P 3750 9450
+F 0 "#PWR031" H 3750 9200 50  0001 C CNN
+F 1 "GND" V 3750 9250 50  0000 C CNN
+F 2 "" H 3750 9450 50  0001 C CNN
+F 3 "" H 3750 9450 50  0001 C CNN
+	1    3750 9450
+	1    0    0    -1
 $EndComp
 Wire Wire Line
@@
 Wire Wire Line
 	3750 9350 4000 9350
-Text Notes 2400 8125 0    50   ~ 0
+Text Notes 2400 8175 0    50   ~ 0
 To ALU low byte output
-Text Notes 2400 8925 0    50   ~ 0
+Text Notes 2375 9075 0    50   ~ 0
 To ALU high byte output
+Text Label 3750 8650 0    50   ~ 0
+ALU_H7
 Text Label 3750 9350 0    50   ~ 0
-ALU_H7
-Text Label 3750 8650 0    50   ~ 0
 ALU_H0
 $Comp
