File: MUX8x1-100x150-r2/MUX8x1-100x150-r2.kicad_pcb (KiCad board)
At the start: 2 copper layers, 149.9 x 99.1 mm, 49 parts, among them J1 Conn_01x09_Male, J10 Conn_01x03_Male, J11 Conn_01x09_Male, J12 Conn_01x09_Male, J13 Conn_01x01_Male, J15 Conn_01x09_Male, J16 Conn_01x09_Male, J2 Conn_01x09_Male, J20 Conn_01x01_Male, J21 Conn_01x09_Male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

Commit message: MUX 8:1 r2 in work
Parts:
- moved J13 26.5 mm to (180.3, 73.7)
- moved R7 26.4 mm to (176.3, 73.7), turned to 180 degrees
Other:
- board size 149.9 x 99.1 mm -> 160 x 99.1 mm
- board text added: "15.12.2024"
- board text removed: "15.09.2024"
