File: !REGS/RegCntLedDualPort/Reg.sch (KiCad schematic (older format))
At the start: 42 parts, among them J1 Conn_01x08_Male, J10 Conn_01x01_Male, J11 Conn_01x08_Male, J2 Conn_01x08_Male, J3 Conn_01x02_Male, J4 Conn_01x03_Male, J5 Conn_01x02_Male, J6 Conn_01x02_Male, J7 Conn_01x01_Male, J8 Conn_01x01_Male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

Commit message: Polishing RegCntDualPort
Parts:
- R1: footprint Resistor_THT:R_Axial_DIN0309_L9.0mm_D3.2mm_P15.24mm_Horizontal -> Resistor_SMD:R_0805_2012Metric_Pad1.20x1.40mm_HandSolder
Changed lines of the file:
@@
 F 0 "R1" V 5100 2175 50  0000 C CNN
 F 1 "10k" V 5200 2250 50  0000 C CNN
-F 2 "Resistor_THT:R_Axial_DIN0309_L9.0mm_D3.2mm_P15.24mm_Horizontal" V 5130 2250 50  0001 C CNN
+F 2 "Resistor_SMD:R_0805_2012Metric_Pad1.20x1.40mm_HandSolder" V 5130 2250 50  0001 C CNN
 F 3 "~" H 5200 2250 50  0001 C CNN
 	1    5200 2250
