File: hard/!REGS/RegLed273/Reg.kicad_pcb (KiCad board)
At the start: 2 copper layers, 73.3 x 39.4 mm, 26 parts, among them J1 Conn_01x08_Male, J2 Conn_01x08_Male, J3 Conn_01x02_Male, J4 Conn_01x03_Male, J5 Conn_01x01_Male, U1 74HC273, U2 74HC245, U3 74LS27

Commit message: Polishing Reg273
Parts:
- moved C2 2.54 mm to (109.2, 47.0)
- moved U1 2.54 mm to (53.3, 45.7)
- moved U2 2.54 mm to (83.8, 45.7)
- moved C1 2.54 mm to (78.7, 47.0)
- moved U3 1.27 mm to (116.2, 41.3)
Routing:
- net /L1: track 42.7 -> 36.6 mm
- net /L2: track 53.5 -> 48.4 mm
- net /L0: track 44.0 -> 38.9 mm
- net /L3: track 49.1 -> 45.1 mm
- net /L4: track 54.2 -> 50.6 mm
- net /L5: track 66.6 -> 63.4 mm
- net /L6: track 72.4 -> 69.5 mm
- net GND: track 128.1 -> 125.3 mm
- net /L7: track 70.7 -> 68.2 mm
- net /~CS: track 49.3 -> 51.3 mm
- net VCC: track 95.7 -> 94.4 mm
- net /Q7: track 7.62 -> 8.67 mm
- net /Q6: track 7.62 -> 8.67 mm
- net /Q4: track 7.62 -> 8.67 mm
- net /Q2: track 7.62 -> 8.67 mm
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Other:
- board size 73.3 x 39.4 mm -> 71.1 x 39.4 mm
- board text added: "30.01.2025"
- board text removed: "21.03.2024"
